File: KiCad/MCU/M_MUC.kicad_pcb (KiCad board)
At the start: 2 copper layers, 43.2 x 38.1 mm, 13 parts, among them J1 6pin, J2 Conn_01x10, SW1 SW_Push_Open, U1 ATmega328PB-A, Y1 Crystal

Commit message: aua
Connections:
- net Net-(C3-Pad2) renamed /rst
- net Net-(J2-Pad5) renamed /rx
- net Net-(J2-Pad6) renamed /tx
- D1 pad 2: 5V -> unconnected-(D1-A-Pad2)
- U1 pad 12: unconnected-(U1-Pad12) -> unconnected-(D1-A-Pad2)
- U1 pad 13: unconnected-(U1-Pad13) -> unconnected-(D1-A-Pad2)
Routing:
- net 5V: track 54.5 -> 41.1 mm
- net unconnected-(D1-A-Pad2): track 0.00 -> 6.47 mm
