File: KiCad/MCU/M_MUC.kicad_sch (KiCad schematic)
At the start: 11 parts, among them J1 6pin, J2 Conn_01x10, SW1 SW_Push_Open, U1 ATmega328PB-A, Y1 Crystal

Commit message: aua
Connections:
- net +5V: now also U1.12 (PB0), U1.13 (PB1)
- no-connect marks 16 -> 15
Changed lines of the file:
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@@
   (junction (at 157.48 102.87) (diameter 0) (color 0 0 0 0)
+  )
+  (junction (at 148.59 64.77) (diameter 0) (color 0 0 0 0)
   )
   (junction (at 142.24 100.33) (diameter 0) (color 0 0 0 0)
@@
   (no_connect (at 149.86 92.71))
   (no_connect (at 148.59 64.77))
-  (no_connect (at 148.59 67.31))
   (no_connect (at 111.76 107.95))
   (no_connect (at 142.24 125.73))
@@
     (stroke (width 0) (type default))
   )
-  (wire (pts (xy 88.9 111.76) (xy 91.44 111.76))
-    (stroke (width 0) (type default))
-  )
   (wire (pts (xy 168.91 132.08) (xy 177.8 132.08))
     (stroke (width 0) (type default))
@@
     (stroke (width 0) (type default))
   )
+  (wire (pts (xy 148.59 67.31) (xy 148.59 64.77))
+    (stroke (width 0) (type default))
+  )
   (wire (pts (xy 143.51 107.95) (xy 143.51 109.22))
     (stroke (width 0) (type default))
@@
     (stroke (width 0) (type default))
   )
+  (wire (pts (xy 100.33 53.34) (xy 100.33 111.76))
+    (stroke (width 0) (type default))
+  )
   (wire (pts (xy 171.45 64.77) (xy 171.45 67.31))
     (stroke (width 0) (type default))
@@
     (stroke (width 0) (type default))
   )
+  (wire (pts (xy 148.59 64.77) (xy 148.59 53.34))
+    (stroke (width 0) (type default))
+  )
   (wire (pts (xy 173.99 116.84) (xy 177.8 116.84))
     (stroke (width 0) (type default))
@@
     (stroke (width 0) (type default))
   )
+  (wire (pts (xy 148.59 53.34) (xy 100.33 53.34))
+    (stroke (width 0) (type default))
+  )
   (wire (pts (xy 142.24 72.39) (xy 158.75 72.39))
     (stroke (width 0) (type default))
@@
   )
   (wire (pts (xy 142.24 64.77) (xy 148.59 64.77))
+    (stroke (width 0) (type default))
+  )
+  (wire (pts (xy 88.9 111.76) (xy 100.33 111.76))
     (stroke (width 0) (type default))
   )
@@
   (text "INT0" (at 149.86 113.03 0)
     (effects (font (size 0.9 0.9)) (justify left bottom))
+  )
+  (text "OC1A" (at 93.98 111.76 0)
+    (effects (font (size 0.8 0.8)) (justify left bottom))
   )
   (text "ADC0" (at 149.86 87.63 0)
@@
         )
       )
-    )
-  )
-  (symbol (lib_id "power:+5V") (at 91.44 111.76 270) (unit 1)
-    (in_bom yes) (on_board yes) (dnp no)
-    (property "Reference" "#PWR0106" (at 87.63 111.76 0)
-      (effects (font (size 1.27 1.27)) hide)
-    )
-    (property "Value" "+5V" (at 95.25 111.76 0)
-      (effects (font (size 1.27 1.27)))
-    )
-    (property "Footprint" "" (at 91.44 111.76 0)
-      (effects (font (size 1.27 1.27)) hide)
-    )
-    (property "Datasheet" "" (at 91.44 111.76 0)
-      (effects (font (size 1.27 1.27)) hide)
-    )
-    (pin "1")
-    (instances
-      (project "M_MUC"
-        (path "/8f0e16c9-4bd2-4a25-a569-54925ece9d23"
-          (reference "#PWR0106") (unit 1)
-        )
-      )
