File: KiCad/RPS01/5V_Buck.kicad_sch (KiCad schematic)
At the start: 0 parts

Commit message: 5V Buck Schematic and Some Components
Parts:
- added C(STBYMD)1, Css1: 0.001u, Capacitor_SMD:C_1206_3216Metric, symbol Device:C
- added C(lowESR)1: 4.7u, Mechatronic Footprints:LOWESRCAPMP7.6X4.3_3.1N_KEM, symbol Device:C
- added Ca(SW1)1, Cb(SW2)1: 0.22u, Capacitor_SMD:C_1206_3216Metric, symbol Device:C
- added Cb(out)1: 330u, Mechatronic Footprints:LargeCAPSCAPPRD350W60D800H1200, symbol Device:C_Polarized
- added Cc(out)1: 47u, Capacitor_SMD:C_1206_3216Metric, symbol Device:C
- added Cin(b)1: 270u, Mechatronic Footprints:LargeCAPSCAPPRD350W60D800H1200, symbol Device:C
- added Cin(c)1: 10u, Capacitor_SMD:C_1206_3216Metric, symbol Device:C
- added Cout(filter)1: 330u, Mechatronic Footprints:LargeCAPSCAPPRD350W60D800H1200, symbol Device:C
- added Cs1: 100p, Capacitor_SMD:C_1206_3216Metric, symbol Device:C
- added Cth1: 10000p, Capacitor_SMD:C_1206_3216Metric, symbol Device:C
- added Cthp1: 47p, Capacitor_SMD:C_1206_3216Metric, symbol Device:C
- added D(Zener)2: D_Zener, Mechatronic Footprints:SOD123_DIO, symbol Device:D_Zener
- added D1, D2, D4, D5: D_Schottky, Mechatronic Footprints:CR_SMA_320-340AE_DIO, symbol Device:D_Schottky
- added L1: 6.8u, Mechatronic Footprints:IND_410680_WRE, symbol Device:L
- added Q1, Q2, Q3, Q4: NMOS, Mechatronic Footprints:Q1Q2TRANS_FDMC86520L, symbol Device:Q_NMOS_DGS
- added R(pgood)1: 100k, LED_SMD:LED_1206_3216Metric, symbol Device:R
- added R4, R5: 100, Resistor_SMD:R_1206_3216Metric, symbol Device:R
- added Rb1: 4.3K, Resistor_SMD:R_1206_3216Metric, symbol Device:R
- added Rin(Run)1: 51K, Resistor_SMD:R_1206_3216Metric, symbol Device:R
- added Rs1, Rsen1: 6m, Resistor_SMD:R_2512_6332Metric, symbol Device:R
- added Rt1: 100K, Resistor_SMD:R_1206_3216Metric, symbol Device:R
- added Rth1: 124K, Resistor_SMD:R_1206_3216Metric, symbol Device:R
- added U1: LTC3780EG-TRPBF, LTC3780:SSOP-24_G_LIT, symbol LTC3780-24-SSOP:LTC3780EG-TRPBF
Connections:
- new net: D2.2 (A), Q2.3 (S), Q4.3 (S), R4.1, Rs1.1, Rsen1.1
- new net: Cs1.2, R4.2, U1.3 (SENSE+)
- new net: R(pgood)1.2, U1.1 (PGOOD)
- new net: C(STBYMD)1.1, U1.12 (STBYMD)
- new net: Cb(SW2)1.2, D5.1 (K), U1.13 (BOOST2)
- new net: Q1.2 (G), U1.14 (TG2)
- new net: Cb(SW2)1.1, D2.1 (K), L1.1, Q1.3 (S), Q2.1 (D), U1.15 (SW2)
- new net: Q2.2 (G), U1.16 (BG2)
- new net: Q4.2 (G), U1.18 (BG1)
- new net: C(lowESR)1.1, D4.2 (A), D5.2 (A), R(pgood)1.1, U1.19 (INTVCC)
- new net: Css1.2, U1.2 (SS)
- new net: Ca(SW1)1.2, D1.2 (A), L1.2, Q3.3 (S), Q4.1 (D), U1.22 (SW1)
- new net: Q3.2 (G), U1.23 (TG1)
- new net: Ca(SW1)1.1, D4.1 (K), U1.24 (BOOST1)
- new net: Cs1.1, R5.1, U1.4 (SENSE-)
- new net: Cthp1.1, Rth1.2, U1.5 (ITH)
- new net: Rb1.1, Rt1.2, U1.6 (VOSENSE)
- new net: D(Zener)2.1 (K), Rin(Run)1.2, U1.8 (RUN)
- new net: Cth1.1, Rth1.1
- new net GND: C(STBYMD)1.2, C(lowESR)1.2, Cb(out)1.2, Cc(out)1.2, Cin(b)1.2, Cin(c)1.2, Cout(filter)1.2, Css1.1, Cth1.2, Cthp1.2, D(Zener)2.2 (A), R5.2, Rb1.2, Rs1.2, Rsen1.2, U1.10 (PLLFLTR), U1.17 (PGND), U1.20 (EXTVCC), U1.7 (SGND), U1.9 (FCB)
- new net Vin: Cin(b)1.1, Cin(c)1.1, Q1.1 (D), Rin(Run)1.1, U1.21 (VIN)
- new net Vout: Cb(out)1.1, Cc(out)1.1, Cout(filter)1.1, D1.1 (K), Q3.1 (D), Rt1.1
- no-connect marks 0 -> 1

Commit message: Changed footprints on my end only
Parts:
- U1: footprint LTC3780:SSOP-24_G_LIT -> Mechatronics LTC3780:SSOP-24_G_LIT
Changed lines of the file:
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@@
       (effects (font (size 1.524 1.524)))
     )
-    (property "Footprint" "LTC3780:SSOP-24_G_LIT" (at 99.0854 109.8804 0)
+    (property "Footprint" "Mechatronics LTC3780:SSOP-24_G_LIT" (at 99.0854 109.8804 0)
       (effects (font (size 1.27 1.27) italic) hide)
     )

Commit message: All Footprints Load from Mechatronics Folder
Parts:
- U1: footprint Mechatronics LTC3780:SSOP-24_G_LIT -> Mechatronic Footprints:LTC3780_SSOP-24_G_LIT
Changed lines of the file:
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@@
       (effects (font (size 1.524 1.524)))
     )
-    (property "Footprint" "Mechatronics LTC3780:SSOP-24_G_LIT" (at 99.0854 109.8804 0)
+    (property "Footprint" "Mechatronic Footprints:LTC3780_SSOP-24_G_LIT" (at 99.0854 109.8804 0)
       (effects (font (size 1.27 1.27) italic) hide)
     )
