File: KiCad/RPS01/LLC.kicad_sch (KiCad schematic)
At the start: 0 parts

Commit message: LLC schematic
Parts:
- added Q1, Q2: BSS138, Package_TO_SOT_SMD:SOT-23, symbol Transistor_FET:BSS138
- added R3 (x2), R4 (x2): 10K, symbol Device:R
Connections:
- new net +3.3V: Q1.1 (G), Q2.1 (G), R3.1, R3.1
- new net +5V: R4.1, R4.1
- new net LV1: Q1.2 (S), Q2.2 (S), R3.2, R3.2
- new net SCL: Q1.3 (D), R4.2
- new net SDA: Q2.3 (D), R4.2

Commit message: 4.7K R
Parts:
- removed Q1, Q2: BSS138, Package_TO_SOT_SMD:SOT-23, symbol Transistor_FET:BSS138
- removed R3 (x2), R4 (x2): 10K, symbol Device:R

Commit message: fix LLC and add temperature sensor  page
Parts:
- added Q1, Q2: BSS138, Package_TO_SOT_SMD:SOT-23, symbol Transistor_FET:BSS138
- added R3 (x2), R4 (x2): 10K, symbol Device:R
Connections:
- new net +3.3V: Q1.1 (G), Q2.1 (G), R3.1, R3.1
- new net +5V: R4.1, R4.1
- new net LV1: Q1.2 (S), Q2.2 (S), R3.2, R3.2
- new net SCL: Q1.3 (D), R4.2
- new net SDA: Q2.3 (D), R4.2

Commit message: Large Schematic Update
Parts:
- added R10, R9: 0, symbol Device:R_Small
- added R4 (x2): 4.7K, Resistor_SMD:R_0603_1608Metric, symbol Device:R
Connections:
- net SCL: now also Q2.2 (S), R3.2, R10.1; no longer Q1.3 (D), R4.2
- net SDA: now also Q1.2 (S), R3.2, R9.1; no longer Q2.3 (D), R4.2
- removed net LV1: Q1.2 (S), Q2.2 (S), R3.2, R3.2
- new net GND: R4.1, R4.1
- new net SCL 5V: Q2.3 (D), R10.2, R4.2
- new net SDA 5V: Q1.3 (D), R4.2, R9.2

Commit message: Finished most of the Schematics. Needs polishing
Parts:
- renumbered R3 to R11, R3 to R12, R9 to R13, R10 to R14, R4 to R15, R4 to R16
Connections:
- net SCL 5V: now also R4.2
- net SDA 5V: now also R4.2
- net +5V renamed LOGIC 5V
Other:
- moved on the sheet: R4
