File: KiCad/RPS01/Inputs.kicad_sch (KiCad schematic)
At the start: 4 parts, among them SW1 Display Button, SW1 RST

Commit message: Finished Updating Footprints and Reorganized Reference Designators
Finished Updating Footprints and Reorganized Reference Designators

Starting to work on Final PCB, except for 19V Boost. Please check Schematic for errors
Parts:
- renumbered R4 to R?, SW1 to SW?
Changed lines of the file:
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@@
   (symbol (lib_id "power:GND") (at 78.74 44.196 0) (unit 1)
     (in_bom yes) (on_board yes) (dnp no) (fields_autoplaced)
-    (property "Reference" "#PWR03" (at 78.74 50.546 0)
+    (property "Reference" "#PWR?" (at 78.74 50.546 0)
       (effects (font (size 1.27 1.27)) hide)
     )
@@
       (project "MCU2"
         (path "/049009a7-95d1-4ccf-a10c-7859cfd6b188"
-          (reference "#PWR03") (unit 1)
-        )
-      )
-      (project "rps01"
-        (path "/14930f15-c0a0-4b55-93e6-b112548415f6/a2e49fe6-126d-427d-b045-54fb7f662aa7"
-          (reference "#PWR024") (unit 1)
-        )
-        (path "/14930f15-c0a0-4b55-93e6-b112548415f6/423e72dd-bb18-4d03-a22d-0f9c41f98256"
-          (reference "#PWR053") (unit 1)
-        )
-      )
-      (project "M_MUC"
-        (path "/8f0e16c9-4bd2-4a25-a569-54925ece9d23"
-          (reference "#PWR0105") (unit 1)
+          (reference "#PWR?") (unit 1)
+        )
+      )
+      (project "rps01"
+        (path "/14930f15-c0a0-4b55-93e6-b112548415f6/a2e49fe6-126d-427d-b045-54fb7f662aa7"
+          (reference "#PWR?") (unit 1)
+        )
+        (path "/14930f15-c0a0-4b55-93e6-b112548415f6/423e72dd-bb18-4d03-a22d-0f9c41f98256"
+          (reference "#PWR055") (unit 1)
+        )
+      )
+      (project "M_MUC"
+        (path "/8f0e16c9-4bd2-4a25-a569-54925ece9d23"
+          (reference "#PWR?") (unit 1)
         )
       )
@@
   (symbol (lib_id "power:GND") (at 78.994 66.548 0) (unit 1)
     (in_bom yes) (on_board yes) (dnp no) (fields_autoplaced)
-    (property "Reference" "#PWR03" (at 78.994 72.898 0)
+    (property "Reference" "#PWR?" (at 78.994 72.898 0)
       (effects (font (size 1.27 1.27)) hide)
     )
@@
       (project "MCU2"
         (path "/049009a7-95d1-4ccf-a10c-7859cfd6b188"
-          (reference "#PWR03") (unit 1)
-        )
-      )
-      (project "rps01"
-        (path "/14930f15-c0a0-4b55-93e6-b112548415f6/a2e49fe6-126d-427d-b045-54fb7f662aa7"
-          (reference "#PWR024") (unit 1)
-        )
-        (path "/14930f15-c0a0-4b55-93e6-b112548415f6/423e72dd-bb18-4d03-a22d-0f9c41f98256"
-          (reference "#PWR054") (unit 1)
-        )
-      )
-      (project "M_MUC"
-        (path "/8f0e16c9-4bd2-4a25-a569-54925ece9d23"
-          (reference "#PWR0105") (unit 1)
+          (reference "#PWR?") (unit 1)
+        )
+      )
+      (project "rps01"
+        (path "/14930f15-c0a0-4b55-93e6-b112548415f6/a2e49fe6-126d-427d-b045-54fb7f662aa7"
+          (reference "#PWR?") (unit 1)
+        )
+        (path "/14930f15-c0a0-4b55-93e6-b112548415f6/423e72dd-bb18-4d03-a22d-0f9c41f98256"
+          (reference "#PWR056") (unit 1)
+        )
+      )
+      (project "M_MUC"
+        (path "/8f0e16c9-4bd2-4a25-a569-54925ece9d23"
+          (reference "#PWR?") (unit 1)
         )
       )
@@
   (symbol (lib_id "Device:R") (at 67.564 74.168 90) (unit 1)
     (in_bom yes) (on_board yes) (dnp no)
-    (property "Reference" "R4" (at 67.564 69.088 90)
+    (property "Reference" "R?" (at 67.564 69.088 90)
       (effects (font (size 1.27 1.27)))
     )
@@
       (project "MCU2"
         (path "/049009a7-95d1-4ccf-a10c-7859cfd6b188"
-          (reference "R4") (unit 1)
-        )
-      )
-      (project "rps01"
-        (path "/14930f15-c0a0-4b55-93e6-b112548415f6/a2e49fe6-126d-427d-b045-54fb7f662aa7"
-          (reference "R3") (unit 1)
-        )
-        (path "/14930f15-c0a0-4b55-93e6-b112548415f6/423e72dd-bb18-4d03-a22d-0f9c41f98256"
-          (reference "R29") (unit 1)
-        )
-      )
-      (project "M_MUC"
-        (path "/8f0e16c9-4bd2-4a25-a569-54925ece9d23"
-          (reference "R1") (unit 1)
+          (reference "R?") (unit 1)
+        )
+      )
+      (project "rps01"
+        (path "/14930f15-c0a0-4b55-93e6-b112548415f6/a2e49fe6-126d-427d-b045-54fb7f662aa7"
+          (reference "R?") (unit 1)
+        )
+        (path "/14930f15-c0a0-4b55-93e6-b112548415f6/423e72dd-bb18-4d03-a22d-0f9c41f98256"
+          (reference "R35") (unit 1)
+        )
+      )
+      (project "M_MUC"
+        (path "/8f0e16c9-4bd2-4a25-a569-54925ece9d23"
+          (reference "R?") (unit 1)
         )
       )
@@
   (symbol (lib_id "Device:R") (at 67.31 51.816 90) (unit 1)
     (in_bom yes) (on_board yes) (dnp no)
-    (property "Reference" "R4" (at 67.31 46.736 90)
+    (property "Reference" "R?" (at 67.31 46.736 90)
       (effects (font (size 1.27 1.27)))
     )
@@
       (project "MCU2"
         (path "/049009a7-95d1-4ccf-a10c-7859cfd6b188"
-          (reference "R4") (unit 1)
-        )
-      )
-      (project "rps01"
-        (path "/14930f15-c0a0-4b55-93e6-b112548415f6/a2e49fe6-126d-427d-b045-54fb7f662aa7"
-          (reference "R3") (unit 1)
-        )
-        (path "/14930f15-c0a0-4b55-93e6-b112548415f6/423e72dd-bb18-4d03-a22d-0f9c41f98256"
-          (reference "R28") (unit 1)
-        )
-      )
-      (project "M_MUC"
-        (path "/8f0e16c9-4bd2-4a25-a569-54925ece9d23"
-          (reference "R1") (unit 1)
+          (reference "R?") (unit 1)
+        )
+      )
+      (project "rps01"
+        (path "/14930f15-c0a0-4b55-93e6-b112548415f6/a2e49fe6-126d-427d-b045-54fb7f662aa7"
+          (reference "R?") (unit 1)
+        )
+        (path "/14930f15-c0a0-4b55-93e6-b112548415f6/423e72dd-bb18-4d03-a22d-0f9c41f98256"
+          (reference "R34") (unit 1)
+        )
+      )
+      (project "M_MUC"
+        (path "/8f0e16c9-4bd2-4a25-a569-54925ece9d23"
+          (reference "R?") (unit 1)
         )
       )
@@
   (symbol (lib_id "Switch:SW_Push_Open") (at 70.104 66.548 180) (unit 1)
     (in_bom yes) (on_board yes) (dnp no) (fields_autoplaced)
-    (property "Reference" "SW1" (at 70.104 62.23 0)
+    (property "Reference" "SW?" (at 70.104 62.23 0)
       (effects (font (size 1.27 1.27)))
     )
@@
       (project "MCU2"
         (path "/049009a7-95d1-4ccf-a10c-7859cfd6b188"
+          (reference "SW?") (unit 1)
+        )
+      )
+      (project "rps01"
+        (path "/14930f15-c0a0-4b55-93e6-b112548415f6/a2e49fe6-126d-427d-b045-54fb7f662aa7"
+          (reference "SW?") (unit 1)
+        )
+        (path "/14930f15-c0a0-4b55-93e6-b112548415f6/423e72dd-bb18-4d03-a22d-0f9c41f98256"
+          (reference "SW2") (unit 1)
+        )
+      )
+      (project "M_MUC"
+        (path "/8f0e16c9-4bd2-4a25-a569-54925ece9d23"
+          (reference "SW?") (unit 1)
+        )
+      )
+    )
+  )
+  (symbol (lib_id "Switch:SW_Push_Open") (at 69.85 44.196 180) (unit 1)
+    (in_bom yes) (on_board yes) (dnp no) (fields_autoplaced)
+    (property "Reference" "SW?" (at 69.85 39.37 0)
+      (effects (font (size 1.27 1.27)))
+    )
+    (property "Value" "RST" (at 69.85 41.91 0)
+      (effects (font (size 1.27 1.27)))
+    )
+    (property "Footprint" "Button_Switch_SMD:SW_SPST_PTS645" (at 69.85 49.276 0)
+      (effects (font (size 1.27 1.27)) hide)
+    )
+    (property "Datasheet" "~" (at 69.85 49.276 0)
+      (effects (font (size 1.27 1.27)) hide)
+    )
+    (pin "1")
+    (pin "2")
+    (instances
+      (project "MCU2"
+        (path "/049009a7-95d1-4ccf-a10c-7859cfd6b188"
+          (reference "SW?") (unit 1)
+        )
+      )
+      (project "rps01"
+        (path "/14930f15-c0a0-4b55-93e6-b112548415f6/a2e49fe6-126d-427d-b045-54fb7f662aa7"
+          (reference "SW?") (unit 1)
+        )
+        (path "/14930f15-c0a0-4b55-93e6-b112548415f6/423e72dd-bb18-4d03-a22d-0f9c41f98256"
           (reference "SW1") (unit 1)
         )
       )
-      (project "rps01"
-        (path "/14930f15-c0a0-4b55-93e6-b112548415f6/a2e49fe6-126d-427d-b045-54fb7f662aa7"
-          (reference "SW1") (unit 1)
-        )
-        (path "/14930f15-c0a0-4b55-93e6-b112548415f6/423e72dd-bb18-4d03-a22d-0f9c41f98256"
-          (reference "SW2") (unit 1)
-        )
-      )
-      (project "M_MUC"
-        (path "/8f0e16c9-4bd2-4a25-a569-54925ece9d23"
-          (reference "SW1") (unit 1)
-        )
-      )
-    )
-  )
-  (symbol (lib_id "Switch:SW_Push_Open") (at 69.85 44.196 180) (unit 1)
-    (in_bom yes) (on_board yes) (dnp no) (fields_autoplaced)
-    (property "Reference" "SW1" (at 69.85 39.37 0)
-      (effects (font (size 1.27 1.27)))
-    )
-    (property "Value" "RST" (at 69.85 41.91 0)
-      (effects (font (size 1.27 1.27)))
-    )
-    (property "Footprint" "Button_Switch_SMD:SW_SPST_PTS645" (at 69.85 49.276 0)
-      (effects (font (size 1.27 1.27)) hide)
-    )
-    (property "Datasheet" "~" (at 69.85 49.276 0)
-      (effects (font (size 1.27 1.27)) hide)
-    )
-    (pin "1")
-    (pin "2")
-    (instances
-      (project "MCU2"
-        (path "/049009a7-95d1-4ccf-a10c-7859cfd6b188"
-          (reference "SW1") (unit 1)
-        )
-      )
-      (project "rps01"
-        (path "/14930f15-c0a0-4b55-93e6-b112548415f6/a2e49fe6-126d-427d-b045-54fb7f662aa7"
-          (reference "SW1") (unit 1)
-        )
-        (path "/14930f15-c0a0-4b55-93e6-b112548415f6/423e72dd-bb18-4d03-a22d-0f9c41f98256"
-          (reference "SW1") (unit 1)
-        )
-      )
-      (project "M_MUC"
-        (path "/8f0e16c9-4bd2-4a25-a569-54925ece9d23"
-          (reference "SW1") (unit 1)
-        )
-      )
+      (project "M_MUC"
+        (path "/8f0e16c9-4bd2-4a25-a569-54925ece9d23"
+          (reference "SW?") (unit 1)
+        )
+      )
