File: KiCad/RPS01/TempSensors.kicad_sch (KiCad schematic)
At the start: 5 parts, among them U17 DS18B20+, U18 DS18B20+

Commit message: Getting THERE. ALMOST THERE
Parts:
- U17, U18: footprint Mechatronics TEMP:21-0248A_Q3-1_MXM -> Package_TO_SOT_THT:TO-92L_Inline
Changed lines of the file:
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@@
       (effects (font (size 1.524 1.524)))
     )
-    (property "Footprint" "Mechatronics TEMP:21-0248A_Q3-1_MXM" (at 52.578 153.416 0)
+    (property "Footprint" "Package_TO_SOT_THT:TO-92L_Inline" (at 52.578 153.416 0)
       (effects (font (size 1.27 1.27) italic) hide)
     )
@@
       (effects (font (size 1.524 1.524)))
     )
-    (property "Footprint" "Mechatronics TEMP:21-0248A_Q3-1_MXM" (at 53.086 124.968 0)
+    (property "Footprint" "Package_TO_SOT_THT:TO-92L_Inline" (at 53.086 124.968 0)
       (effects (font (size 1.27 1.27) italic) hide)
     )
