File: KiCad/RPS01/Probe.kicad_sch (KiCad schematic)
At the start: 19 parts

Commit message: update probe text and start fuse model
Parts:
- TP13: value VOLT1 -> 3.3V
- TP14: value VOLT2 -> 5V
- TP15: value AREF -> 12V
- TP16: value LOGIC 5V -> 19V
- TP17: value LOGIC 5V -> GND
Changed lines of the file:
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@@
   (symbol (lib_id "Connector:TestPoint_Probe") (at 92.964 138.938 0) (unit 1)
     (in_bom yes) (on_board yes) (dnp no) (fields_autoplaced)
-    (property "Reference" "TP13" (at 97.536 136.7155 0)
-      (effects (font (size 1.27 1.27)) (justify left))
-    )
-    (property "Value" "VOLT1" (at 97.536 139.2555 0)
+    (property "Reference" "TP13" (at 97.79 136.7155 0)
+      (effects (font (size 1.27 1.27)) (justify left))
+    )
+    (property "Value" "3.3V" (at 97.79 139.2555 0)
       (effects (font (size 1.27 1.27)) (justify left))
     )
@@
   (symbol (lib_id "Connector:TestPoint_Probe") (at 92.71 165.608 0) (unit 1)
     (in_bom yes) (on_board yes) (dnp no) (fields_autoplaced)
-    (property "Reference" "TP17" (at 97.282 163.3855 0)
-      (effects (font (size 1.27 1.27)) (justify left))
-    )
-    (property "Value" "LOGIC 5V" (at 97.282 165.9255 0)
+    (property "Reference" "TP17" (at 96.52 163.3855 0)
+      (effects (font (size 1.27 1.27)) (justify left))
+    )
+    (property "Value" "GND" (at 96.52 165.9255 0)
       (effects (font (size 1.27 1.27)) (justify left))
     )
@@
   (symbol (lib_id "Connector:TestPoint_Probe") (at 92.964 159.258 0) (unit 1)
     (in_bom yes) (on_board yes) (dnp no) (fields_autoplaced)
-    (property "Reference" "TP16" (at 97.536 157.0355 0)
-      (effects (font (size 1.27 1.27)) (justify left))
-    )
-    (property "Value" "LOGIC 5V" (at 97.536 159.5755 0)
+    (property "Reference" "TP16" (at 97.79 157.0355 0)
+      (effects (font (size 1.27 1.27)) (justify left))
+    )
+    (property "Value" "19V" (at 97.79 159.5755 0)
       (effects (font (size 1.27 1.27)) (justify left))
     )
@@
   (symbol (lib_id "Connector:TestPoint_Probe") (at 92.964 152.654 0) (unit 1)
     (in_bom yes) (on_board yes) (dnp no) (fields_autoplaced)
-    (property "Reference" "TP15" (at 97.536 150.4315 0)
-      (effects (font (size 1.27 1.27)) (justify left))
-    )
-    (property "Value" "AREF" (at 97.536 152.9715 0)
+    (property "Reference" "TP15" (at 97.79 150.4315 0)
+      (effects (font (size 1.27 1.27)) (justify left))
+    )
+    (property "Value" "12V" (at 97.79 152.9715 0)
       (effects (font (size 1.27 1.27)) (justify left))
     )
@@
   (symbol (lib_id "Connector:TestPoint_Probe") (at 92.964 145.796 0) (unit 1)
     (in_bom yes) (on_board yes) (dnp no) (fields_autoplaced)
-    (property "Reference" "TP14" (at 97.536 143.5735 0)
-      (effects (font (size 1.27 1.27)) (justify left))
-    )
-    (property "Value" "VOLT2" (at 97.536 146.1135 0)
-      (effects (font (size 1.27 1.27)) (justify left))
-    )
+    (property "Reference" "TP14" (at 97.79 143.5735 0)
+      (effects (font (size 1.27 1.27)) (justify left))
+    )
+    (property "Value" "5V" (at 97.79 146.1135 0)
+      (effects (font (size 1.27 1.27)) (justify left))
+    )
