File: KiCad/MCU2/MCU2.kicad_pcb (KiCad board)
At the start: 2 copper layers, 9 parts, among them J1 Conn_02x03_Counter_Clockwise, J2 Conn_01x06, J3 Conn_01x03, SW1 MCU_Button, U1 ATmega328P-A

Commit message: New Update
Parts:
- added C2: 0.1uf, Capacitor_SMD:C_1206_3216Metric, F.Cu at (108.3, 86.2)
- added C3: 0.1uf, Capacitor_SMD:C_1206_3216Metric, F.Cu at (113.3, 86.2)
- added J4: Conn_01x02_Pin, Connector_PinHeader_2.54mm:PinHeader_1x02_P2.54mm_Vertical, F.Cu at (118.0, 84.8)
- added J5: XT30, Connector_AMASS:AMASS_XT30U-F_1x02_P5.0mm_Vertical, F.Cu at (108.1, 62.1)
- added J6: AandDpin, Connector_PinHeader_2.54mm:PinHeader_1x02_P2.54mm_Vertical, F.Cu at (124.6, 87.6)
- added U2: AMS1117, Package_TO_SOT_SMD:SOT-223-3_TabPin2, F.Cu at (110.4, 71.4)
- added U3: ADR02AUJZ-REEL7, footprints:UJ_5_ADI, F.Cu at (110.6, 81.2)
- C1: footprint Capacitor_SMD:C_1206_3216Metric -> Connector_PinHeader_2.54mm:PinHeader_1x02_P2.54mm_Vertical
- moved R4 31.7 mm to (125.9, 61.3), turned to 180 degrees
- moved C1 28.2 mm to (125.9, 66.0), turned to -90 degrees
- moved J1 18.1 mm to (142.5, 74.8)
- moved J3 17.6 mm to (141.4, 67.9), turned to 180 degrees
- moved SW1 9.79 mm to (135.6, 60.5), turned to -90 degrees
- moved R1 7.63 mm to (138.3, 86.5)
- moved J2 6.52 mm to (118.0, 67.3)
- moved D1 5.63 mm to (133.4, 86.7), turned to 180 degrees
Connections:
- net Net-(J2-Pin_5) renamed /RST
- J1 pad 1: GND -> /MISO
- J1 pad 2: /RESET -> /SCK
- J1 pad 3: Net-(J1-Pin_3) -> /RESET
- J1 pad 4: Net-(J1-Pin_4) -> GND
- J1 pad 5: Net-(J1-Pin_5) -> /MOSI
- J1 pad 6: Net-(J1-Pin_6) -> +5V
- J2 pad 1: Net-(J2-Pin_1) -> +5V
- J3 pad 2: /SCK -> /SCL
- R4 pad 2: Net-(R4-Pad2) -> +5V
- U1 pad 10: unconnected-(U1-PD6-Pad10) -> /Analog
- U1 pad 15: Net-(J1-Pin_3) -> /MOSI
- U1 pad 16: Net-(J1-Pin_6) -> /MISO
- U1 pad 17: Net-(J1-Pin_4) -> /SCK
- U1 pad 20: unconnected-(U1-AREF-Pad20) -> /AREF
- U1 pad 28: /SCK -> /SCL
- U1 pad 4: Net-(U1-VCC-Pad4) -> +5V
- U1 pad 6: Net-(U1-VCC-Pad4) -> +5V
- U1 pad 9: unconnected-(U1-PD5-Pad9) -> /Digital
Routing:
- net +5V: track 0.00 -> 68.9 mm, vias 0 -> 4
- net /RESET: track 0.00 -> 41.8 mm, vias 0 -> 2
- net /AREF: track 0.00 -> 30.7 mm, vias 0 -> 2
- net /RST: track 0.00 -> 17.6 mm, vias 0 -> 2
- net /RX: track 0.00 -> 14.1 mm
- net /SCL: track 0.00 -> 13.6 mm
- net /TX: track 0.00 -> 13.5 mm
- net /MOSI: track 0.00 -> 13.2 mm
- net /SCK: track 0.00 -> 13.0 mm
- net /SDA: track 0.00 -> 11.9 mm
- net /MISO: track 0.00 -> 11.5 mm
- net /VI: track 0.00 -> 11.3 mm
- net /Analog: track 0.00 -> 9.13 mm
- net Net-(D1-A): track 0.00 -> 6.72 mm
- net /Digital: track 0.00 -> 6.26 mm
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- added copper zone on B.Cu, net GND
- added copper zone on F.Cu, net GND

Commit message: update
Routing:
- net /VI: track 11.3 -> 37.3 mm
- net /VOUT: track 4.16 -> 11.4 mm
- net /RESET: track 41.8 -> 45.9 mm
- net /Analog: track 9.13 -> 10.8 mm
- net +5V: track 68.9 -> 70.6 mm
- net GND: vias 0 -> 12
Other:
- board outline added: 47.6 x 37.1 mm

Commit message: update
Routing:
- net GND: track 0.00 -> 7.14 mm
Changed lines of the file:
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@@
         (effects (font (size 0.5 0.5) (thickness 0.125)))
     )
-    (fp_text value "MCU_LED" (at 5.461 -0.254 90) (layer "F.Fab")
+    (fp_text value "MCU_LED" (at 1.402 -3.556 180) (layer "F.Fab")
         (effects (font (size 0.5 0.5) (thickness 0.125)))
     )
@@
   (segment (start 130.727 80.057) (end 130.727 86.653) (width 0.25) (layer "F.Cu") (net 3))
   (segment (start 130.727 86.653) (end 130.815 86.741) (width 0.25) (layer "F.Cu") (net 3))
+  (segment (start 126.077 76.207) (end 127.12 76.207) (width 0.25) (layer "F.Cu") (net 4))
+  (segment (start 127.12 76.207) (end 127.889 75.438) (width 0.25) (layer "F.Cu") (net 4))
+  (segment (start 134.577 75.407) (end 132.938 75.407) (width 0.25) (layer "F.Cu") (net 4))
+  (segment (start 126.077 74.607) (end 127.058 74.607) (width 0.25) (layer "F.Cu") (net 4))
+  (segment (start 127.058 74.607) (end 127.889 75.438) (width 0.25) (layer "F.Cu") (net 4))
+  (segment (start 132.938 75.407) (end 132.08 74.549) (width 0.25) (layer "F.Cu") (net 4))
   (via (at 127.889 75.438) (size 0.8) (drill 0.4) (layers "F.Cu" "B.Cu") (free) (net 4))
   (via (at 127.127 84.455) (size 0.8) (drill 0.4) (layers "F.Cu" "B.Cu") (free) (net 4))

Commit message: 0.0
Routing:
- net +5V: track 70.6 -> 76.9 mm
Changed lines of the file:
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@@
     (property "ki_keywords" "capacitor cap")
     (attr through_hole)
-    (fp_text reference "C1" (at 0 -2.33 90) (layer "F.SilkS")
-        (effects (font (size 1 1) (thickness 0.15)))
-    )
-    (fp_text value "100nF" (at 0 4.87 90) (layer "F.Fab")
-        (effects (font (size 1 1) (thickness 0.15)))
-    )
-    (fp_text user "${REFERENCE}" (at -2.667 0.132) (layer "F.Fab")
+    (fp_text reference "C1" (at -1.905 -3.043 90) (layer "F.SilkS")
+        (effects (font (size 1 1) (thickness 0.15)))
+    )
+    (fp_text value "100nF" (at -2.286 1.021) (layer "F.Fab")
+        (effects (font (size 0.5 0.5) (thickness 0.125)))
+    )
+    (fp_text user "${REFERENCE}" (at -9.398 0.259) (layer "F.Fab")
         (effects (font (size 1 1) (thickness 0.15)))
     )
@@
         (effects (font (size 0.5 0.5) (thickness 0.125)))
     )
-    (fp_text value "10K" (at 0 1.82) (layer "F.Fab")
+    (fp_text value "10K" (at 0.127 2.159) (layer "F.Fab")
         (effects (font (size 1 1) (thickness 0.15)))
     )
@@
   (segment (start 137.414 79.629) (end 137.414 75.184) (width 0.25) (layer "B.Cu") (net 35))
   (segment (start 122.682 82.042) (end 135.001 82.042) (width 0.25) (layer "B.Cu") (net 35))
+  (segment (start 110.363 74.524) (end 110.363 68.224) (width 0.25) (layer "F.Cu") (net 36))
   (segment (start 117.983 67.31) (end 119.761 67.31) (width 0.25) (layer "F.Cu") (net 36))
   (segment (start 111.438 66.899) (end 117.572 66.899) (width 0.25) (layer "F.Cu") (net 36))
