File: KiCad/MCU2/MCU2.kicad_sch (KiCad schematic)
At the start: 9 parts, among them J1 Conn_02x03_Counter_Clockwise, J2 Conn_01x06, J3 Conn_01x03, SW1 MCU_Button, U1 ATmega328P-A

Commit message: update
Parts:
- added C2, C3: 0.1uf, Capacitor_SMD:C_1206_3216Metric, symbol Device:C_Small
- added J4: Conn_01x02_Pin, Connector_PinHeader_2.54mm:PinHeader_1x02_P2.54mm_Vertical, symbol Connector:Conn_01x02_Pin
- added J5: XT30, Connector_AMASS:AMASS_XT30U-F_1x02_P5.0mm_Vertical, symbol Connector:Conn_01x02_Pin
- added U2: AMS1117, Package_TO_SOT_SMD:SOT-223-3_TabPin2, symbol Regulator_Linear:AMS1117
- added U3: ADR02AUJZ-REEL7, footprints:UJ_5_ADI, symbol 2023-06-26_00-14-37:ADR02AUJZ-REEL7
Connections:
- net GND: now also J1.4 (Pin_4), C2.2, C3.2, J5.2 (Pin_2), U2.1 (ADJ), U3.2 (GND); no longer J1.1 (Pin_1)
- net RESET: now also J1.3 (Pin_3); no longer J1.2 (Pin_2)
- net SCK: now also J1.2 (Pin_2), U1.17 (PB5); no longer J3.2 (Pin_2), U1.28 (PC5)
- net MOSI: now reaches U1.15 (PB3)
- net MOSI: now also J1.5 (Pin_5); no longer J1.3 (Pin_3)
- net at J1.6 (Pin_6): no longer U1.16 (PB4)
- net at U1.20 (AREF): now also J4.2 (Pin_2)
- net at U1.4 (VCC), U1.6 (VCC): now also U2.2 (VO)
- new net: C2.1, J5.1 (Pin_1), U2.3 (VI), U3.3 (VIN)
- new net: C3.1, J4.1 (Pin_1), U3.4 (VOUT)
- new net MISO: J1.1 (Pin_1), U1.16 (PB4)
- new net SCL: J3.2 (Pin_2), U1.28 (PC5)
- no-connect marks 19 -> 20
Other:
- moved on the sheet: C1, D1, J1, J2, J3, R1, R4, SW1, U1

Commit message: New Update
Parts:
- added J6: AandDpin, Connector_PinHeader_2.54mm:PinHeader_1x02_P2.54mm_Vertical, symbol Connector:Conn_01x02_Pin
- C1: footprint Capacitor_SMD:C_1206_3216Metric -> Connector_PinHeader_2.54mm:PinHeader_1x02_P2.54mm_Vertical
Connections:
- net +5V: now reaches J2.1 (Pin_1)
- net +5V: now also J1.6 (Pin_6), R4.2, U1.4 (VCC), U1.6 (VCC), U2.2 (VO)
- net RST: now reaches C1.2, J2.5 (Pin_5)
- net VI: now reaches C2.1, J5.1 (Pin_1), U2.3 (VI), U3.3 (VIN)
- net Analog: now reaches U1.10 (PD6)
- net Analog: now also J6.1 (Pin_1)
- net AREF: now reaches J4.2 (Pin_2), U1.20 (AREF)
- net Digital: now reaches U1.9 (PD5)
- net Digital: now also J6.2 (Pin_2)
- net VOUT: now reaches C3.1, J4.1 (Pin_1), U3.4 (VOUT)
- no-connect marks 20 -> 18

Commit message: update
Parts:
- added C4, C5: 0.22pf, Capacitor_THT:C_Disc_D3.0mm_W1.6mm_P2.50mm, symbol Device:C_Small
- added Y1: Crystal, Crystal:Crystal_HC49-4H_Vertical, symbol Device:Crystal
- C1: footprint Connector_PinHeader_2.54mm:PinHeader_1x02_P2.54mm_Vertical -> Capacitor_THT:C_Disc_D3.0mm_W1.6mm_P2.50mm
Connections:
- net GND: now also C4.2, C5.2
- net at U1.7 (XTAL1/PB6): now also C4.1, Y1.1
- net at U1.8 (XTAL2/PB7): now also C5.1, Y1.2
- no-connect marks 18 -> 16
Changed lines of the file:
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@@
   (junction (at 165.506 113.3348) (diameter 0) (color 0 0 0 0)
   )
+  (junction (at 176.1744 48.006) (diameter 0) (color 0 0 0 0)
+  )
   (junction (at 81.1628 73.6092) (diameter 0) (color 0 0 0 0)
   )
-  (no_connect (at 134.0612 94.3864))
+  (junction (at 199.0852 48.006) (diameter 0) (color 0 0 0 0)
+  )
   (no_connect (at 16.4084 68.5292))
   (no_connect (at 134.0612 124.8664))
@@
   (no_connect (at 134.0612 137.5664))
   (no_connect (at 134.0612 81.6864))
-  (no_connect (at 134.0612 91.8464))
   (no_connect (at 134.0612 107.0864))
   (no_connect (at 103.5812 81.6864))
@@
     (stroke (width 0) (type default))
   )
+  (wire (pts (xy 186.69 48.006) (xy 199.0852 48.006))
+    (stroke (width 0) (type default))
+  )
   (wire (pts (xy 165.506 90.0684) (xy 172.6692 90.0684))
     (stroke (width 0) (type default))
@@
     (stroke (width 0) (type default))
   )
+  (wire (pts (xy 147.4216 72.6948) (xy 171.7548 72.6948))
+    (stroke (width 0) (type default))
+  )
   (wire (pts (xy 204.9272 120.9548) (xy 211.9376 120.9548))
     (stroke (width 0) (type default))
@@
     (stroke (width 0) (type default))
   )
+  (wire (pts (xy 134.0612 91.8464) (xy 147.4216 91.8464))
+    (stroke (width 0) (type default))
+  )
+  (wire (pts (xy 199.0852 48.006) (xy 207.6704 48.006))
+    (stroke (width 0) (type default))
+  )
   (wire (pts (xy 172.6692 90.0684) (xy 172.6692 90.1192))
     (stroke (width 0) (type default))
@@
     (stroke (width 0) (type default))
   )
+  (wire (pts (xy 207.6704 48.006) (xy 207.6704 94.3864))
+    (stroke (width 0) (type default))
+  )
   (wire (pts (xy 145.288 99.4664) (xy 154.7876 99.4664))
     (stroke (width 0) (type default))
@@
     (stroke (width 0) (type default))
   )
+  (wire (pts (xy 176.1744 48.006) (xy 179.07 48.006))
+    (stroke (width 0) (type default))
+  )
   (wire (pts (xy 96.012 66.0908) (xy 96.012 67.5132))
     (stroke (width 0) (type default))
   )
+  (wire (pts (xy 199.0852 63.9572) (xy 199.0344 63.9572))
+    (stroke (width 0) (type default))
+  )
   (wire (pts (xy 148.082 102.0064) (xy 154.7876 102.0064))
     (stroke (width 0) (type default))
@@
     (stroke (width 0) (type default))
   )
+  (wire (pts (xy 171.7548 72.6948) (xy 171.7548 48.006))
+    (stroke (width 0) (type default))
+  )
+  (wire (pts (xy 147.4216 91.8464) (xy 147.4216 72.6948))
+    (stroke (width 0) (type default))
+  )
   (wire (pts (xy 70.8152 48.26) (xy 72.7456 48.26))
     (stroke (width 0) (type default))
@@
     (stroke (width 0) (type default))
   )
+  (wire (pts (xy 171.7548 48.006) (xy 176.1744 48.006))
+    (stroke (width 0) (type default))
+  )
   (wire (pts (xy 187.9092 90.1192) (xy 187.9092 90.0684))
     (stroke (width 0) (type default))
@@
     (stroke (width 0) (type default))
   )
+  (wire (pts (xy 176.1744 58.5724) (xy 176.1744 63.1952))
+    (stroke (width 0) (type default))
+  )
   (wire (pts (xy 139.7 108.4072) (xy 145.288 108.4072))
     (stroke (width 0) (type default))
@@
     (stroke (width 0) (type default))
   )
+  (wire (pts (xy 176.1744 63.1952) (xy 176.3268 63.1952))
+    (stroke (width 0) (type default))
+  )
   (wire (pts (xy 92.2528 86.106) (xy 92.2528 84.328))
     (stroke (width 0) (type default))
@@
     (stroke (width 0) (type default))
   )
+  (wire (pts (xy 176.1744 53.4924) (xy 176.1744 48.006))
+    (stroke (width 0) (type default))
+  )
   (wire (pts (xy 103.5812 76.6064) (xy 103.2256 76.6064))
     (stroke (width 0) (type default))
@@
     (stroke (width 0) (type default))
   )
+  (wire (pts (xy 207.6704 94.3864) (xy 134.0612 94.3864))
+    (stroke (width 0) (type default))
+  )
+  (wire (pts (xy 199.0852 58.7756) (xy 199.0852 63.9572))
+    (stroke (width 0) (type default))
+  )
   (wire (pts (xy 134.0612 119.8372) (xy 148.8563 119.8372))
     (stroke (width 0) (type default))
@@
   )
   (wire (pts (xy 103.2256 76.6064) (xy 103.2256 66.0908))
+    (stroke (width 0) (type default))
+  )
+  (wire (pts (xy 199.0852 53.6956) (xy 199.0852 48.006))
     (stroke (width 0) (type default))
   )
@@
     )
   )
+  (symbol (lib_id "power:GND") (at 199.0344 63.9572 0) (unit 1)
+    (in_bom yes) (on_board yes) (dnp no) (fields_autoplaced)
+    (property "Reference" "#PWR016" (at 199.0344 70.3072 0)
+      (effects (font (size 1.27 1.27)) hide)
+    )
+    (property "Value" "GND" (at 199.0344 68.7324 0)
+      (effects (font (size 1.27 1.27)))
+    )
+    (property "Footprint" "" (at 199.0344 63.9572 0)
+      (effects (font (size 1.27 1.27)) hide)
+    )
+    (property "Datasheet" "" (at 199.0344 63.9572 0)
+      (effects (font (size 1.27 1.27)) hide)
+    )
+    (pin "1")
+    (instances
+      (project "MCU2"
+        (path "/049009a7-95d1-4ccf-a10c-7859cfd6b188"
+          (reference "#PWR016") (unit 1)
+        )
+      )
+    )
+  )
+  (symbol (lib_id "Device:C_Small") (at 176.1744 56.0324 0) (unit 1)
+    (in_bom yes) (on_board yes) (dnp no)
+    (property "Reference" "C4" (at 178.7144 53.4924 0)
+      (effects (font (size 0.5 0.5)) (justify left))
+    )
+    (property "Value" "0.22pf" (at 178.7144 54.7624 0)
+      (effects (font (size 0.6 0.6)) (justify left))
+    )
+    (property "Footprint" "Capacitor_THT:C_Disc_D3.0mm_W1.6mm_P2.50mm" (at 176.1744 56.0324 0)
+      (effects (font (size 1.27 1.27)) hide)
+    )
+    (property "Datasheet" "~" (at 176.1744 56.0324 0)
+      (effects (font (size 1.27 1.27)) hide)
+    )
+    (pin "1")
+    (pin "2")
+    (instances
+      (project "MCU2"
+        (path "/049009a7-95d1-4ccf-a10c-7859cfd6b188"
+          (reference "C4") (unit 1)
+        )
+      )
+      (project "rps01"
+        (path "/14930f15-c0a0-4b55-93e6-b112548415f6/a2e49fe6-126d-427d-b045-54fb7f662aa7"
+          (reference "C3") (unit 1)
+        )
+      )
+    )
+  )
+  (symbol (lib_id "Device:Crystal") (at 182.88 48.006 0) (unit 1)
+    (in_bom yes) (on_board yes) (dnp no) (fields_autoplaced)
+    (property "Reference" "Y1" (at 182.88 41.91 0)
+      (effects (font (size 1.27 1.27)))
+    )
+    (property "Value" "Crystal" (at 182.88 44.45 0)
+      (effects (font (size 1.27 1.27)))
+    )
+    (property "Footprint" "Crystal:Crystal_HC49-4H_Vertical" (at 182.88 48.006 0)
+      (effects (font (size 1.27 1.27)) hide)
+    )
+    (property "Datasheet" "~" (at 182.88 48.006 0)
+      (effects (font (size 1.27 1.27)) hide)
+    )
+    (pin "1")
+    (pin "2")
+    (instances
+      (project "MCU2"
+        (path "/049009a7-95d1-4ccf-a10c-7859cfd6b188"
+          (reference "Y1") (unit 1)
+        )
+      )
+    )
+  )
   (symbol (lib_id "Device:R") (at 148.336 58.4708 90) (unit 1)
     (in_bom yes) (on_board yes) (dnp no)
@@
         (path "/049009a7-95d1-4ccf-a10c-7859cfd6b188"
           (reference "#PWR07") (unit 1)
+        )
+      )
+    )
+  )
+  (symbol (lib_id "Device:C_Small") (at 199.0852 56.2356 0) (unit 1)
+    (in_bom yes) (on_board yes) (dnp no)
+    (property "Reference" "C5" (at 201.6252 53.6956 0)
+      (effects (font (size 0.5 0.5)) (justify left))
+    )
+    (property "Value" "0.22pf" (at 201.6252 54.9656 0)
+      (effects (font (size 0.6 0.6)) (justify left))
+    )
+    (property "Footprint" "Capacitor_THT:C_Disc_D3.0mm_W1.6mm_P2.50mm" (at 199.0852 56.2356 0)
+      (effects (font (size 1.27 1.27)) hide)
+    )
+    (property "Datasheet" "~" (at 199.0852 56.2356 0)
+      (effects (font (size 1.27 1.27)) hide)
+    )
+    (pin "1")
+    (pin "2")
+    (instances
+      (project "MCU2"
+        (path "/049009a7-95d1-4ccf-a10c-7859cfd6b188"
+          (reference "C5") (unit 1)
+        )
+      )
+      (project "rps01"
+        (path "/14930f15-c0a0-4b55-93e6-b112548415f6/a2e49fe6-126d-427d-b045-54fb7f662aa7"
+          (reference "C3") (unit 1)
         )
       )
@@
     )
   )
+  (symbol (lib_id "power:GND") (at 176.3268 63.1952 0) (unit 1)
+    (in_bom yes) (on_board yes) (dnp no) (fields_autoplaced)
+    (property "Reference" "#PWR015" (at 176.3268 69.5452 0)
+      (effects (font (size 1.27 1.27)) hide)
+    )
+    (property "Value" "GND" (at 176.3268 68.8848 0)
+      (effects (font (size 1.27 1.27)))
+    )
+    (property "Footprint" "" (at 176.3268 63.1952 0)
+      (effects (font (size 1.27 1.27)) hide)
+    )
+    (property "Datasheet" "" (at 176.3268 63.1952 0)
+      (effects (font (size 1.27 1.27)) hide)
+    )
+    (pin "1")
+    (instances
+      (project "MCU2"
+        (path "/049009a7-95d1-4ccf-a10c-7859cfd6b188"
+          (reference "#PWR015") (unit 1)
+        )
+      )
+    )
+  )
   (symbol (lib_id "Connector:Conn_01x02_Pin") (at 101.092 70.0532 180) (unit 1)
     (in_bom yes) (on_board yes) (dnp no)
@@
       (effects (font (size 0.6 0.6)) (justify left))
     )
-    (property "Footprint" "Connector_PinHeader_2.54mm:PinHeader_1x02_P2.54mm_Vertical" (at 204.9272 118.4148 0)
-      (effects (font (size 1.27 1.27)) hide)
-    )
+    (property "Footprint" "Capacitor_THT:C_Disc_D3.0mm_W1.6mm_P2.50mm" (at 204.9272 118.4148 0)
+      (effects (font (size 1.27 1.27)) hide)
+    )

Commit message: update
Connections:
- net SCK: now also D1.2 (A)
- net at U1.13 (PB1): no longer D1.2 (A)
- no-connect marks 16 -> 17
Changed lines of the file:
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@@
   (junction (at 165.506 113.3348) (diameter 0) (color 0 0 0 0)
+  )
+  (junction (at 159.302 89.3064) (diameter 0) (color 0 0 0 0)
   )
   (junction (at 176.1744 48.006) (diameter 0) (color 0 0 0 0)
@@
   (no_connect (at 134.0612 127.4064))
   (no_connect (at 121.3612 68.9864))
+  (no_connect (at 134.0612 79.1464))
   (no_connect (at 77.3684 68.5292))
   (no_connect (at 134.0612 137.5664))
@@
     (stroke (width 0) (type default))
   )
+  (wire (pts (xy 147.4216 72.6948) (xy 147.4216 91.8464))
+    (stroke (width 0) (type default))
+  )
   (wire (pts (xy 77.3684 73.6092) (xy 81.1628 73.6092))
     (stroke (width 0) (type default))
@@
     (stroke (width 0) (type default))
   )
-  (wire (pts (xy 163.576 67.3608) (xy 138.3792 67.3608))
-    (stroke (width 0) (type default))
-  )
   (wire (pts (xy 140.716 58.4708) (xy 144.526 58.4708))
     (stroke (width 0) (type default))
@@
     (stroke (width 0) (type default))
   )
-  (wire (pts (xy 163.576 62.2808) (xy 163.576 67.3608))
+  (wire (pts (xy 159.302 88.3412) (xy 159.302 89.3064))
     (stroke (width 0) (type default))
   )
@@
     (stroke (width 0) (type default))
   )
-  (wire (pts (xy 147.4216 91.8464) (xy 147.4216 72.6948))
-    (stroke (width 0) (type default))
-  )
   (wire (pts (xy 70.8152 48.26) (xy 72.7456 48.26))
     (stroke (width 0) (type default))
@@
     (stroke (width 0) (type default))
   )
+  (wire (pts (xy 163.576 62.2808) (xy 163.576 88.3412))
+    (stroke (width 0) (type default))
+  )
   (wire (pts (xy 139.7 108.4072) (xy 145.288 108.4072))
     (stroke (width 0) (type default))
@@
     (stroke (width 0) (type default))
   )
+  (wire (pts (xy 159.302 89.3064) (xy 169.672 89.3064))
+    (stroke (width 0) (type default))
+  )
   (wire (pts (xy 148.8563 119.8372) (xy 148.8563 125.4252))
     (stroke (width 0) (type default))
   )
-  (wire (pts (xy 138.3792 67.3608) (xy 138.3792 79.1464))
-    (stroke (width 0) (type default))
-  )
   (wire (pts (xy 204.9272 113.3348) (xy 204.9272 114.6048))
     (stroke (width 0) (type default))
@@
     (stroke (width 0) (type default))
   )
-  (wire (pts (xy 138.3792 79.1464) (xy 134.0612 79.1464))
+  (wire (pts (xy 163.576 88.3412) (xy 159.302 88.3412))
     (stroke (width 0) (type default))
   )
@@
     (stroke (width 0) (type default))
   )
-  (wire (pts (xy 134.0612 89.3064) (xy 169.672 89.3064))
-    (stroke (width 0) (type default))
-  )
+  (wire (pts (xy 134.0612 89.3064) (xy 159.302 89.3064))
+    (stroke (width 0) (type default))
+  )

Commit message: 111
Parts:
- added J7: Conn_01x03, Connector_PinHeader_2.54mm:PinHeader_1x03_P2.54mm_Vertical, symbol Connector_Generic:Conn_01x03
Connections:
- net at U1.23 (PC0): now also J7.3 (Pin_3)
- net at U1.24 (PC1): now also J7.2 (Pin_2)
- net at U1.25 (PC2): now also J7.1 (Pin_1)
- no-connect marks 17 -> 13
Other:
- moved on the sheet: J3
Changed lines of the file:
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@@
   (no_connect (at 134.0612 124.8664))
   (no_connect (at 134.0612 76.6064))
-  (no_connect (at 134.0612 104.5464))
   (no_connect (at 134.0612 127.4064))
   (no_connect (at 121.3612 68.9864))
@@
   (no_connect (at 103.5812 81.6864))
   (no_connect (at 134.0612 129.9464))
-  (no_connect (at 103.5812 84.2264))
-  (no_connect (at 134.0612 99.4664))
   (no_connect (at 165.608 133.0452))
-  (no_connect (at 134.0612 102.0064))
   (wire (pts (xy 112.2172 49.022) (xy 118.8212 49.022))
     (stroke (width 0) (type default))
@@
     (stroke (width 0) (type default))
   )
+  (wire (pts (xy 224.9932 79.5528) (xy 226.7204 79.5528))
+    (stroke (width 0) (type default))
+  )
   (wire (pts (xy 221.4372 106.9848) (xy 225.2472 106.9848))
     (stroke (width 0) (type default))
   )
+  (wire (pts (xy 136.8044 98.9584) (xy 226.1108 98.9584))
+    (stroke (width 0) (type default))
+  )
   (wire (pts (xy 164.084 120.396) (xy 165.608 120.396))
     (stroke (width 0) (type default))
   )
-  (wire (pts (xy 154.7876 104.4956) (xy 154.7876 104.5464))
-    (stroke (width 0) (type default))
-  )
-  (wire (pts (xy 145.288 108.4072) (xy 145.288 99.4664))
-    (stroke (width 0) (type default))
-  )
-  (wire (pts (xy 148.082 111.2134) (xy 148.082 102.0064))
+  (wire (pts (xy 155.3972 107.5944) (xy 155.3972 107.6452))
+    (stroke (width 0) (type default))
+  )
+  (wire (pts (xy 145.288 108.4072) (xy 145.288 102.5652))
+    (stroke (width 0) (type default))
+  )
+  (wire (pts (xy 148.082 111.2134) (xy 148.082 105.1052))
     (stroke (width 0) (type default))
   )
@@
     (stroke (width 0) (type default))
   )
+  (wire (pts (xy 226.1108 77.0128) (xy 226.7204 77.0128))
+    (stroke (width 0) (type default))
+  )
+  (wire (pts (xy 224.9932 97.79) (xy 224.9932 79.5528))
+    (stroke (width 0) (type default))
+  )
+  (wire (pts (xy 222.4024 82.0928) (xy 226.7204 82.0928))
+    (stroke (width 0) (type default))
+  )
   (wire (pts (xy 80.4164 51.5112) (xy 80.4164 48.9712))
     (stroke (width 0) (type default))
@@
     (stroke (width 0) (type default))
   )
-  (wire (pts (xy 145.288 99.4664) (xy 154.7876 99.4664))
+  (wire (pts (xy 145.288 102.5652) (xy 155.3972 102.5652))
     (stroke (width 0) (type default))
   )
@@
     (stroke (width 0) (type default))
   )
+  (wire (pts (xy 222.4024 96.1644) (xy 222.4024 82.0928))
+    (stroke (width 0) (type default))
+  )
   (wire (pts (xy 140.716 58.4708) (xy 144.526 58.4708))
     (stroke (width 0) (type default))
@@
     (stroke (width 0) (type default))
   )
-  (wire (pts (xy 148.082 102.0064) (xy 154.7876 102.0064))
+  (wire (pts (xy 226.1108 98.9584) (xy 226.1108 77.0128))
+    (stroke (width 0) (type default))
+  )
+  (wire (pts (xy 148.082 105.1052) (xy 155.3972 105.1052))
     (stroke (width 0) (type default))
   )
@@
     (stroke (width 0) (type default))
   )
-  (wire (pts (xy 152.2984 104.4956) (xy 154.7876 104.4956))
+  (wire (pts (xy 151.9428 107.5944) (xy 155.3972 107.5944))
     (stroke (width 0) (type default))
   )
@@
     (stroke (width 0) (type default))
   )
+  (wire (pts (xy 134.0612 99.4664) (xy 134.0612 96.1644))
+    (stroke (width 0) (type default))
+  )
   (wire (pts (xy 81.1628 51.5112) (xy 80.4164 51.5112))
     (stroke (width 0) (type default))
   )
+  (wire (pts (xy 136.8044 104.5464) (xy 136.8044 98.9584))
+    (stroke (width 0) (type default))
+  )
   (wire (pts (xy 118.8212 49.022) (xy 118.8212 68.9864))
     (stroke (width 0) (type default))
@@
     (stroke (width 0) (type default))
   )
+  (wire (pts (xy 134.0612 96.1644) (xy 222.4024 96.1644))
+    (stroke (width 0) (type default))
+  )
   (wire (pts (xy 204.9272 114.6048) (xy 204.9272 115.8748))
     (stroke (width 0) (type default))
@@
     (stroke (width 0) (type default))
   )
+  (wire (pts (xy 134.0612 102.0064) (xy 135.5344 102.0064))
+    (stroke (width 0) (type default))
+  )
   (wire (pts (xy 176.1744 63.1952) (xy 176.3268 63.1952))
     (stroke (width 0) (type default))
@@
     (stroke (width 0) (type default))
   )
+  (wire (pts (xy 135.5344 97.79) (xy 224.9932 97.79))
+    (stroke (width 0) (type default))
+  )
   (wire (pts (xy 84.4296 99.1616) (xy 84.4296 100.2792))
     (stroke (width 0) (type default))
@@
     (stroke (width 0) (type default))
   )
+  (wire (pts (xy 135.5344 102.0064) (xy 135.5344 97.79))
+    (stroke (width 0) (type default))
+  )
   (wire (pts (xy 78.8416 48.9712) (xy 78.8416 45.72))
     (stroke (width 0) (type default))
@@
   )
   (wire (pts (xy 204.9272 114.6048) (xy 208.7372 114.6048))
+    (stroke (width 0) (type default))
+  )
+  (wire (pts (xy 134.0612 104.5464) (xy 136.8044 104.5464))
     (stroke (width 0) (type default))
   )
@@
     (effects (font (size 1.27 1.27)) (justify left bottom))
   )
-  (label "SDA" (at 148.1933 99.4664 0) (fields_autoplaced)
+  (label "SDA" (at 148.1933 102.5652 0) (fields_autoplaced)
     (effects (font (size 1.27 1.27)) (justify left bottom))
   )
@@
     (effects (font (size 1.27 1.27)) (justify left bottom))
   )
-  (label "SCL" (at 150.7707 102.0064 0) (fields_autoplaced)
+  (label "SCL" (at 150.7707 105.1052 0) (fields_autoplaced)
     (effects (font (size 1.27 1.27)) (justify left bottom))
   )
@@
     )
   )
-  (symbol (lib_id "power:GND") (at 152.2984 104.4956 270) (unit 1)
+  (symbol (lib_id "power:GND") (at 151.9428 107.5944 270) (unit 1)
     (in_bom yes) (on_board yes) (dnp no)
-    (property "Reference" "#PWR05" (at 145.9484 104.4956 0)
-      (effects (font (size 1.27 1.27)) hide)
-    )
-    (property "Value" "GND" (at 153.9748 107.3404 90)
+    (property "Reference" "#PWR05" (at 145.5928 107.5944 0)
+      (effects (font (size 1.27 1.27)) hide)
+    )
+    (property "Value" "GND" (at 153.6192 110.4392 90)
       (effects (font (size 1.27 1.27)) (justify right))
     )
-    (property "Footprint" "" (at 152.2984 104.4956 0)
-      (effects (font (size 1.27 1.27)) hide)
-    )
-    (property "Datasheet" "" (at 152.2984 104.4956 0)
+    (property "Footprint" "" (at 151.9428 107.5944 0)
+      (effects (font (size 1.27 1.27)) hide)
+    )
+    (property "Datasheet" "" (at 151.9428 107.5944 0)
       (effects (font (size 1.27 1.27)) hide)
     )
@@
         (path "/049009a7-95d1-4ccf-a10c-7859cfd6b188"
           (reference "#PWR06") (unit 1)
+        )
+      )
+    )
+  )
+  (symbol (lib_id "Connector_Generic:Conn_01x03") (at 231.8004 79.5528 0) (unit 1)
+    (in_bom yes) (on_board yes) (dnp no) (fields_autoplaced)
+    (property "Reference" "J7" (at 234.95 78.9178 0)
+      (effects (font (size 1.27 1.27)) (justify left))
+    )
+    (property "Value" "Conn_01x03" (at 234.95 81.4578 0)
+      (effects (font (size 1.27 1.27)) (justify left))
+    )
+    (property "Footprint" "Connector_PinHeader_2.54mm:PinHeader_1x03_P2.54mm_Vertical" (at 231.8004 79.5528 0)
+      (effects (font (size 1.27 1.27)) hide)
+    )
+    (property "Datasheet" "~" (at 231.8004 79.5528 0)
+      (effects (font (size 1.27 1.27)) hide)
+    )
+    (pin "1")
+    (pin "2")
+    (pin "3")
+    (instances
+      (project "MCU2"
+        (path "/049009a7-95d1-4ccf-a10c-7859cfd6b188"
+          (reference "J7") (unit 1)
         )
       )
@@
     )
   )
-  (symbol (lib_id "Connector_Generic:Conn_01x03") (at 159.8676 102.0064 0) (unit 1)
-    (in_bom yes) (on_board yes) (dnp no) (fields_autoplaced)
-    (property "Reference" "J3" (at 162.6616 101.3714 0)
+  (symbol (lib_id "Connector_Generic:Conn_01x03") (at 160.4772 105.1052 0) (unit 1)
+    (in_bom yes) (on_board yes) (dnp no) (fields_autoplaced)
+    (property "Reference" "J3" (at 163.2712 104.4702 0)
       (effects (font (size 1.27 1.27)) (justify left))
     )
-    (property "Value" "Conn_01x03" (at 162.6616 103.9114 0)
+    (property "Value" "Conn_01x03" (at 163.2712 107.0102 0)
       (effects (font (size 1.27 1.27)) (justify left))
     )
-    (property "Footprint" "Connector_PinHeader_2.54mm:PinHeader_1x03_P2.54mm_Vertical" (at 159.8676 102.0064 0)
-      (effects (font (size 1.27 1.27)) hide)
-    )
-    (property "Datasheet" "~" (at 159.8676 102.0064 0)
-      (effects (font (size 1.27 1.27)) hide)
-    )
+    (property "Footprint" "Connector_PinHeader_2.54mm:PinHeader_1x03_P2.54mm_Vertical" (at 160.4772 105.1052 0)
+      (effects (font (size 1.27 1.27)) hide)
+    )
+    (property "Datasheet" "~" (at 160.4772 105.1052 0)
+      (effects (font (size 1.27 1.27)) hide)
+    )
