File: KiCad/MCU2/MCU2.kicad_sch (KiCad schematic)
At the start: 20 parts, among them J1 Conn_02x03_Counter_Clockwise, J2 Conn_01x06, J3 Conn_01x03, J4 Conn_01x02_Pin, J5 XT30, J6 AandDpin, J7 Conn_01x03, SW1 MCU_Button, U1 ATmega328P-A, U2 AMS1117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

Commit message: More
Connections:
- net GND: now also J5.1 (Pin_1); no longer J5.2 (Pin_2)
- net VI: now also J5.2 (Pin_2); no longer J5.1 (Pin_1)
Changed lines of the file:
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@@
     (stroke (width 0) (type default))
   )
-  (wire (pts (xy 78.8416 48.9712) (xy 80.4164 48.9712))
+  (wire (pts (xy 70.8152 48.9712) (xy 80.4164 48.9712))
     (stroke (width 0) (type default))
   )
@@
     (stroke (width 0) (type default))
   )
-  (wire (pts (xy 72.7456 48.26) (xy 72.7456 48.3108))
-    (stroke (width 0) (type default))
-  )
   (wire (pts (xy 81.1628 73.6092) (xy 84.5312 73.6092))
     (stroke (width 0) (type default))
@@
     (stroke (width 0) (type default))
   )
-  (wire (pts (xy 70.8152 48.26) (xy 72.7456 48.26))
-    (stroke (width 0) (type default))
-  )
   (wire (pts (xy 84.5312 94.0816) (xy 84.4296 94.0816))
     (stroke (width 0) (type default))
@@
     (stroke (width 0) (type default))
   )
+  (wire (pts (xy 70.8152 45.72) (xy 74.93 45.72))
+    (stroke (width 0) (type default))
+  )
   (wire (pts (xy 187.9092 90.1192) (xy 187.9092 90.0684))
     (stroke (width 0) (type default))
@@
     (stroke (width 0) (type default))
   )
+  (wire (pts (xy 70.8152 48.9712) (xy 70.8152 48.26))
+    (stroke (width 0) (type default))
+  )
   (wire (pts (xy 139.7 109.6264) (xy 134.0612 109.6264))
     (stroke (width 0) (type default))
@@
     (stroke (width 0) (type default))
   )
-  (wire (pts (xy 78.8416 48.9712) (xy 78.8416 45.72))
-    (stroke (width 0) (type default))
-  )
-  (wire (pts (xy 78.8416 45.72) (xy 70.8152 45.72))
-    (stroke (width 0) (type default))
-  )
   (wire (pts (xy 211.2772 106.9848) (xy 208.7372 106.9848))
     (stroke (width 0) (type default))
@@
   )
   (wire (pts (xy 165.506 113.3348) (xy 165.506 90.0684))
+    (stroke (width 0) (type default))
+  )
+  (wire (pts (xy 74.93 45.72) (xy 74.93 45.8216))
     (stroke (width 0) (type default))
   )
@@
     )
   )
-  (symbol (lib_id "power:GND") (at 72.7456 48.3108 90) (unit 1)
+  (symbol (lib_id "power:GND") (at 74.93 45.8216 90) (unit 1)
     (in_bom yes) (on_board yes) (dnp no)
-    (property "Reference" "#PWR07" (at 79.0956 48.3108 0)
-      (effects (font (size 1.27 1.27)) hide)
-    )
-    (property "Value" "GND" (at 71.7296 51.6636 90)
+    (property "Reference" "#PWR07" (at 81.28 45.8216 0)
+      (effects (font (size 1.27 1.27)) hide)
+    )
+    (property "Value" "GND" (at 73.1012 43.5356 90)
       (effects (font (size 1.27 1.27)) (justify right))
     )
-    (property "Footprint" "" (at 72.7456 48.3108 0)
-      (effects (font (size 1.27 1.27)) hide)
-    )
-    (property "Datasheet" "" (at 72.7456 48.3108 0)
-      (effects (font (size 1.27 1.27)) hide)
-    )
+    (property "Footprint" "" (at 74.93 45.8216 0)
+      (effects (font (size 1.27 1.27)) hide)
+    )
+    (property "Datasheet" "" (at 74.93 45.8216 0)
+      (effects (font (size 1.27 1.27)) hide)
+    )
