File: KiCad/FuseTestBoard/fuse_test/fuse_test.kicad_sch (KiCad schematic)
At the start: 1 part

Commit message: adjustments to main board revision
Parts:
- removed F1: 0PAL4100XP_VERTICAL, Mechatronic Footprints:0PAL4100XP_VERTICAL, symbol 0pal4100xp:0PAL4100XP_VERTICAL
- added F1: Fuse, Mechatronic Footprints:0PAL1100XP_VERTICAL, symbol Device:Fuse
- added F2: Fuse, Mechatronic Footprints:0PAL4100XP_NO_HOLES, symbol Device:Fuse
Changed lines of the file:
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@@
 (kicad_sch (version 20230121) (generator eeschema)
   (paper "A4")
-  (wire (pts (xy 121.4882 90.5764) (xy 125.8062 90.5764))
+  (wire (pts (xy 143.51 91.44) (xy 160.02 91.44))
     (stroke (width 0) (type default))
   )
-  (wire (pts (xy 153.7462 90.7796) (xy 153.7462 90.5764))
+  (wire (pts (xy 143.51 101.6) (xy 160.02 101.6))
     (stroke (width 0) (type default))
   )
-  (wire (pts (xy 158.3436 90.7796) (xy 153.7462 90.7796))
+  (wire (pts (xy 116.84 91.44) (xy 135.89 91.44))
     (stroke (width 0) (type default))
   )
-  (symbol (lib_id "power:GND") (at 158.3436 90.7796 90) (unit 1)
+  (wire (pts (xy 116.84 101.6) (xy 135.89 101.6))
+    (stroke (width 0) (type default))
+  )
+  (symbol (lib_id "Device:Fuse") (at 139.7 101.6 90) (unit 1)
     (in_bom yes) (on_board yes) (dnp no) (fields_autoplaced)
-    (property "Reference" "#PWR01" (at 164.6936 90.7796 0)
+    (property "Reference" "F2" (at 139.7 96.52 90)
+      (effects (font (size 1.27 1.27)))
+    )
+    (property "Value" "Fuse" (at 139.7 99.06 90)
+      (effects (font (size 1.27 1.27)))
+    )
+    (property "Footprint" "Mechatronic Footprints:0PAL4100XP_NO_HOLES" (at 139.7 103.378 90)
       (effects (font (size 1.27 1.27)) hide)
     )
-    (property "Value" "GND" (at 162.56 91.4146 90)
-      (effects (font (size 1.27 1.27)) (justify right))
-    )
-    (property "Footprint" "" (at 158.3436 90.7796 0)
-      (effects (font (size 1.27 1.27)) hide)
-    )
-    (property "Datasheet" "" (at 158.3436 90.7796 0)
+    (property "Datasheet" "~" (at 139.7 101.6 0)
       (effects (font (size 1.27 1.27)) hide)
     )
     (pin "1")
+    (pin "2")
     (instances
       (project "fuse_test"
         (path "/e5212c57-ae42-434b-bc9f-ebcb13638ff2"
-          (reference "#PWR01") (unit 1)
+          (reference "F2") (unit 1)
         )
       )
     )
   )
-  (symbol (lib_id "0pal4100xp:0PAL4100XP_VERTICAL") (at 139.7762 90.5764 0) (unit 1)
+  (symbol (lib_id "Device:Fuse") (at 139.7 91.44 90) (unit 1)
     (in_bom yes) (on_board yes) (dnp no) (fields_autoplaced)
-    (property "Reference" "F1" (at 139.7762 82.55 0)
+    (property "Reference" "F1" (at 139.7 86.36 90)
       (effects (font (size 1.27 1.27)))
     )
-    (property "Value" "0PAL4100XP_VERTICAL" (at 139.7762 85.09 0)
+    (property "Value" "Fuse" (at 139.7 88.9 90)
       (effects (font (size 1.27 1.27)))
     )
-    (property "Footprint" "Mechatronic Footprints:0PAL4100XP_VERTICAL" (at 139.7762 96.9264 0)
+    (property "Footprint" "Mechatronic Footprints:0PAL1100XP_VERTICAL" (at 139.7 93.218 90)
       (effects (font (size 1.27 1.27)) hide)
     )
-    (property "Datasheet" "" (at 139.7762 86.7664 0)
+    (property "Datasheet" "~" (at 139.7 91.44 0)
       (effects (font (size 1.27 1.27)) hide)
     )
@@
         )
       )
-    )
-  )
-  (symbol (lib_id "power:PWR_FLAG") (at 121.4882 90.5764 90) (unit 1)
-    (in_bom yes) (on_board yes) (dnp no) (fields_autoplaced)
-    (property "Reference" "#FLG01" (at 119.5832 90.5764 0)
-      (effects (font (size 1.27 1.27)) hide)
-    )
-    (property "Value" "PWR_FLAG" (at 118.11 91.2114 90)
-      (effects (font (size 1.27 1.27)) (justify left))
-    )
-    (property "Footprint" "" (at 121.4882 90.5764 0)
-      (effects (font (size 1.27 1.27)) hide)
-    )
-    (property "Datasheet" "~" (at 121.4882 90.5764 0)
-      (effects (font (size 1.27 1.27)) hide)
-    )
-    (pin "1")
-    (instances
-      (project "fuse_test"
-        (path "/e5212c57-ae42-434b-bc9f-ebcb13638ff2"
-          (reference "#FLG01") (unit 1)
-        )
-      )
