File: KiCad/Buck Converter (LM2596)/Buck Converter/Buck Converter.kicad_sch (KiCad schematic)
At the start: 10 parts, among them J1 Conn_01x02_Socket, J2 Conn_01x02_Socket, U1 LM2596S-ADJ

Commit message: Buck Converter
Parts:
- C_FF1: renamed from C_FF; footprint (none) -> Capacitor_SMD:C_1206_3216Metric
- C_IN1: renamed from C_IN; footprint (none) -> Capacitor_SMD:CP_Elec_8x10
- C_OUT1: renamed from C_OUT; footprint (none) -> Capacitor_SMD:CP_Elec_8x10
- D1: footprint (none) -> Mechatronic Footprints:CR_SMA_320-340AE_DIO
- J2: footprint Mechatronic Footprints:AMASS_XT60-M_1x02_P7.20mm_Vertical -> Mechatronic Footprints:AMASS_XT60-F_1x02_P7.20mm_Vertical
- L1: footprint (none) -> CDRH127_LDNP-470MC:IND_CDRH127_LDNP-470MC_SUM
- R1, R2: footprint (none) -> Resistor_SMD:R_1206_3216Metric
Connections:
- net GND: now also J1.1 (Pin_1), J2.1 (Pin_1); no longer J1.2 (Pin_2), J2.2 (Pin_2)
- net at C_IN1.1, U1.1 (VIN): now also J1.2 (Pin_2); no longer J1.1 (Pin_1)
- net at C_FF1.2, C_OUT1.1, L1.2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: now also J2.2 (Pin_2); no longer J2.1 (Pin_1)
Other:
- moved on the sheet: C_FF1, C_IN1, C_OUT1, D1, J1, J2, L1, R1, R2, U1
