File: KiCad/RPS01-Revision 1/Rails.kicad_sch (KiCad schematic)
At the start: 68 parts, among them U20 LTC3780EUH-TRPBF

Commit message: C9 update
Parts:
- C_FF?: value 10.75n -> 9.49n
Changed lines of the file:
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@@
       (effects (font (size 1.27 1.27)))
     )
-    (property "Value" "10.75n" (at 113.538 122.936 90)
+    (property "Value" "9.49n" (at 113.538 122.936 90)
       (effects (font (size 1.27 1.27)))
     )
