File: KiCad/RPS01-Revision 2/rps01.kicad_pcb (KiCad board)
At the start: 2 copper layers, 150 x 100 mm, 199 parts, among them J1 Header Pins, J1 XT90 Battery VOUT 1, J10 IIC Connector, J11 ISCP, J12 Serial, J13 JST_PH_TEMP_SENSOR_1, J14 JST_PH_TEMP_SENSOR_2, J16 RGB LED, J2 BATT IN 1 XT90, J2 Power In, J3 Power Out, J3 XT90 Battery VOUT 2, J4 XT30PW Batt VOUT, J5 BATT IN 2 XT90, J6 XT30 3.3V, J7 XT30 5V, J8 XT30 12V, J9 XT30PW 19V, Q1 BSC009NE2LS5IATMA1 A (TG2)(1A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, Q1 BSS138, Q2 BSC009NE2LS5IATMA1 B (BG2)(1B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, Q2 BSS138, Q3 BSC009NE2LS5IATMA1 C (BG1)(2A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, Q4 BSC009NE2LS5IATMA1 D (TG1)(2B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, SW1 RST, SW2 Display Button, U1 LTC3780EUH-TRPBF, U1 NP100P04PLG-E1-AY, U10 ATmega328P-A, U11 5V AMS1117, U12 3.3V AMS1117, U13 5V AMS1117, U13 UA741CDT, U14 LM2596S-5V, U15 UA741CDT, U16 LM2596S-12V, U17 DS18B20+, U18 DS18B20+, U19 INA139QPWRQ1, U2 NP100P04PLG-E1-AY, U22 ADR02AUJZ-REEL7, U3 NP100P04PLG-E1-AY, U4 LTC4416EMS-1-TRPBF, U5 NP100P04PLG-E1-AY, U6 NP100P04PLG-E1-AY, U7 NP100P04PLG-E1-AY, U8 INA139QPWRQ1, U9 ADR02AUJZ-REEL7, Y1 16M

Commit message: Updates to PCB
Parts:
- removed Q_(A1)1, Q_(B2)1, Q_(C4)1, Q_(D3)1: BSC009NE2LS5IATMA1, Mechatronics MOSFET:PG-TDSON-8_INF
- removed the U13 at (88.1, 123.0)
- added D1: MM3Z5V1ST1G, Diode_SMD:D_SOD-323, F.Cu at (244.6, 108.0)
- added D1_VSENSE1: MMSZ5247BT1G, Diode_SMD:D_SOD-123, F.Cu at (253.1, 101.5)
- added D2: MM3Z5V1ST1G, Diode_SMD:D_SOD-323, F.Cu at (244.6, 111.0)
- added D2_VSENSE1: MMSZ5247BT1G, Diode_SMD:D_SOD-123, F.Cu at (253.1, 104.9)
- added D5: B0540W-7-F, Diode_SMD:D_SOD-123, F.Cu at (245.3, 101.5)
- added D6: B0540W-7-F, Diode_SMD:D_SOD-123, F.Cu at (245.3, 104.9)
- added REF**: MountingHole_3.2mm_M3_Pad_Via, MountingHole:MountingHole_3.2mm_M3_Pad_Via, F.Cu at (101.9, 68.5)
- added R_S2: 3m, Mechatronic Footprints:CSS2H-5930R, B.Cu at (89.5, 68.6)
- added U21: LM340MPX-5.0/NOPB, Package_TO_SOT_SMD:SOT-223-3_TabPin2, F.Cu at (89.1, 52.6)
- C1_CS1: renamed from C1; value 82p -> 0.1uF
- C4, C5: moved to F.Cu
- CF_5VB1: renamed from C9; value 10.25n -> 10.25n OR DNI
- D_12VB1: renamed from D_12VB_1; footprint Mechatronic Footprints:CR_SMA_320-340AE_DIO -> Mechatronic Footprints:SSB43L-E352T_DIODE_DO214AA_MBRS
- D_5VB1: renamed from D_S8; footprint Mechatronic Footprints:CR_SMA_320-340AE_DIO -> Mechatronic Footprints:SSB43L-E352T_DIODE_DO214AA_MBRS
- L2: value 47u -> 53u; footprint Mechatronics BUCK INDUCTOR:IND_CDRH127&slash_LDNP-470MC_SUM -> Mechatronic Footprints:PE-54039SNL_IND_HCI-68_PUL
- L3: value 47u -> 37u; footprint Mechatronics BUCK INDUCTOR:IND_CDRH127&slash_LDNP-470MC_SUM -> Mechatronic Footprints:PE-53932SNLT_IND_HCI-44_PUL
- R17: value 0 -> 0 DNI
- R1_CS1: renamed from R5; value 100k -> 150k
- R1_CS2: renamed from R31; value 100k -> 55.6K
- U11: value 5V AMS1117 -> LM340MPX-5.0/NOPB; moved to F.Cu
- U12: value 3.3V AMS1117 -> 3.3V NCV1117ST33T3G
- U22, U9: footprint Mechatronics VREF:UJ_5_ADI -> Mechatronic Footprints:ADR02AUJZ_REEL7_UJ_5_ADI
- moved REF** 101.6 mm to (201.4, 78.7)
- moved G*** 86.9 mm to (202.2, 44.5)
- moved G*** 84.0 mm to (199.1, 59.7)
- moved U11 70.4 mm to (88.2, 123.0), turned to 0 degrees
- moved R1_CS2 48.5 mm to (164.8, 63.1)
- moved U19 48.5 mm to (158.5, 61.9)
- moved C2_CS2 48.5 mm to (153.7, 62.3)
- moved C1_CS2 48.5 mm to (163.2, 63.1)
- moved F_5LOGIC1 44.1 mm to (128.7, 90.1)
- moved TP17 42.9 mm to (152.2, 131.4)
- moved R3_VSENSE1 38.0 mm to (130.0, 96.5), turned to 0 degrees
- moved R1_VSENSE1 35.9 mm to (125.4, 96.4), turned to 180 degrees
- moved R4_VSENSE1 35.0 mm to (130.0, 98.8), turned to 180 degrees
- moved R2 34.4 mm to (122.2, 97.0), turned to 90 degrees
- moved R3 34.3 mm to (117.7, 96.9), turned to -90 degrees
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- renumbered C_P6 to C1_12VB1, C_FF1 to C1_3LOGIC1, C_F_5_LOGIC_1 to C1_5LOGIC1, C6 to C1_5PREC1, C_P1 to C1_5VB1, C22 to C1_CS2, C_P7 to C2_12VB1, C_FF2 to C2_3LOGIC1, C_FF5 to C2_5LOGIC1, C7 to C2_5PREC1, C_P2 to C2_5VB1, Cf_2 to C2_CS1, Cf_1 to C2_CS2, C_FF3 to C3_5LOGIC1, C16 to C3_5PREC1, C_FF4 to C4_5LOGIC1, C18 to C4_5PREC1, C20 to CF1_VSENSE1, C21 to CF2_VSENSE1, C_12VB_FC1 to CF_12VB1, F5 to F_12VB1, F1 to F_3LOGIC1, F2 to F_5LOGIC1, F4 to F_5VB1, R_12VB_FR1 to R1_12VB1, R_P1 to R1_5VB1, R_P7 to R1_VSENSE1, R_12VB_FR2 to R2_12VB1, R_P2 to R2_5VB1, R_P8 to R2_VSENSE1, R1_12VB_DIV1 to R3_12VB1, R1_5VB_DIV1 to R3_5VB1, R_P9 to R3_VSENSE1, R2_12VB_DIV1 to R4_12VB1, R2_5VB_DIV1 to R4_5VB1, R_P10 to R4_VSENSE1, R30 to RBLUE1, R_V1_Buf_Enable1 to REN1_VSENSE1, R_V2_Buf_Enable1 to REN2_VSENSE1, R28 to RGREEN1, R29 to RRED1, R_V1_Prec_Enable1 to R_5PREC_ENABLE1, R_V2_Prec_Enable1 to R_5PREC_ENABLE2
Connections:
- C2_5LOGIC1 pad 2: Net-(U11-OUT) -> /Voltage Regulator Rails/LOGIC 5V OUT
- C4_5LOGIC1 pad 2: Net-(U11-OUT) -> /Voltage Regulator Rails/LOGIC 5V OUT
- F_5LOGIC1 pad 1: Net-(U11-OUT) -> /Voltage Regulator Rails/LOGIC 5V OUT
- U11 pad 1: GND -> Net-(D2-K)
- U11 pad 2: /Voltage Regulator Rails/LOGIC 5V OUT -> GND
- U11 pad 3: BATTVIN1 -> /Voltage Regulator Rails/LOGIC 5V OUT
Routing:
- net +BATT: track 273.3 -> 76.5 mm, vias 3 -> 1
- net Net-(C2_5VB1-Pad1): track 56.4 -> 0.00 mm
- net LOGIC 5V: track 144.3 -> 96.9 mm
- net (no net): track 616.2 -> 661.8 mm
- net RST: track 35.0 -> 0.00 mm
- net /Voltage Regulator Rails/LOGIC 5V OUT: track 12.6 -> 0.00 mm
- net /Logic Level Converter/IIC VOLT: track 8.46 -> 0.00 mm
- net PD4: track 7.96 -> 0.00 mm
- net unconnected-(J10-Pin_3-Pad3): track 7.95 -> 0.00 mm
- net BATTVIN1: track 51.3 -> 44.0 mm
- net /DPIN5: track 81.1 -> 77.7 mm
- net GND: track 48.3 -> 45.3 mm
- net Net-(J12-Pin_5): track 2.70 -> 0.00 mm
- net Net-(D_5VB1-K): track 23.5 -> 21.6 mm
- net +3.3V: track 16.3 -> 15.3 mm
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
Commit message: updated PCB
Parts:
- removed TP16: 19V, Mechatronics TestP:CONN1_RCU-0C_TEC
- D_5VB1, R3_12VB1, R3_5VB1, R4_12VB1, R4_5VB1: moved to F.Cu
- moved D1 330.2 mm to (-83.7, 71.8)
- moved D1_VSENSE1 330.2 mm to (-75.1, 65.3)
- moved D2 330.2 mm to (-83.7, 74.7)
- moved D2_VSENSE1 330.2 mm to (-75.1, 68.6)
- moved D5 330.2 mm to (-82.9, 65.3)
- moved D6 330.2 mm to (-82.9, 68.6)
- moved D_5VB1 37.1 mm to (168.5, 128.3), turned to 0 degrees
- turned R3_12VB1 to 0 degrees
- turned R3_5VB1 to 0 degrees
- turned R4_12VB1 to 180 degrees
- turned R4_5VB1 to 180 degrees
Routing:
- net +BATT: track 76.5 -> 21.6 mm
- net +19V: track 23.4 -> 0.00 mm
- net Net-(D_5VB1-K): track 21.6 -> 0.00 mm
- net GND: track 45.3 -> 55.2 mm
- net +5V: track 9.34 -> 3.89 mm
- net ADC7: track 2.51 -> 0.00 mm

Commit message: zzzzzzzzzzzupdates
Parts:
- removed TP11: VSHUNT2-, Mechatronics TestP:CONN1_RCU-0C_TEC
- removed TP12: VSHUNT2+, Mechatronics TestP:CONN1_RCU-0C_TEC
- moved TP3 24.3 mm to (137.3, 148.9)
- moved TP4 24.3 mm to (142.5, 149.0)
- moved TP6 24.3 mm to (128.5, 149.9)
- moved TP9 23.2 mm to (121.5, 148.1)
- moved TP8 23.2 mm to (115.8, 148.3)
- moved TP7 23.1 mm to (109.7, 149.1)
- moved TP17 18.4 mm to (155.4, 149.5)
- moved TP10 18.4 mm to (150.4, 149.4)
Changed lines of the file:
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@@
   )
   (footprint "Mechatronics TestP:CONN1_RCU-0C_TEC" (layer "F.Cu")
-    (at 94.15 132.05)
+    (at 109.728 149.098)
     (tags "RCU-0C ")
     (property "Sheetfile" "Probe.kicad_sch")
@@
   )
   (footprint "Mechatronics TestP:CONN1_RCU-0C_TEC" (layer "F.Cu")
-    (at 99.2549 132.1017)
+    (at 115.824 148.336)
     (tags "RCU-0C ")
     (property "Sheetfile" "Probe.kicad_sch")
@@
   )
   (footprint "Mechatronics TestP:CONN1_RCU-0C_TEC" (layer "F.Cu")
-    (at 125.35 131.75)
+    (at 142.474 148.96)
     (tags "RCU-0C ")
     (property "Sheetfile" "Probe.kicad_sch")
@@
   )
   (footprint "Mechatronics TestP:CONN1_RCU-0C_TEC" (layer "F.Cu")
-    (at 147.15 131.25)
+    (at 150.368 149.352)
     (tags "RCU-0C ")
     (property "Sheetfile" "Probe.kicad_sch")
@@
       (net 39 "LOAD SHARING VOUT") (pinfunction "V-") (pintype "power_in"))
   )
-  (footprint "Mechatronics TestP:CONN1_RCU-0C_TEC" (layer "F.Cu")
-    (at 128.8669 31.6357)
-    (tags "RCU-0C ")
-    (property "Sheetfile" "CurrentSense2_sch.kicad_sch")
-    (property "Sheetname" "Current Sense Rails")
-    (property "ki_description" "test point (alternative probe-style design)")
-    (property "ki_keywords" "test point tp")
-    (attr smd)
-    (fp_text reference "TP12" (at 0.111821 -1.37768 unlocked) (layer "F.SilkS")
-        (effects (font (size 1 1) (thickness 0.15)))
-    )
-    (fp_text value "VSHUNT2+" (at 0 0 unlocked) (layer "F.Fab")
-        (effects (font (size 1 1) (thickness 0.15)))
-    )
-    (fp_text user "VSHUNT2+" (at 0.001283 1.275643 unlocked) (layer "F.SilkS")
-        (effects (font (size 0.5 0.5) (thickness 0.125)))
-    )
-    (fp_text user "${REFERENCE}" (at 0 0 unlocked) (layer "F.Fab")
-        (effects (font (size 1 1) (thickness 0.15)))
-    )
-    (fp_circle (center -2.7051 0) (end -2.3241 0)
-      (stroke (width 0.508) (type solid)) (fill none) (layer "B.SilkS"))
-    (fp_circle (center -2.7051 0) (end -2.3241 0)
-      (stroke (width 0.508) (type solid)) (fill none) (layer "F.SilkS"))
-    (fp_line (start -1.0541 -0.6604) (end -1.0541 0.6604)
-      (stroke (width 0.1524) (type solid)) (layer "F.CrtYd"))
-    (fp_line (start -1.0541 0.6604) (end 1.0541 0.6604)
-      (stroke (width 0.1524) (type solid)) (layer "F.CrtYd"))
-    (fp_line (start 1.0541 -0.6604) (end -1.0541 -0.6604)
-      (stroke (width 0.1524) (type solid)) (layer "F.CrtYd"))
-    (fp_line (start 1.0541 0.6604) (end 1.0541 -0.6604)
-      (stroke (width 0.1524) (type solid)) (layer "F.CrtYd"))
-    (fp_line (start -0.8001 -0.4064) (end -0.8001 0.4064)
-      (stroke (width 0.0254) (type solid)) (layer "F.Fab"))
-    (fp_line (start -0.8001 0.4064) (end 0.8001 0.4064)
-      (stroke (width 0.0254) (type solid)) (layer "F.Fab"))
-    (fp_line (start 0.8001 -0.4064) (end -0.8001 -0.4064)
-      (stroke (width 0.0254) (type solid)) (layer "F.Fab"))
-    (fp_line (start 0.8001 0.4064) (end 0.8001 -0.4064)
-      (stroke (width 0.0254) (type solid)) (layer "F.Fab"))
-    (fp_circle (center 0 -1.905) (end 0.381 -1.905)
-      (stroke (width 0.508) (type solid)) (fill none) (layer "F.Fab"))
-    (pad "1" smd rect (at 0 0) (size 1.6002 0.8128) (layers "F.Cu" "F.Paste" "F.Mask")
-      (net 18 "+BATT") (pinfunction "1") (pintype "passive"))
-  )
   (footprint "Resistor_SMD:R_0603_1608Metric" (layer "F.Cu")
     (at 135.925 110.725 90)
@@
   )
   (footprint "Mechatronics TestP:CONN1_RCU-0C_TEC" (layer "F.Cu")
-    (at 104.902 131.826)
+    (at 121.4711 148.0603)
     (tags "RCU-0C ")
     (property "Sheetfile" "Probe.kicad_sch")
@@
     )
   )
-  (footprint "Mechatronics TestP:CONN1_RCU-0C_TEC" (layer "F.Cu")
-    (at 123.444 30.988)
-    (tags "RCU-0C ")
-    (property "Sheetfile" "CurrentSense2_sch.kicad_sch")
-    (property "Sheetname" "Current Sense Rails")
-    (property "ki_description" "test point (alternative probe-style design)")
-    (property "ki_keywords" "test point tp")
-    (attr smd)
-    (fp_text reference "TP11" (at 0 2.07832 unlocked) (layer "F.SilkS")
-        (effects (font (size 1 1) (thickness 0.15)))
-    )
-    (fp_text value "VSHUNT2-" (at 0 0 unlocked) (layer "F.Fab")
-        (effects (font (size 1 1) (thickness 0.15)))
-    )
-    (fp_text user "VSHUNT2-" (at 0 -1.09668 unlocked) (layer "F.SilkS")
-        (effects (font (size 0.5 0.5) (thickness 0.125)))
-    )
-    (fp_text user "${REFERENCE}" (at 0 0 unlocked) (layer "F.Fab")
-        (effects (font (size 1 1) (thickness 0.15)))
-    )
-    (fp_circle (center -2.7051 0) (end -2.3241 0)
-      (stroke (width 0.508) (type solid)) (fill none) (layer "B.SilkS"))
-    (fp_circle (center -2.7051 0) (end -2.3241 0)
-      (stroke (width 0.508) (type solid)) (fill none) (layer "F.SilkS"))
-    (fp_line (start -1.0541 -0.6604) (end -1.0541 0.6604)
-      (stroke (width 0.1524) (type solid)) (layer "F.CrtYd"))
-    (fp_line (start -1.0541 0.6604) (end 1.0541 0.6604)
-      (stroke (width 0.1524) (type solid)) (layer "F.CrtYd"))
-    (fp_line (start 1.0541 -0.6604) (end -1.0541 -0.6604)
-      (stroke (width 0.1524) (type solid)) (layer "F.CrtYd"))
-    (fp_line (start 1.0541 0.6604) (end 1.0541 -0.6604)
-      (stroke (width 0.1524) (type solid)) (layer "F.CrtYd"))
-    (fp_line (start -0.8001 -0.4064) (end -0.8001 0.4064)
-      (stroke (width 0.0254) (type solid)) (layer "F.Fab"))
-    (fp_line (start -0.8001 0.4064) (end 0.8001 0.4064)
-      (stroke (width 0.0254) (type solid)) (layer "F.Fab"))
-    (fp_line (start 0.8001 -0.4064) (end -0.8001 -0.4064)
-      (stroke (width 0.0254) (type solid)) (layer "F.Fab"))
-    (fp_line (start 0.8001 0.4064) (end 0.8001 -0.4064)
-      (stroke (width 0.0254) (type solid)) (layer "F.Fab"))
-    (fp_circle (center 0 -1.905) (end 0.381 -1.905)
-      (stroke (width 0.508) (type solid)) (fill none) (layer "F.Fab"))
-    (pad "1" smd rect (at 0 0) (size 1.6002 0.8128) (layers "F.Cu" "F.Paste" "F.Mask")
-      (net 18 "+BATT") (pinfunction "1") (pintype "passive"))
-  )
   (footprint "MountingHole:MountingHole_3.2mm_M3_Pad_Via" locked (layer "F.Cu")
     (at 37.4 37.7)
@@
   )
   (footprint "Mechatronics TestP:CONN1_RCU-0C_TEC" (layer "F.Cu")
-    (at 152.2 131.4)
+    (at 155.418 149.502)
     (tags "RCU-0C ")
     (property "Sheetfile" "Probe.kicad_sch")
@@
   )
   (footprint "Mechatronics TestP:CONN1_RCU-0C_TEC" (layer "F.Cu")
-    (at 120.2 131.65)
+    (at 137.324 148.86)
     (tags "RCU-0C ")
     (property "Sheetfile" "Probe.kicad_sch")
@@
   )
   (footprint "Mechatronics TestP:CONN1_RCU-0C_TEC" (layer "F.Cu")
-    (at 111.4 132.65)
+    (at 128.524 149.86)
     (tags "RCU-0C ")
     (property "Sheetfile" "Probe.kicad_sch")
@@
   (segment (start 159.125999 60.96) (end 161.422 60.96) (width 0.25) (layer "F.Cu") (net 18))
   (segment (start 155.58 60.96) (end 155.58 61.609998) (width 0.25) (layer "F.Cu") (net 18))
-  (segment (start 147.549179 39.394821) (end 147.574 39.37) (width 4) (layer "F.Cu") (net 18))
   (segment (start 147.549179 49.4) (end 147.549179 39.394821) (width 4) (layer "F.Cu") (net 18))
   (via (at 77.4 83.2) (size 1) (drill 0.6) (layers "F.Cu" "B.Cu") (remove_unused_layers) (keep_end_layers) (free) (zone_layer_connections) (net 18))

Commit message: updates
Parts:
- added TP11: VSHUNT2-, Mechatronics TestP:CONN1_RCU-0C_TEC, F.Cu at (102.6, 149.6)
- added TP12: VSHUNT2+, Mechatronics TestP:CONN1_RCU-0C_TEC, F.Cu at (102.6, 153.9)
- added TP16: 19V, Mechatronics TestP:CONN1_RCU-0C_TEC, F.Cu at (102.6, 143.4)
- moved L2 341.2 mm to (486.0, 60.5)
- moved C2_5VB1 292.8 mm to (446.9, 48.5)
- moved F_5VB1 292.8 mm to (424.4, 48.1)
- moved C1_5VB1 292.8 mm to (457.8, 48.5)
- moved CF_5VB1 292.8 mm to (444.8, 61.1)
- moved D_5VB1 292.8 mm to (456.1, 73.4)
- moved R1_5VB1 292.8 mm to (441.8, 61.1)
- moved R2_5VB1 292.8 mm to (441.8, 62.7)
- moved R3_5VB1 292.8 mm to (465.3, 35.1)
- moved R4_5VB1 292.8 mm to (465.3, 32.6)
- moved U14 292.8 mm to (443.6, 65.8)
- moved CF_12VB1 197.8 mm to (333.9, 204.5)
- moved R1_12VB1 197.8 mm to (333.2, 202.2)
- moved R2_12VB1 197.8 mm to (333.9, 206.0)
- moved U16 197.8 mm to (327.7, 210.6)
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Routing:
- net (no net): track 661.8 -> 607.1 mm
- net Net-(C2_12VB1-Pad1): track 24.5 -> 0.00 mm
- net +3.3V: track 15.3 -> 0.00 mm
- net LOGIC 5V: track 96.9 -> 86.9 mm
- net /Microcontroller/PC4: track 7.61 -> 0.00 mm
- net +12V: track 7.59 -> 0.00 mm
- net Net-(D_12VB1-K): track 7.40 -> 0.00 mm
- net /Microcontroller/PC5: track 5.25 -> 0.00 mm
- net +5V: track 3.89 -> 0.00 mm
- net SCL: track 3.47 -> 0.00 mm
- net Net-(U14-FB): track 3.02 -> 0.00 mm
- net Net-(U16-FB): track 2.80 -> 0.00 mm
- net SDA: track 2.05 -> 0.00 mm
- net Net-(J16-Pin_2): track 1.93 -> 0.00 mm
- net Net-(J16-Pin_1): track 1.93 -> 0.00 mm
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
Commit message: saving
Parts:
- moved R2 285.2 mm to (192.2, 373.4)
- moved R3 285.2 mm to (187.7, 373.4)
- moved R4 285.2 mm to (189.2, 373.4)
- moved R1 285.2 mm to (190.7, 373.4)
- moved R4_VSENSE1 226.5 mm to (-93.2, 137.2)
- moved CF1_VSENSE1 226.5 mm to (-97.4, 140.4)
- moved CF2_VSENSE1 226.5 mm to (-93.2, 140.4)
- moved R1_VSENSE1 226.5 mm to (-97.8, 134.8)
- moved R2_VSENSE1 226.5 mm to (-97.9, 137.1)
- moved R3_VSENSE1 226.5 mm to (-93.2, 134.8)
- moved F_5LOGIC1 154.4 mm to (269.2, 154.2)
- moved C5 144.9 mm to (202.0, 360.1)
- moved U10 144.9 mm to (213.1, 368.8)
- moved Y1 144.9 mm to (202.1, 371.9)
- moved C2 144.9 mm to (206.2, 371.3)
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Routing:
- net /Load Sharing/E2: track 1.47 -> 73.5 mm
- net /Load Sharing/E1: track 1.47 -> 57.1 mm
- net Net-(J16-Pin_1): track 0.00 -> 14.2 mm
- net Net-(J16-Pin_2): track 0.00 -> 12.8 mm
- net Net-(J16-Pin_3): track 0.00 -> 10.9 mm
- net PD4: track 0.00 -> 10.2 mm
- net VOLT1: track 6.08 -> 0.00 mm
- net VOLT2: track 5.88 -> 0.00 mm
- net /DPIN5: track 77.7 -> 79.1 mm
- net LOGIC 5V: track 86.9 -> 87.7 mm
Other:
- board text added: "locked"
- board text removed: "MCU RESET"
- board text removed: "PROG"
- board text removed: "Q2"

Commit message: traces for load sharing done
Parts:
- SW1, SW2: footprint Button_Switch_SMD:SW_SPST_PTS645 -> Button_Switch_SMD:SW_SPST_TL3305A
- moved CF1_VSENSE1 795.4 mm to (672.6, 340.0)
- moved CF2_VSENSE1 795.4 mm to (676.8, 340.0)
- moved R2_VSENSE1 795.4 mm to (672.1, 336.7)
- moved R3_VSENSE1 795.4 mm to (676.8, 334.4)
- moved REN1_VSENSE1 795.4 mm to (674.7, 344.7)
- moved REN2_VSENSE1 795.4 mm to (674.7, 348.0)
- moved C1_3LOGIC1 795.4 mm to (608.3, 248.2)
- moved C1_5LOGIC1 795.4 mm to (612.4, 250.8)
- moved C1_5PREC1 795.4 mm to (604.3, 248.2)
- moved C2_3LOGIC1 795.4 mm to (608.3, 250.8)
- moved C2_5LOGIC1 795.4 mm to (612.4, 248.2)
- moved C2_5PREC1 795.4 mm to (604.3, 250.8)
- moved C3_5LOGIC1 795.4 mm to (608.3, 253.3)
- moved C3_5PREC1 795.4 mm to (604.3, 253.3)
- moved C4_5LOGIC1 795.4 mm to (608.3, 255.8)
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Routing:
- net BATTVIN2: track 49.1 -> 204.0 mm, vias 1 -> 2
- net CURRENT1: track 3.62 -> 144.3 mm, vias 0 -> 1
- net BATTVIN1: track 44.0 -> 184.7 mm, vias 1 -> 2
- net /Load Sharing/E1: track 57.1 -> 134.0 mm
- net GND: track 55.2 -> 130.4 mm, vias 40 -> 41
- net /DPIN5: track 79.1 -> 144.7 mm
- net LOGIC 5V: track 87.7 -> 153.1 mm
- net /Load Sharing/E2: track 73.5 -> 137.9 mm
- net Net-(J16-Pin_3): track 10.9 -> 38.7 mm, vias 0 -> 1
- net Net-(J16-Pin_1): track 14.2 -> 40.9 mm, vias 0 -> 1
- net Net-(J16-Pin_2): track 12.8 -> 38.9 mm, vias 0 -> 1
- net PD4: track 10.2 -> 31.0 mm
- net /Load Sharing/G2: track 45.3 -> 44.4 mm

Commit message: Update PCB
Parts:
- removed TP1: VSHUNT-, Mechatronics TestP:CONN1_RCU-0C_TEC
- removed TP10: LOGIC 5V, Mechatronics TestP:CONN1_RCU-0C_TEC
- removed TP11: VSHUNT2-, Mechatronics TestP:CONN1_RCU-0C_TEC
- removed TP12: VSHUNT2+, Mechatronics TestP:CONN1_RCU-0C_TEC
- removed TP13: 3.3V, Mechatronics TestP:CONN1_RCU-0C_TEC
- removed TP14: 5V, Mechatronics TestP:CONN1_RCU-0C_TEC
- removed TP15: 12V, Mechatronics TestP:CONN1_RCU-0C_TEC
- removed TP16: 19V, Mechatronics TestP:CONN1_RCU-0C_TEC
- removed TP17: GND, Mechatronics TestP:CONN1_RCU-0C_TEC
- removed TP3: SDA, Mechatronics TestP:CONN1_RCU-0C_TEC
- removed TP4: SCL, Mechatronics TestP:CONN1_RCU-0C_TEC
- removed TP6: CURRENT2, Mechatronics TestP:CONN1_RCU-0C_TEC
- removed TP7: VOLT1, Mechatronics TestP:CONN1_RCU-0C_TEC
- removed TP8: VOLT2, Mechatronics TestP:CONN1_RCU-0C_TEC
- removed TP9: AREF, Mechatronics TestP:CONN1_RCU-0C_TEC
- U11, U21: moved to B.Cu
- moved D1 616.1 mm to (111.5, 49.8)
- moved D6 614.5 mm to (111.5, 53.0), turned to 180 degrees
- moved D2 606.5 mm to (99.6, 120.6)
- moved D5 603.7 mm to (100.3, 122.7)
- moved U9 548.2 mm to (117.2, 50.8)
- moved U22 541.0 mm to (101.2, 117.2)
- moved U21 6.25 mm to (89.0, 46.4), turned to 90 degrees
Routing:
- net /Voltage Regulator Rails/LOGIC 5V OUT: track 0.00 -> 18.5 mm
- net PD4: track 31.0 -> 47.3 mm
- net Net-(D2-K): track 0.00 -> 15.9 mm
- net Net-(J16-Pin_3): track 38.7 -> 30.3 mm
- net BATTVIN2: track 204.0 -> 211.4 mm
- net Net-(J16-Pin_1): track 40.9 -> 33.9 mm
- net Net-(J16-Pin_2): track 38.9 -> 32.1 mm
- net LOGIC 5V: track 153.1 -> 158.7 mm
- net BATTVIN1: track 184.7 -> 189.8 mm
- net /DPIN5: track 144.7 -> 149.3 mm
- net CURRENT1: track 144.3 -> 140.8 mm
- net GND: track 130.4 -> 132.4 mm, vias 41 -> 43
Other:
- board text removed: "!~WARNING~! HIGH CURRENT HIGH TEMPERATURES"
- board text removed: "FALL 2023"
- board text removed: "KENNETH ISHIO PETER KOTTIS KELVIN LIN"
- board text removed: "SENIOR DESIGN TEAM 9 ROBOT POWER SYSTEMS"
- board text removed: "YECHAO CHEN BRENDAN DENNISH"
