File: KiCad/RPS01-Revision 2/rps01.kicad_pcb (KiCad board)
At the start: 2 copper layers, 150 x 100 mm, 188 parts, among them J1 Header Pins, J1 XT90 Battery VOUT 1, J10 IIC Connector, J11 ISCP, J12 Serial, J13 JST_PH_TEMP_SENSOR_1, J14 JST_PH_TEMP_SENSOR_2, J16 RGB LED, J2 BATT IN 1 XT90, J2 Power In, J3 Power Out, J3 XT90 Battery VOUT 2, J4 XT30PW Batt VOUT, J5 BATT IN 2 XT90, J6 XT30 3.3V, J7 XT30 5V, J8 XT30 12V, J9 XT30PW 19V, Q1 BSC009NE2LS5IATMA1 A (TG2)(1A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, Q1 BSS138, Q2 BSC009NE2LS5IATMA1 B (BG2)(1B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, Q2 BSS138, Q3 BSC009NE2LS5IATMA1 C (BG1)(2A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, Q4 BSC009NE2LS5IATMA1 D (TG1)(2B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, SW1 RST, SW2 Display Button, U1 LTC3780EUH-TRPBF, U1 NP100P04PLG-E1-AY, U10 ATmega328P-A, U11 LM340MPX-5.0/NOPB, U12 3.3V NCV1117ST33T3G, U13 UA741CDT, U14 LM2596S-5V, U15 UA741CDT, U16 LM2596S-12V, U17 DS18B20+, U18 DS18B20+, U19 INA139QPWRQ1, U2 NP100P04PLG-E1-AY, U21 LM340MPX-5.0/NOPB, U22 ADR02AUJZ-REEL7, U3 NP100P04PLG-E1-AY, U4 LTC4416EMS-1-TRPBF, U5 NP100P04PLG-E1-AY, U6 NP100P04PLG-E1-AY, U7 NP100P04PLG-E1-AY, U8 INA139QPWRQ1, U9 ADR02AUJZ-REEL7, Y1 16M

Commit message: Update
Parts:
- moved R4 12.8 mm to (109.4, 129.9)
- moved R1 12.8 mm to (109.5, 128.4)
- moved R2 12.8 mm to (109.5, 126.9)
- moved R3 12.8 mm to (109.4, 131.4)
- moved U22 1.32 mm to (100.0, 117.8)
Routing:
- net /Load Sharing/E1: track 133.6 -> 111.4 mm
- net /Load Sharing/E2: track 138.0 -> 129.3 mm
- net PD4: track 47.3 -> 41.2 mm
- net BATTVIN2: track 211.4 -> 205.4 mm
Changed lines of the file:
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@@
   )
   (footprint "Resistor_SMD:R_0603_1608Metric" (layer "F.Cu")
-    (at 113.143 114.651 180)
+    (at 109.475 126.925 180)
     (descr "Resistor SMD 0603 (1608 Metric), square (rectangular) end terminal, IPC_7351 nominal, (Body size source: IPC-SM-782 page 72, https://www.pcb-3d.com/wordpress/wp-content/uploads/ipc-sm-782a_amendment_1_and_2.pdf), generated with kicad-footprint-generator")
     (tags "resistor")
@@
   )
   (footprint "Resistor_SMD:R_0603_1608Metric" (layer "F.Cu")
-    (at 113.093 117.651)
+    (at 109.425 129.925)
     (descr "Resistor SMD 0603 (1608 Metric), square (rectangular) end terminal, IPC_7351 nominal, (Body size source: IPC-SM-782 page 72, https://www.pcb-3d.com/wordpress/wp-content/uploads/ipc-sm-782a_amendment_1_and_2.pdf), generated with kicad-footprint-generator")
     (tags "resistor")
@@
   )
   (footprint "Resistor_SMD:R_0603_1608Metric" (layer "F.Cu")
-    (at 113.118 116.151 180)
+    (at 109.45 128.425 180)
     (descr "Resistor SMD 0603 (1608 Metric), square (rectangular) end terminal, IPC_7351 nominal, (Body size source: IPC-SM-782 page 72, https://www.pcb-3d.com/wordpress/wp-content/uploads/ipc-sm-782a_amendment_1_and_2.pdf), generated with kicad-footprint-generator")
     (tags "resistor")
@@
   )
   (footprint "Mechatronic Footprints:ADR02AUJZ_REEL7_UJ_5_ADI" (layer "F.Cu")
-    (at 101.17635 117.25)
+    (at 99.97365 117.799999)
     (tags "ADR02AUJZ-REEL7 ")
     (property "Sheetfile" "Rails.kicad_sch")
@@
   )
   (footprint "Resistor_SMD:R_0603_1608Metric" (layer "F.Cu")
-    (at 113.093 119.126)
+    (at 109.425 131.4)
     (descr "Resistor SMD 0603 (1608 Metric), square (rectangular) end terminal, IPC_7351 nominal, (Body size source: IPC-SM-782 page 72, https://www.pcb-3d.com/wordpress/wp-content/uploads/ipc-sm-782a_amendment_1_and_2.pdf), generated with kicad-footprint-generator")
     (tags "resistor")
@@
   (segment locked (start 39.199559 84.02706) (end 40.165558 84.993059) (width 0.25) (layer "F.Cu") (net 28))
   (segment locked (start 37.275098 88.597141) (end 37.275098 88.825098) (width 0.25) (layer "F.Cu") (net 28))
-  (segment (start 96 130.5) (end 100.25 126.25) (width 0.25) (layer "F.Cu") (net 28))
   (segment locked (start 37.275098 88.825098) (end 38.95 90.5) (width 0.25) (layer "F.Cu") (net 28))
   (segment locked (start 39.100517 87.701181) (end 38.171058 87.701181) (width 0.25) (layer "F.Cu") (net 28))
@@
   (via locked (at 67.725098 83.3016) (size 0.8) (drill 0.4) (layers "F.Cu" "B.Cu") (remove_unused_layers) (keep_end_layers) (zone_layer_connections) (net 39))
   (via locked (at 41.550098 77.7516) (size 0.8) (drill 0.4) (layers "F.Cu" "B.Cu") (remove_unused_layers) (keep_end_layers) (zone_layer_connections) (net 39))
-  (segment (start 95.1 130.05) (end 99.4 125.75) (width 0.25) (layer "F.Cu") (net 43))
   (segment locked (start 85.148326 125.923054) (end 89.473054 125.923054) (width 0.25) (layer "F.Cu") (net 43))
   (segment locked (start 93.6 130.05) (end 95.1 130.05) (width 0.25) (layer "F.Cu") (net 43))
@@
   (segment locked (start 63.51375 128.86375) (end 64.199501 129.549501) (width 0.25) (layer "F.Cu") (net 52))
   (via locked (at 63.513749 126.243938) (size 0.8) (drill 0.4) (layers "F.Cu" "B.Cu") (net 52))
-  (segment (start 97.835191 129.300499) (end 99.143501 129.300499) (width 0.25) (layer "F.Cu") (net 59))
   (segment locked (start 46.426624 133.248004) (end 79.116306 133.248004) (width 0.25) (layer "F.Cu") (net 59))
   (segment locked (start 93.173238 130.949501) (end 96.186189 130.949501) (width 0.25) (layer "F.Cu") (net 59))
@@
   (segment locked (start 35.599501 116.049501) (end 40.3 120.75) (width 0.25) (layer "F.Cu") (net 59))
   (segment locked (start 85.519499 126.824501) (end 86.511189 126.824501) (width 0.25) (layer "F.Cu") (net 59))
-  (segment (start 99.143501 129.300499) (end 112.293 116.151) (width 0.25) (layer "F.Cu") (net 59))
   (segment locked (start 83.798004 128.545996) (end 85.519499 126.824501) (width 0.25) (layer "F.Cu") (net 59))
   (segment locked (start 86.513135 126.822555) (end 89.046292 126.822555) (width 0.25) (layer "F.Cu") (net 59))
@@
   (segment locked (start 36.322 84.074) (end 35.599501 84.796499) (width 0.25) (layer "F.Cu") (net 59))
   (segment locked (start 37.592 84.074) (end 36.322 84.074) (width 0.25) (layer "F.Cu") (net 59))
-  (segment locked (start 96.186189 130.949501) (end 97.835191 129.300499) (width 0.25) (layer "F.Cu") (net 59))
   (segment locked (start 89.046292 126.822555) (end 93.173238 130.949501) (width 0.25) (layer "F.Cu") (net 59))
   (segment locked (start 40.3 120.75) (end 40.3 127.12138) (width 0.25) (layer "F.Cu") (net 59))
@@
   (segment locked (start 38.1 83.312) (end 36.068 83.312) (width 0.25) (layer "F.Cu") (net 60))
   (segment locked (start 92.987049 131.399002) (end 99.994998 131.399002) (width 0.25) (layer "F.Cu") (net 60))
-  (segment (start 99.994998 131.399002) (end 112.268 119.126) (width 0.25) (layer "F.Cu") (net 60))
-  (segment (start 112.268 117.651) (end 112.268 119.126) (width 0.25) (layer "F.Cu") (net 60))
+  (segment (start 108.6 129.925) (end 108.6 131.4) (width 0.25) (layer "F.Cu") (net 60))
   (segment locked (start 39.199559 84.88998) (end 38.354 84.044421) (width 0.25) (layer "F.Cu") (net 60))
   (segment locked (start 39.199559 85.80673) (end 39.199559 84.88998) (width 0.25) (layer "F.Cu") (net 60))
   (segment locked (start 46.240435 133.697505) (end 79.302495 133.697505) (width 0.25) (layer "F.Cu") (net 60))
+  (segment (start 99.994998 131.399002) (end 108.599002 131.399002) (width 0.25) (layer "F.Cu") (net 60))
   (segment locked (start 85.831998 127.274002) (end 86.697378 127.274002) (width 0.25) (layer "F.Cu") (net 60))
   (segment locked (start 37.682327 121.62668) (end 38.224179 122.168532) (width 0.25) (layer "F.Cu") (net 60))
+  (segment (start 108.599002 131.399002) (end 108.6 131.4) (width 0.25) (layer "F.Cu") (net 60))
   (segment locked (start 36.068 83.312) (end 35.15 84.23) (width 0.25) (layer "F.Cu") (net 60))
   (segment locked (start 88.860103 127.272056) (end 92.987049 131.399002) (width 0.25) (layer "F.Cu") (net 60))
