File: KiCad/RPS01-Revision 2/Inputs.kicad_sch (KiCad schematic)
At the start: 4 parts

Commit message: Button Footprints
Changed button footprints
Parts:
- SW? (x2): footprint Button_Switch_SMD:SW_SPST_PTS645 -> Button_Switch_SMD:SW_SPST_TL3305A
Changed lines of the file:
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@@
       (effects (font (size 1.27 1.27)))
     )
-    (property "Footprint" "Button_Switch_SMD:SW_SPST_PTS645" (at 70.104 71.628 0)
+    (property "Footprint" "Button_Switch_SMD:SW_SPST_TL3305A" (at 70.104 71.628 0)
       (effects (font (size 1.27 1.27)) hide)
     )
@@
       (effects (font (size 1.27 1.27)))
     )
-    (property "Footprint" "Button_Switch_SMD:SW_SPST_PTS645" (at 69.85 49.276 0)
+    (property "Footprint" "Button_Switch_SMD:SW_SPST_TL3305A" (at 69.85 49.276 0)
       (effects (font (size 1.27 1.27)) hide)
     )

Commit message: updates
Parts:
- SW? (x2): footprint Button_Switch_SMD:SW_SPST_TL3305A -> Button_Switch_SMD:SW_SPST_PTS645
Changed lines of the file:
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@@
   )
   (symbol (lib_id "Switch:SW_Push_Open") (at 70.104 66.548 180) (unit 1)
-    (in_bom yes) (on_board yes) (dnp no) (fields_autoplaced)
+    (in_bom yes) (on_board yes) (dnp no)
     (property "Reference" "SW?" (at 70.104 62.23 0)
       (effects (font (size 1.27 1.27)))
@@
       (effects (font (size 1.27 1.27)))
     )
-    (property "Footprint" "Button_Switch_SMD:SW_SPST_TL3305A" (at 70.104 71.628 0)
-      (effects (font (size 1.27 1.27)) hide)
+    (property "Footprint" "Button_Switch_SMD:SW_SPST_PTS645" (at 79.756 59.944 0)
+      (effects (font (size 1.27 1.27)))
     )
     (property "Datasheet" "~" (at 70.104 71.628 0)
@@
   )
   (symbol (lib_id "Switch:SW_Push_Open") (at 69.85 44.196 180) (unit 1)
-    (in_bom yes) (on_board yes) (dnp no) (fields_autoplaced)
+    (in_bom yes) (on_board yes) (dnp no)
     (property "Reference" "SW?" (at 69.85 39.37 0)
       (effects (font (size 1.27 1.27)))
@@
       (effects (font (size 1.27 1.27)))
     )
-    (property "Footprint" "Button_Switch_SMD:SW_SPST_TL3305A" (at 69.85 49.276 0)
-      (effects (font (size 1.27 1.27)) hide)
+    (property "Footprint" "Button_Switch_SMD:SW_SPST_PTS645" (at 69.088 35.052 0)
+      (effects (font (size 1.27 1.27)))
     )
     (property "Datasheet" "~" (at 69.85 49.276 0)

Commit message: Update Inputs.kicad_sch
Parts:
- SW? (x2): footprint Button_Switch_SMD:SW_SPST_PTS645 -> Button_Switch_SMD:SW_SPST_TL3305A
Changed lines of the file:
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@@
       (effects (font (size 1.27 1.27)))
     )
-    (property "Footprint" "Button_Switch_SMD:SW_SPST_PTS645" (at 79.756 59.944 0)
+    (property "Footprint" "Button_Switch_SMD:SW_SPST_TL3305A" (at 79.756 59.944 0)
       (effects (font (size 1.27 1.27)))
     )
@@
       (effects (font (size 1.27 1.27)))
     )
-    (property "Footprint" "Button_Switch_SMD:SW_SPST_PTS645" (at 69.088 35.052 0)
+    (property "Footprint" "Button_Switch_SMD:SW_SPST_TL3305A" (at 69.088 35.052 0)
       (effects (font (size 1.27 1.27)))
     )

Commit message: Push before Jason changes 3.3V
Parts:
- R? (x2): value 10K -> 4.7K
Changed lines of the file:
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@@
       (effects (font (size 1.27 1.27)))
     )
-    (property "Value" "10K" (at 67.564 71.628 90)
+    (property "Value" "4.7K" (at 67.564 71.628 90)
       (effects (font (size 1 1)))
     )
@@
       (effects (font (size 1.27 1.27)))
     )
-    (property "Value" "10K" (at 67.31 49.276 90)
+    (property "Value" "4.7K" (at 67.31 49.276 90)
       (effects (font (size 1 1)))
     )
