File: KiCad/RPS01-Revision 2/Rails.kicad_sch (KiCad schematic)
At the start: 45 parts, among them U11 LM340MPX-5.0/NOPB, U21 LM340MPX-5.0/NOPB

Commit message: Voltage rail update
Parts:
- C_FF?: value 10.25n -> 10.25n OR DNI
- D1, D2: value D_Zener -> MM3Z5V1ST1G; footprint (none) -> Diode_SMD:D_SOD-323
- D5, D6: value D_Schottky -> B0540W-7-F; footprint (none) -> Diode_SMD:D_SOD-123
- D? (x2): footprint Mechatronic Footprints:CR_SMA_320-340AE_DIO -> Mechatronic Footprints:SSB43L-E352T_DIODE_DO214AA_MBRS
- L?: value 47u -> 53u; footprint Mechatronics BUCK INDUCTOR:IND_CDRH127&slash_LDNP-470MC_SUM -> Mechatronic Footprints:PE-54039SNL_IND_HCI-68_PUL
- L?: value 47u -> 37u; footprint Mechatronics BUCK INDUCTOR:IND_CDRH127&slash_LDNP-470MC_SUM -> Mechatronic Footprints:PE-53932SNLT_IND_HCI-44_PUL
- U11, U21: footprint MP04A_TEX -> Package_TO_SOT_SMD:SOT-223-3_TabPin2
- U?: value 3.3V AMS1117 -> 3.3V NCV1117ST33T3G; footprint SOT223-3_ONS -> Package_TO_SOT_SMD:SOT-223-3_TabPin2
- U? (x2): footprint Mechatronics VREF:UJ_5_ADI -> Mechatronic Footprints:ADR02AUJZ_REEL7_UJ_5_ADI
- renumbered F5 to F_12VB, F1 to F_3LOGIC, F2 to F_5LOGIC, F4 to F_5VB, R1_12VB_DIV1 to R3_12VB, R1_5VB_DIV1 to R3_5VB, R2_12VB_DIV1 to R4_12VB, R2_5VB_DIV1 to R4_5VB
Connections:
- net LOGIC 5V OUT: now also C_FF?.2, C_FF?.2, F_5LOGIC.1, U11.3 (OUT), U21.3 (OUT)
Other:
- note added: "R1_12VB - Feedback Resistor 1 R2_12VB - Feedback Resistor 2 CF_12VB - Feedback Capacitor"
- note added: "R1_5VB - Feedback Resistor 1 R2_5VB - Feedback Resistor 2 CF_5VB - Feedback Capacitor"
- note removed: "R_12VB_FR1 - Feedback Resistor 1 R_12VB_FR2 - Feedback Resistor 2 C_12VB_FC - Feedback Capacitor"
- moved on the sheet: C?, C_FF?, C_IN?, C_OUT?, D1, D2, D5, D6, D?, F_12VB, F_3LOGIC, F_5LOGIC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

Commit message: Button Footprints
Changed button footprints
Parts:
- renumbered F_12VB to F_12VB1, F_3LOGIC to F_3LOGIC1, F_5LOGIC to F_5LOGIC1, F_5VB to F_5VB1, R3_12VB to R3_12VB1, R3_5VB to R3_5VB1, R4_12VB to R4_12VB1, R4_5VB to R4_5VB1
Changed lines of the file:
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@@
   (symbol (lib_id "Device:Fuse_Small") (at 143.51 36.83 180) (unit 1)
     (in_bom yes) (on_board yes) (dnp no)
-    (property "Reference" "F_3LOGIC" (at 142.24 40.64 0)
+    (property "Reference" "F_3LOGIC1" (at 142.24 40.64 0)
       (effects (font (size 1.27 1.27)))
     )
@@
       (project "rps01"
         (path "/14930f15-c0a0-4b55-93e6-b112548415f6/6ed54b0f-f89c-4a82-b1ab-c92c0c126d05"
-          (reference "F_3LOGIC") (unit 1)
+          (reference "F_3LOGIC1") (unit 1)
         )
       )
@@
         )
         (path "/14930f15-c0a0-4b55-93e6-b112548415f6/6ed54b0f-f89c-4a82-b1ab-c92c0c126d05"
-          (reference "C3_5PREC") (unit 1)
+          (reference "C3_5PREC1") (unit 1)
         )
       )
@@
       (project "rps01"
         (path "/14930f15-c0a0-4b55-93e6-b112548415f6/6ed54b0f-f89c-4a82-b1ab-c92c0c126d05"
-          (reference "C3_5LOGIC") (unit 1)
+          (reference "C3_5LOGIC1") (unit 1)
         )
       )
@@
   (symbol (lib_id "Device:R_Small") (at 531.622 117.094 0) (unit 1)
     (in_bom yes) (on_board yes) (dnp no) (fields_autoplaced)
-    (property "Reference" "R3_12VB" (at 533.4 116.459 0)
+    (property "Reference" "R3_12VB1" (at 533.4 116.459 0)
       (effects (font (size 1.27 1.27)) (justify left))
     )
@@
       (project "rps01"
         (path "/14930f15-c0a0-4b55-93e6-b112548415f6/6ed54b0f-f89c-4a82-b1ab-c92c0c126d05"
-          (reference "R3_12VB") (unit 1)
+          (reference "R3_12VB1") (unit 1)
         )
       )
@@
   (symbol (lib_id "Device:Fuse_Small") (at 351.282 110.49 0) (unit 1)
     (in_bom yes) (on_board yes) (dnp no)
-    (property "Reference" "F_5VB" (at 351.282 106.68 0)
+    (property "Reference" "F_5VB1" (at 351.282 106.68 0)
       (effects (font (size 1.27 1.27)))
     )
@@
       (project "rps01"
         (path "/14930f15-c0a0-4b55-93e6-b112548415f6/6ed54b0f-f89c-4a82-b1ab-c92c0c126d05"
-          (reference "F_5VB") (unit 1)
+          (reference "F_5VB1") (unit 1)
         )
       )
@@
       (project "rps01"
         (path "/14930f15-c0a0-4b55-93e6-b112548415f6/6ed54b0f-f89c-4a82-b1ab-c92c0c126d05"
-          (reference "C2_5VB") (unit 1)
+          (reference "C2_5VB1") (unit 1)
         )
       )
@@
   (symbol (lib_id "Device:Fuse_Small") (at 177.6573 124.714 0) (unit 1)
     (in_bom yes) (on_board yes) (dnp no)
-    (property "Reference" "F_5LOGIC" (at 177.6573 120.904 0)
+    (property "Reference" "F_5LOGIC1" (at 177.6573 120.904 0)
       (effects (font (size 1.27 1.27)))
     )
@@
       (project "rps01"
         (path "/14930f15-c0a0-4b55-93e6-b112548415f6/6ed54b0f-f89c-4a82-b1ab-c92c0c126d05"
-          (reference "F_5LOGIC") (unit 1)
+          (reference "F_5LOGIC1") (unit 1)
         )
       )
@@
       (project "rps01"
         (path "/14930f15-c0a0-4b55-93e6-b112548415f6/6ed54b0f-f89c-4a82-b1ab-c92c0c126d05"
-          (reference "C2_12VB") (unit 1)
+          (reference "C2_12VB1") (unit 1)
         )
       )
@@
       (project "rps01"
         (path "/14930f15-c0a0-4b55-93e6-b112548415f6/6ed54b0f-f89c-4a82-b1ab-c92c0c126d05"
-          (reference "C2_3LOGIC") (unit 1)
+          (reference "C2_3LOGIC1") (unit 1)
         )
       )
@@
         )
         (path "/14930f15-c0a0-4b55-93e6-b112548415f6/6ed54b0f-f89c-4a82-b1ab-c92c0c126d05"
-          (reference "C1_5PREC") (unit 1)
+          (reference "C1_5PREC1") (unit 1)
         )
       )
@@
         )
         (path "/14930f15-c0a0-4b55-93e6-b112548415f6/6ed54b0f-f89c-4a82-b1ab-c92c0c126d05"
-          (reference "C2_5PREC") (unit 1)
+          (reference "C2_5PREC1") (unit 1)
         )
       )
@@
       (project "rps01"
         (path "/14930f15-c0a0-4b55-93e6-b112548415f6/6ed54b0f-f89c-4a82-b1ab-c92c0c126d05"
-          (reference "CF_12VB") (unit 1)
+          (reference "CF_12VB1") (unit 1)
         )
       )
@@
   (symbol (lib_id "Device:R_Small") (at 534.162 125.984 90) (unit 1)
     (in_bom yes) (on_board yes) (dnp no)
-    (property "Reference" "R4_12VB" (at 539.75 121.92 90)
+    (property "Reference" "R4_12VB1" (at 539.75 121.92 90)
       (effects (font (size 1.27 1.27)))
     )
@@
       (project "rps01"
         (path "/14930f15-c0a0-4b55-93e6-b112548415f6/6ed54b0f-f89c-4a82-b1ab-c92c0c126d05"
-          (reference "R4_12VB") (unit 1)
+          (reference "R4_12VB1") (unit 1)
         )
       )
@@
         )
         (path "/14930f15-c0a0-4b55-93e6-b112548415f6/6ed54b0f-f89c-4a82-b1ab-c92c0c126d05"
-          (reference "C4_5PREC") (unit 1)
+          (reference "C4_5PREC1") (unit 1)
         )
       )
@@
       (project "rps01"
         (path "/14930f15-c0a0-4b55-93e6-b112548415f6/6ed54b0f-f89c-4a82-b1ab-c92c0c126d05"
-          (reference "C1_3LOGIC") (unit 1)
+          (reference "C1_3LOGIC1") (unit 1)
         )
       )
@@
       (project "rps01"
         (path "/14930f15-c0a0-4b55-93e6-b112548415f6/6ed54b0f-f89c-4a82-b1ab-c92c0c126d05"
-          (reference "D_5VB") (unit 1)
+          (reference "D_5VB1") (unit 1)
         )
       )
@@
       (project "rps01"
         (path "/14930f15-c0a0-4b55-93e6-b112548415f6/6ed54b0f-f89c-4a82-b1ab-c92c0c126d05"
-          (reference "C1_5LOGIC") (unit 1)
+          (reference "C1_5LOGIC1") (unit 1)
         )
       )
@@
   (symbol (lib_id "Device:Fuse_Small") (at 525.272 111.76 0) (unit 1)
     (in_bom yes) (on_board yes) (dnp no)
-    (property "Reference" "F_12VB" (at 525.272 107.95 0)
+    (property "Reference" "F_12VB1" (at 525.272 107.95 0)
       (effects (font (size 1.27 1.27)))
     )
@@
       (project "rps01"
         (path "/14930f15-c0a0-4b55-93e6-b112548415f6/6ed54b0f-f89c-4a82-b1ab-c92c0c126d05"
-          (reference "F_12VB") (unit 1)
+          (reference "F_12VB1") (unit 1)
         )
       )
@@
       (project "rps01"
         (path "/14930f15-c0a0-4b55-93e6-b112548415f6/6ed54b0f-f89c-4a82-b1ab-c92c0c126d05"
-          (reference "CF_5VB") (unit 1)
+          (reference "CF_5VB1") (unit 1)
         )
       )
@@
       (project "rps01"
         (path "/14930f15-c0a0-4b55-93e6-b112548415f6/6ed54b0f-f89c-4a82-b1ab-c92c0c126d05"
-          (reference "D_12VB") (unit 1)
+          (reference "D_12VB1") (unit 1)
         )
       )
@@
       (project "rps01"
         (path "/14930f15-c0a0-4b55-93e6-b112548415f6/6ed54b0f-f89c-4a82-b1ab-c92c0c126d05"
-          (reference "C1_5VB") (unit 1)
+          (reference "C1_5VB1") (unit 1)
         )
       )
@@
       (project "rps01"
         (path "/14930f15-c0a0-4b55-93e6-b112548415f6/6ed54b0f-f89c-4a82-b1ab-c92c0c126d05"
-          (reference "R1_5VB") (unit 1)
+          (reference "R1_5VB1") (unit 1)
         )
       )
@@
       (project "rps01"
         (path "/14930f15-c0a0-4b55-93e6-b112548415f6/6ed54b0f-f89c-4a82-b1ab-c92c0c126d05"
-          (reference "R2_12VB") (unit 1)
+          (reference "R2_12VB1") (unit 1)
         )
       )
@@
       (project "rps01"
         (path "/14930f15-c0a0-4b55-93e6-b112548415f6/6ed54b0f-f89c-4a82-b1ab-c92c0c126d05"
-          (reference "R1_12VB") (unit 1)
+          (reference "R1_12VB1") (unit 1)
         )
       )
@@
       (project "rps01"
         (path "/14930f15-c0a0-4b55-93e6-b112548415f6/6ed54b0f-f89c-4a82-b1ab-c92c0c126d05"
-          (reference "R2_5VB") (unit 1)
+          (reference "R2_5VB1") (unit 1)
         )
       )
@@
       (project "rps01"
         (path "/14930f15-c0a0-4b55-93e6-b112548415f6/6ed54b0f-f89c-4a82-b1ab-c92c0c126d05"
-          (reference "C2_5LOGIC") (unit 1)
+          (reference "C2_5LOGIC1") (unit 1)
         )
       )
@@
   (symbol (lib_id "Device:R_Small") (at 357.632 113.03 0) (unit 1)
     (in_bom yes) (on_board yes) (dnp no) (fields_autoplaced)
-    (property "Reference" "R3_5VB" (at 359.41 112.395 0)
+    (property "Reference" "R3_5VB1" (at 359.41 112.395 0)
       (effects (font (size 1.27 1.27)) (justify left))
     )
@@
       (project "rps01"
         (path "/14930f15-c0a0-4b55-93e6-b112548415f6/6ed54b0f-f89c-4a82-b1ab-c92c0c126d05"
-          (reference "R3_5VB") (unit 1)
+          (reference "R3_5VB1") (unit 1)
         )
       )
@@
       (project "rps01"
         (path "/14930f15-c0a0-4b55-93e6-b112548415f6/6ed54b0f-f89c-4a82-b1ab-c92c0c126d05"
-          (reference "C1_12VB") (unit 1)
+          (reference "C1_12VB1") (unit 1)
         )
       )
@@
   (symbol (lib_id "Device:R_Small") (at 360.172 122.936 90) (unit 1)
     (in_bom yes) (on_board yes) (dnp no)
-    (property "Reference" "R4_5VB" (at 364.998 118.364 90)
+    (property "Reference" "R4_5VB1" (at 364.998 118.364 90)
       (effects (font (size 1.27 1.27)))
     )
@@
       (project "rps01"
         (path "/14930f15-c0a0-4b55-93e6-b112548415f6/6ed54b0f-f89c-4a82-b1ab-c92c0c126d05"
-          (reference "R4_5VB") (unit 1)
+          (reference "R4_5VB1") (unit 1)
         )
       )
@@
       (project "rps01"
         (path "/14930f15-c0a0-4b55-93e6-b112548415f6/6ed54b0f-f89c-4a82-b1ab-c92c0c126d05"
-          (reference "C4_5LOGIC") (unit 1)
-        )
-      )
+          (reference "C4_5LOGIC1") (unit 1)
+        )
+      )

Commit message: Update Rails.kicad_sch
Added DNI to component values
Parts:
- C? (x4), C_FF? (x2): value 0.1u -> 0.1u DNI
- C_FF? (x2): value 0.22u -> 0.22u DNI
- C_FF?: value 22u -> 22u DNI
- C_FF?: value 3.65n -> 3.65n DNI
- C_FF?: value 0.47u -> 0.47u DNI
- C_IN? (x2): value 100u -> 100u DNI
- C_OUT? (x2): value 220u -> 220u DNI
- L?: value 53u -> 53u DNI
- L?: value 37u -> 37u DNI
- R? (x2): value 1k -> 1k DNI
- R?: value 8.87k -> 8.87k DNI
- R?: value 3.16k -> 3.16k DNI
Changed lines of the file:
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@@
       (effects (font (size 1.27 1.27)) (justify left))
     )
-    (property "Value" "0.1u" (at 114.3508 271.2212 0)
+    (property "Value" "0.1u DNI" (at 114.3508 271.2212 0)
       (effects (font (size 1.27 1.27)) (justify left))
     )
@@
       (effects (font (size 1.27 1.27)) (justify right))
     )
-    (property "Value" "0.22u" (at 89.963 104.3448 90)
+    (property "Value" "0.22u DNI" (at 89.963 104.3448 90)
       (effects (font (size 1.27 1.27)) (justify right))
     )
@@
   (symbol (lib_id "Device:C_Polarized") (at 341.63 120.396 0) (unit 1)
     (in_bom yes) (on_board yes) (dnp no) (fields_autoplaced)
-    (property "Reference" "C_OUT?" (at 345.44 118.872 0)
-      (effects (font (size 1.27 1.27)) (justify left))
-    )
-    (property "Value" "220u" (at 345.44 121.412 0)
+    (property "Reference" "C_OUT?" (at 345.44 118.237 0)
+      (effects (font (size 1.27 1.27)) (justify left))
+    )
+    (property "Value" "220u DNI" (at 345.44 120.777 0)
       (effects (font (size 1.27 1.27)) (justify left))
     )
@@
   (symbol (lib_id "Device:C_Polarized") (at 513.08 121.92 0) (unit 1)
     (in_bom yes) (on_board yes) (dnp no) (fields_autoplaced)
-    (property "Reference" "C_OUT?" (at 516.89 120.396 0)
-      (effects (font (size 1.27 1.27)) (justify left))
-    )
-    (property "Value" "220u" (at 516.89 122.936 0)
+    (property "Reference" "C_OUT?" (at 516.89 119.761 0)
+      (effects (font (size 1.27 1.27)) (justify left))
+    )
+    (property "Value" "220u DNI" (at 516.89 122.301 0)
       (effects (font (size 1.27 1.27)) (justify left))
     )
@@
       (effects (font (size 1.27 1.27)))
     )
-    (property "Value" "53u" (at 329.1552 108.8207 90)
+    (property "Value" "53u DNI" (at 329.1552 108.8207 90)
       (effects (font (size 1.27 1.27)))
     )
@@
       (effects (font (size 1.27 1.27)) (justify right))
     )
-    (property "Value" "22u" (at 91.44 35.56 90)
+    (property "Value" "22u DNI" (at 91.44 35.56 90)
       (effects (font (size 1.27 1.27)) (justify right))
     )
@@
       (effects (font (size 1.27 1.27)) (justify left))
     )
-    (property "Value" "0.1u" (at 115.57 224.79 0)
+    (property "Value" "0.1u DNI" (at 115.57 224.79 0)
       (effects (font (size 1.27 1.27)) (justify left))
     )
@@
   (symbol (lib_id "Device:C_Small") (at 130.302 210.058 0) (unit 1)
     (in_bom yes) (on_board yes) (dnp no) (fields_autoplaced)
-    (property "Reference" "C?" (at 133.35 209.4293 0)
-      (effects (font (size 1.27 1.27)) (justify left))
-    )
-    (property "Value" "0.1u" (at 133.35 211.9693 0)
+    (property "Reference" "C?" (at 133.35 208.7943 0)
+      (effects (font (size 1.27 1.27)) (justify left))
+    )
+    (property "Value" "0.1u DNI" (at 133.35 211.3343 0)
       (effects (font (size 1.27 1.27)) (justify left))
     )
@@
       (effects (font (size 1.27 1.27)) (justify right))
     )
-    (property "Value" "3.65n" (at 502.92 76.2 90)
+    (property "Value" "3.65n DNI" (at 502.92 76.2 90)
       (effects (font (size 1.27 1.27)) (justify right))
     )
@@
   (symbol (lib_id "Device:C_Small") (at 130.302 255.778 0) (unit 1)
     (in_bom yes) (on_board yes) (dnp no) (fields_autoplaced)
-    (property "Reference" "C?" (at 133.35 255.1493 0)
-      (effects (font (size 1.27 1.27)) (justify left))
-    )
-    (property "Value" "0.1u" (at 133.35 257.6893 0)
+    (property "Reference" "C?" (at 133.35 254.5143 0)
+      (effects (font (size 1.27 1.27)) (justify left))
+    )
+    (property "Value" "0.1u DNI" (at 133.35 257.0543 0)
       (effects (font (size 1.27 1.27)) (justify left))
     )
@@
       (effects (font (size 1.27 1.27)) (justify right))
     )
-    (property "Value" "0.47u" (at 91.1688 53.3982 90)
+    (property "Value" "0.47u DNI" (at 91.1688 53.3982 90)
       (effects (font (size 1.27 1.27)) (justify right))
     )
@@
       (effects (font (size 1.27 1.27)) (justify right))
     )
-    (property "Value" "0.22u" (at 88.2127 136.3649 90)
+    (property "Value" "0.22u DNI" (at 88.2127 136.3649 90)
       (effects (font (size 1.27 1.27)) (justify right))
     )
@@
   (symbol (lib_id "Device:C_Polarized") (at 266.7 118.11 0) (unit 1)
     (in_bom yes) (on_board yes) (dnp no) (fields_autoplaced)
-    (property "Reference" "C_IN?" (at 270.51 116.586 0)
-      (effects (font (size 1.27 1.27)) (justify left))
-    )
-    (property "Value" "100u" (at 270.51 119.126 0)
+    (property "Reference" "C_IN?" (at 270.51 115.951 0)
+      (effects (font (size 1.27 1.27)) (justify left))
+    )
+    (property "Value" "100u DNI" (at 270.51 118.491 0)
       (effects (font (size 1.27 1.27)) (justify left))
     )
@@
       (effects (font (size 1.27 1.27)) (justify right))
     )
-    (property "Value" "1k" (at 307.34 88.9 90)
+    (property "Value" "1k DNI" (at 307.34 88.9 90)
       (effects (font (size 1.27 1.27)) (justify right))
     )
@@
       (effects (font (size 1.27 1.27)) (justify right))
     )
-    (property "Value" "8.87k\n" (at 500.38 90.17 90)
+    (property "Value" "8.87k DNI\n" (at 500.38 90.17 90)
       (effects (font (size 1.27 1.27)) (justify right))
     )
@@
       (effects (font (size 1.27 1.27)) (justify right))
     )
-    (property "Value" "1k" (at 481.33 90.17 90)
+    (property "Value" "1k DNI" (at 481.33 90.17 90)
       (effects (font (size 1.27 1.27)) (justify right))
     )
@@
       (effects (font (size 1.27 1.27)) (justify right))
     )
-    (property "Value" "3.16k" (at 328.93 88.9 90)
+    (property "Value" "3.16k DNI" (at 328.93 88.9 90)
       (effects (font (size 1.27 1.27)) (justify right))
     )
@@
       (effects (font (size 1.27 1.27)) (justify right))
     )
-    (property "Value" "0.1u" (at 130.5444 135.6786 90)
+    (property "Value" "0.1u DNI" (at 130.5444 135.6786 90)
       (effects (font (size 1.27 1.27)) (justify right))
     )
@@
   (symbol (lib_id "Device:C_Polarized") (at 438.15 119.38 0) (unit 1)
     (in_bom yes) (on_board yes) (dnp no) (fields_autoplaced)
-    (property "Reference" "C_IN?" (at 441.96 117.856 0)
-      (effects (font (size 1.27 1.27)) (justify left))
-    )
-    (property "Value" "100u" (at 441.96 120.396 0)
+    (property "Reference" "C_IN?" (at 441.96 117.221 0)
+      (effects (font (size 1.27 1.27)) (justify left))
+    )
+    (property "Value" "100u DNI" (at 441.96 119.761 0)
       (effects (font (size 1.27 1.27)) (justify left))
     )
@@
   (symbol (lib_id "Device:L") (at 500.38 111.76 90) (unit 1)
     (in_bom yes) (on_board yes) (dnp no) (fields_autoplaced)
-    (property "Reference" "L?" (at 500.38 107.95 90)
-      (effects (font (size 1.27 1.27)))
-    )
-    (property "Value" "37u" (at 500.38 110.49 90)
+    (property "Reference" "L?" (at 500.38 106.68 90)
+      (effects (font (size 1.27 1.27)))
+    )
+    (property "Value" "37u DNI" (at 500.38 109.22 90)
       (effects (font (size 1.27 1.27)))
     )
@@
       (effects (font (size 1.27 1.27)) (justify right))
     )
-    (property "Value" "0.1u" (at 131.6717 105.1986 90)
-      (effects (font (size 1.27 1.27)) (justify right))
-    )
+    (property "Value" "0.1u DNI" (at 131.6717 105.1986 90)
+      (effects (font (size 1.27 1.27)) (justify right))
+    )
