File: KiCad/RPS01-Revision 2/Display.kicad_sch (KiCad schematic)
At the start: 5 parts

Commit message: Locking and clean. Prepare for Rework
Parts:
- removed J?: Display, SSD1306:128x64OLED, symbol Connector:Conn_01x04_Pin
Changed lines of the file:
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@@
-    (stroke (width 0) (type default))
-  )
-  (wire (pts (xy 194.818 57.15) (xy 197.104 57.15))
     (stroke (width 0) (type default))
   )
@@
     (stroke (width 0) (type default))
   )
-  (wire (pts (xy 194.818 59.69) (xy 197.104 59.69))
-    (stroke (width 0) (type default))
-  )
   (wire (pts (xy 146.812 47.6504) (xy 146.9136 47.6504))
     (stroke (width 0) (type default))
   )
   (wire (pts (xy 142.2908 63.9064) (xy 144.8308 63.9064))
-    (stroke (width 0) (type default))
-  )
-  (wire (pts (xy 197.104 62.23) (xy 194.818 62.23))
-    (stroke (width 0) (type default))
-  )
-  (wire (pts (xy 194.818 62.23) (xy 194.818 64.516))
     (stroke (width 0) (type default))
   )
@@
     (stroke (width 0) (type default))
   )
-  (wire (pts (xy 194.818 54.61) (xy 197.104 54.61))
-    (stroke (width 0) (type default))
-  )
   (wire (pts (xy 126.3904 58.8264) (xy 126.3904 61.9252))
     (stroke (width 0) (type default))
   )
-  (global_label "LOGIC 5V" (shape bidirectional) (at 194.818 59.69 180) (fields_autoplaced)
-    (effects (font (size 1.27 1.27)) (justify right))
-    (property "Intersheetrefs" "${INTERSHEET_REFS}" (at 182.0318 59.69 0)
-      (effects (font (size 1.27 1.27)) (justify right) hide)
-    )
-  )
   (hierarchical_label "VIN BLUE" (shape bidirectional) (at 126.492 38.608 90) (fields_autoplaced)
     (effects (font (size 1.27 1.27)) (justify left))
-  )
-  (hierarchical_label "SCL" (shape bidirectional) (at 194.818 57.15 180) (fields_autoplaced)
-    (effects (font (size 1.27 1.27)) (justify right))
-  )
-  (hierarchical_label "SDA" (shape bidirectional) (at 194.818 54.61 180) (fields_autoplaced)
-    (effects (font (size 1.27 1.27)) (justify right))
   )
   (hierarchical_label "VIN RED" (shape bidirectional) (at 137.16 38.354 90) (fields_autoplaced)
@@
     (effects (font (size 1.27 1.27)) (justify left))
   )
-  (symbol (lib_id "Connector:Conn_01x04_Pin") (at 202.184 59.69 180) (unit 1)
-    (in_bom yes) (on_board yes) (dnp no) (fields_autoplaced)
-    (property "Reference" "J?" (at 203.2 57.785 0)
-      (effects (font (size 1.27 1.27)) (justify right))
-    )
-    (property "Value" "Display" (at 203.2 60.325 0)
-      (effects (font (size 1.27 1.27)) (justify right))
-    )
-    (property "Footprint" "SSD1306:128x64OLED" (at 202.184 59.69 0)
-      (effects (font (size 1.27 1.27)) hide)
-    )
-    (property "Datasheet" "~" (at 202.184 59.69 0)
-      (effects (font (size 1.27 1.27)) hide)
-    )
-    (pin "1")
-    (pin "2")
-    (pin "3")
-    (pin "4")
-    (instances
-      (project "rps01"
-        (path "/14930f15-c0a0-4b55-93e6-b112548415f6"
-          (reference "J?") (unit 1)
-        )
-        (path "/14930f15-c0a0-4b55-93e6-b112548415f6/a2e49fe6-126d-427d-b045-54fb7f662aa7"
-          (reference "J?") (unit 1)
-        )
-        (path "/14930f15-c0a0-4b55-93e6-b112548415f6/66639be3-b7af-4c3b-a889-0b5ac725a84a"
-          (reference "J15") (unit 1)
-        )
-      )
-    )
-  )
-  (symbol (lib_id "power:GND") (at 194.818 64.516 0) (unit 1)
-    (in_bom yes) (on_board yes) (dnp no) (fields_autoplaced)
-    (property "Reference" "#PWR?" (at 194.818 70.866 0)
-      (effects (font (size 1.27 1.27)) hide)
-    )
-    (property "Value" "GND" (at 194.818 70.104 0)
-      (effects (font (size 1.27 1.27)))
-    )
-    (property "Footprint" "" (at 194.818 64.516 0)
-      (effects (font (size 1.27 1.27)) hide)
-    )
-    (property "Datasheet" "" (at 194.818 64.516 0)
-      (effects (font (size 1.27 1.27)) hide)
-    )
-    (pin "1")
-    (instances
-      (project "rps01"
-        (path "/14930f15-c0a0-4b55-93e6-b112548415f6"
-          (reference "#PWR?") (unit 1)
-        )
-        (path "/14930f15-c0a0-4b55-93e6-b112548415f6/a2e49fe6-126d-427d-b045-54fb7f662aa7"
-          (reference "#PWR?") (unit 1)
-        )
-        (path "/14930f15-c0a0-4b55-93e6-b112548415f6/66639be3-b7af-4c3b-a889-0b5ac725a84a"
-          (reference "#PWR077") (unit 1)
-        )
-      )
-    )
-  )
   (symbol (lib_id "Device:R") (at 126.3904 55.0164 180) (unit 1)

Commit message: update led resistor and voltsense references
Changed lines of the file:
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@@
         )
         (path "/14930f15-c0a0-4b55-93e6-b112548415f6/66639be3-b7af-4c3b-a889-0b5ac725a84a"
-          (reference "R30") (unit 1)
+          (reference "RBLUE") (unit 1)
         )
       )
@@
         )
         (path "/14930f15-c0a0-4b55-93e6-b112548415f6/66639be3-b7af-4c3b-a889-0b5ac725a84a"
-          (reference "R29") (unit 1)
+          (reference "RRED") (unit 1)
         )
       )
@@
   (symbol (lib_id "Device:R") (at 146.9136 53.6956 180) (unit 1)
     (in_bom yes) (on_board yes) (dnp no)
-    (property "Reference" "R?" (at 153.1112 53.594 90)
+    (property "Reference" "R?" (at 149.86 53.34 90)
       (effects (font (size 1.27 1.27)))
     )
@@
         )
         (path "/14930f15-c0a0-4b55-93e6-b112548415f6/66639be3-b7af-4c3b-a889-0b5ac725a84a"
-          (reference "R28") (unit 1)
+          (reference "RGREEN") (unit 1)
         )
       )
