File: KiCad/RPS01-Revision 2/Load_Sharing.kicad_sch (KiCad schematic)
At the start: 11 parts, among them U1 NP100P04PLG-E1-AY, U2 NP100P04PLG-E1-AY, U3 NP100P04PLG-E1-AY, U4 LTC4416EMS-1-TRPBF, U5 NP100P04PLG-E1-AY, U6 NP100P04PLG-E1-AY, U7 NP100P04PLG-E1-AY

Commit message: update some references
Connections:
- net VIN1: now also U1.2 (DRAIN), U1.4 (FIN)
- net VIN2: now also U7.2 (DRAIN), U7.4 (FIN)
- net VOUT: now also U1.3 (SOURCE), U2.3 (SOURCE), U3.3 (SOURCE), U5.3 (SOURCE), U6.3 (SOURCE), U7.3 (SOURCE); no longer U1.2 (DRAIN), U1.4 (FIN), U7.2 (DRAIN), U7.4 (FIN)
Changed lines of the file:
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@@
 (kicad_sch (version 20230121) (generator eeschema)
   (paper "A4")
-  (junction (at 165.1 165.1) (diameter 0) (color 0 0 0 0)
+  (junction (at 162.56 104.14) (diameter 0) (color 0 0 0 0)
+  )
+  (junction (at 162.56 93.98) (diameter 0) (color 0 0 0 0)
+  )
+  (junction (at 160.02 144.78) (diameter 0) (color 0 0 0 0)
   )
   (junction (at 111.76 121.92) (diameter 0) (color 0 0 0 0)
@@
   (junction (at 162.56 66.04) (diameter 0) (color 0 0 0 0)
   )
+  (junction (at 162.56 121.92) (diameter 0) (color 0 0 0 0)
+  )
   (junction (at 36.576 109.22) (diameter 0) (color 0 0 0 0)
   )
@@
   (junction (at 96.52 121.92) (diameter 0) (color 0 0 0 0)
   )
-  (junction (at 165.1 104.14) (diameter 0) (color 0 0 0 0)
-  )
   (junction (at 99.06 111.76) (diameter 0) (color 0 0 0 0)
   )
   (junction (at 160.02 132.08) (diameter 0) (color 0 0 0 0)
   )
+  (junction (at 170.18 63.5) (diameter 0) (color 0 0 0 0)
+  )
+  (junction (at 106.68 147.32) (diameter 0) (color 0 0 0 0)
+  )
   (junction (at 111.76 132.08) (diameter 0) (color 0 0 0 0)
   )
@@
   (junction (at 111.76 97.79) (diameter 0) (color 0 0 0 0)
   )
+  (junction (at 99.06 66.04) (diameter 0) (color 0 0 0 0)
+  )
   (junction (at 99.06 104.14) (diameter 0) (color 0 0 0 0)
   )
@@
   )
   (junction (at 36.322 104.14) (diameter 0) (color 0 0 0 0)
-  )
-  (junction (at 170.18 50.8) (diameter 0) (color 0 0 0 0)
   )
   (no_connect (at 50.8 111.76))
@@
     (stroke (width 0) (type default))
   )
-  (wire (pts (xy 176.53 50.8) (xy 176.53 96.52))
-    (stroke (width 0) (type default))
-  )
-  (wire (pts (xy 165.1 96.52) (xy 165.1 104.14))
-    (stroke (width 0) (type default))
-  )
   (wire (pts (xy 106.68 132.08) (xy 111.76 132.08))
     (stroke (width 0) (type default))
@@
     (stroke (width 0) (type default))
   )
-  (wire (pts (xy 170.18 38.1) (xy 170.18 50.8))
-    (stroke (width 0) (type default))
-  )
   (wire (pts (xy 99.06 104.14) (xy 111.76 104.14))
     (stroke (width 0) (type default))
@@
     (stroke (width 0) (type default))
   )
+  (wire (pts (xy 106.68 167.64) (xy 111.76 167.64))
+    (stroke (width 0) (type default))
+  )
   (wire (pts (xy 99.06 144.78) (xy 99.06 165.1))
     (stroke (width 0) (type default))
@@
     (stroke (width 0) (type default))
   )
-  (wire (pts (xy 157.48 165.1) (xy 165.1 165.1))
-    (stroke (width 0) (type default))
-  )
   (wire (pts (xy 157.48 66.04) (xy 162.56 66.04))
     (stroke (width 0) (type default))
@@
     (stroke (width 0) (type default))
   )
-  (wire (pts (xy 104.14 176.53) (xy 165.1 176.53))
+  (wire (pts (xy 162.56 104.14) (xy 162.56 121.92))
+    (stroke (width 0) (type default))
+  )
+  (wire (pts (xy 106.68 147.32) (xy 106.68 167.64))
+    (stroke (width 0) (type default))
+  )
+  (wire (pts (xy 162.56 104.14) (xy 162.56 93.98))
     (stroke (width 0) (type default))
   )
@@
     (stroke (width 0) (type default))
   )
-  (wire (pts (xy 165.1 176.53) (xy 165.1 165.1))
-    (stroke (width 0) (type default))
-  )
   (wire (pts (xy 32.512 104.14) (xy 36.322 104.14))
     (stroke (width 0) (type default))
@@
     (stroke (width 0) (type default))
   )
-  (wire (pts (xy 111.76 167.64) (xy 104.14 167.64))
-    (stroke (width 0) (type default))
-  )
-  (wire (pts (xy 165.1 104.14) (xy 167.64 104.14))
+  (wire (pts (xy 160.02 165.1) (xy 157.48 165.1))
     (stroke (width 0) (type default))
   )
@@
     (stroke (width 0) (type default))
   )
-  (wire (pts (xy 99.06 50.8) (xy 170.18 50.8))
-    (stroke (width 0) (type default))
-  )
   (wire (pts (xy 96.52 63.5) (xy 96.52 38.1))
     (stroke (width 0) (type default))
@@
     (stroke (width 0) (type default))
   )
-  (wire (pts (xy 170.18 50.8) (xy 176.53 50.8))
-    (stroke (width 0) (type default))
-  )
   (wire (pts (xy 160.02 144.78) (xy 160.02 132.08))
     (stroke (width 0) (type default))
   )
+  (wire (pts (xy 99.06 66.04) (xy 99.06 40.64))
+    (stroke (width 0) (type default))
+  )
   (wire (pts (xy 25.908 95.25) (xy 25.908 104.14))
     (stroke (width 0) (type default))
@@
     (stroke (width 0) (type default))
   )
-  (wire (pts (xy 165.1 165.1) (xy 165.1 104.14))
-    (stroke (width 0) (type default))
-  )
   (wire (pts (xy 160.02 76.2) (xy 160.02 83.82))
     (stroke (width 0) (type default))
@@
     (stroke (width 0) (type default))
   )
-  (wire (pts (xy 104.14 167.64) (xy 104.14 176.53))
-    (stroke (width 0) (type default))
-  )
   (wire (pts (xy 160.02 119.38) (xy 160.02 132.08))
     (stroke (width 0) (type default))
@@
     (stroke (width 0) (type default))
   )
-  (wire (pts (xy 118.11 104.14) (xy 165.1 104.14))
+  (wire (pts (xy 162.56 104.14) (xy 167.64 104.14))
     (stroke (width 0) (type default))
   )
@@
     (stroke (width 0) (type default))
   )
+  (wire (pts (xy 118.11 104.14) (xy 162.56 104.14))
+    (stroke (width 0) (type default))
+  )
   (wire (pts (xy 157.48 38.1) (xy 170.18 38.1))
     (stroke (width 0) (type default))
   )
+  (wire (pts (xy 160.02 144.78) (xy 160.02 165.1))
+    (stroke (width 0) (type default))
+  )
   (wire (pts (xy 162.56 121.92) (xy 157.48 121.92))
     (stroke (width 0) (type default))
@@
     (stroke (width 0) (type default))
   )
-  (wire (pts (xy 99.06 40.64) (xy 99.06 50.8))
+  (wire (pts (xy 170.18 38.1) (xy 170.18 63.5))
     (stroke (width 0) (type default))
   )
@@
     (stroke (width 0) (type default))
   )
-  (wire (pts (xy 176.53 96.52) (xy 165.1 96.52))
-    (stroke (width 0) (type default))
-  )

Commit message: Changed Schematic Refs (pg 2 to 4)
Parts:
- renumbered R2 to R1, R3 to R2, R1 to R3, U4 to U1, U1 to U2, U2 to U3, U3 to U4
Changed lines of the file:
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@@
   (symbol (lib_id "Device:R_Small") (at 29.972 104.14 90) (unit 1)
     (in_bom yes) (on_board yes) (dnp no) (fields_autoplaced)
-    (property "Reference" "R2" (at 29.972 99.06 90)
+    (property "Reference" "R1" (at 29.972 99.06 90)
       (effects (font (size 1.27 1.27)))
     )
@@
       (project "rps01"
         (path "/14930f15-c0a0-4b55-93e6-b112548415f6/8793e482-3b5a-4466-a30c-86f98f7c5620"
-          (reference "R2") (unit 1)
+          (reference "R1") (unit 1)
         )
       )
@@
   (symbol (lib_id "Device:R_Small") (at 29.972 109.22 270) (unit 1)
     (in_bom yes) (on_board yes) (dnp no)
-    (property "Reference" "R3" (at 29.972 111.506 90)
+    (property "Reference" "R2" (at 29.972 111.506 90)
       (effects (font (size 1.27 1.27)))
     )
@@
       (project "rps01"
         (path "/14930f15-c0a0-4b55-93e6-b112548415f6/8793e482-3b5a-4466-a30c-86f98f7c5620"
-          (reference "R3") (unit 1)
+          (reference "R2") (unit 1)
         )
       )
@@
   (symbol (lib_name "NP100P04PLG-E1-AY_1") (lib_id "2023-03-29_08-56-31:NP100P04PLG-E1-AY") (at 111.76 91.44 0) (unit 1)
     (in_bom yes) (on_board yes) (dnp no) (fields_autoplaced)
-    (property "Reference" "U3" (at 134.62 82.169 0)
+    (property "Reference" "U4" (at 134.62 82.169 0)
       (effects (font (size 1.524 1.524)))
     )
@@
       (project "rps01"
         (path "/14930f15-c0a0-4b55-93e6-b112548415f6/8793e482-3b5a-4466-a30c-86f98f7c5620"
-          (reference "U3") (unit 1)
+          (reference "U4") (unit 1)
         )
       )
@@
   (symbol (lib_id "2023-03-29_08-38-13:LTC4416EMS-1-TRPBF") (at 50.8 101.6 0) (unit 1)
     (in_bom yes) (on_board yes) (dnp no) (fields_autoplaced)
-    (property "Reference" "U4" (at 71.12 92.9386 0)
+    (property "Reference" "U1" (at 71.12 92.9386 0)
       (effects (font (size 1.524 1.524)))
     )
@@
       (project "rps01"
         (path "/14930f15-c0a0-4b55-93e6-b112548415f6/8793e482-3b5a-4466-a30c-86f98f7c5620"
-          (reference "U4") (unit 1)
+          (reference "U1") (unit 1)
         )
       )
@@
   (symbol (lib_id "power:GND") (at 49.53 106.68 270) (unit 1)
     (in_bom yes) (on_board yes) (dnp no) (fields_autoplaced)
-    (property "Reference" "#PWR012" (at 43.18 106.68 0)
+    (property "Reference" "#PWR013" (at 43.18 106.68 0)
       (effects (font (size 1.27 1.27)) hide)
     )
@@
       (project "rps01"
         (path "/14930f15-c0a0-4b55-93e6-b112548415f6/8793e482-3b5a-4466-a30c-86f98f7c5620"
-          (reference "#PWR012") (unit 1)
+          (reference "#PWR013") (unit 1)
         )
       )
@@
   (symbol (lib_id "Device:R_Small") (at 36.322 100.33 0) (unit 1)
     (in_bom yes) (on_board yes) (dnp no) (fields_autoplaced)
-    (property "Reference" "R1" (at 38.1 99.695 0)
+    (property "Reference" "R3" (at 38.1 99.695 0)
       (effects (font (size 1.27 1.27)) (justify left))
     )
@@
       (project "rps01"
         (path "/14930f15-c0a0-4b55-93e6-b112548415f6/8793e482-3b5a-4466-a30c-86f98f7c5620"
-          (reference "R1") (unit 1)
+          (reference "R3") (unit 1)
         )
       )
@@
   (symbol (lib_name "NP100P04PLG-E1-AY_1") (lib_id "2023-03-29_08-56-31:NP100P04PLG-E1-AY") (at 111.76 63.5 0) (unit 1)
     (in_bom yes) (on_board yes) (dnp no) (fields_autoplaced)
-    (property "Reference" "U2" (at 134.62 54.229 0)
+    (property "Reference" "U3" (at 134.62 54.229 0)
       (effects (font (size 1.524 1.524)))
     )
@@
       (project "rps01"
         (path "/14930f15-c0a0-4b55-93e6-b112548415f6/8793e482-3b5a-4466-a30c-86f98f7c5620"
-          (reference "U2") (unit 1)
+          (reference "U3") (unit 1)
         )
       )
@@
   (symbol (lib_id "power:GND") (at 25.908 109.22 270) (unit 1)
     (in_bom yes) (on_board yes) (dnp no)
-    (property "Reference" "#PWR013" (at 19.558 109.22 0)
+    (property "Reference" "#PWR012" (at 19.558 109.22 0)
       (effects (font (size 1.27 1.27)) hide)
     )
@@
       (project "rps01"
         (path "/14930f15-c0a0-4b55-93e6-b112548415f6/8793e482-3b5a-4466-a30c-86f98f7c5620"
-          (reference "#PWR013") (unit 1)
+          (reference "#PWR012") (unit 1)
         )
       )
@@
   (symbol (lib_name "NP100P04PLG-E1-AY_1") (lib_id "2023-03-29_08-56-31:NP100P04PLG-E1-AY") (at 111.76 38.1 0) (unit 1)
     (in_bom yes) (on_board yes) (dnp no) (fields_autoplaced)
-    (property "Reference" "U1" (at 134.62 28.829 0)
+    (property "Reference" "U2" (at 134.62 28.829 0)
       (effects (font (size 1.524 1.524)))
     )
@@
       (project "rps01"
         (path "/14930f15-c0a0-4b55-93e6-b112548415f6/8793e482-3b5a-4466-a30c-86f98f7c5620"
-          (reference "U1") (unit 1)
-        )
-      )
+          (reference "U2") (unit 1)
+        )
+      )
