File: KiCad/RPS01-Revision 2/TempSensors.kicad_sch (KiCad schematic)
At the start: 5 parts, among them U17 DS18B20+, U18 DS18B20+

Commit message: Changed Schematic Refs (pg 2 to 4)
Parts:
- renumbered U17 to U19
Changed lines of the file:
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@@
         )
         (path "/14930f15-c0a0-4b55-93e6-b112548415f6/70788b2e-4f8b-415f-94db-6db5f6e45c82"
-          (reference "J14") (unit 1)
+          (reference "J16") (unit 1)
         )
       )
@@
   (symbol (lib_id "power:GND") (at 53.086 124.968 0) (unit 1)
     (in_bom yes) (on_board yes) (dnp no) (fields_autoplaced)
-    (property "Reference" "#PWR070" (at 53.086 131.318 0)
+    (property "Reference" "#PWR085" (at 53.086 131.318 0)
       (effects (font (size 1.27 1.27)) hide)
     )
@@
       (project "rps01"
         (path "/14930f15-c0a0-4b55-93e6-b112548415f6/70788b2e-4f8b-415f-94db-6db5f6e45c82"
-          (reference "#PWR070") (unit 1)
+          (reference "#PWR085") (unit 1)
         )
       )
@@
   (symbol (lib_id "power:GND") (at 149.352 76.2 180) (unit 1)
     (in_bom yes) (on_board yes) (dnp no) (fields_autoplaced)
-    (property "Reference" "#PWR068" (at 149.352 69.85 0)
+    (property "Reference" "#PWR087" (at 149.352 69.85 0)
       (effects (font (size 1.27 1.27)) hide)
     )
@@
       (project "rps01"
         (path "/14930f15-c0a0-4b55-93e6-b112548415f6/70788b2e-4f8b-415f-94db-6db5f6e45c82"
-          (reference "#PWR068") (unit 1)
+          (reference "#PWR087") (unit 1)
         )
       )
@@
   (symbol (lib_id "power:GND") (at 125.73 88.392 270) (unit 1)
     (in_bom yes) (on_board yes) (dnp no) (fields_autoplaced)
-    (property "Reference" "#PWR069" (at 119.38 88.392 0)
+    (property "Reference" "#PWR086" (at 119.38 88.392 0)
       (effects (font (size 1.27 1.27)) hide)
     )
@@
       (project "rps01"
         (path "/14930f15-c0a0-4b55-93e6-b112548415f6/70788b2e-4f8b-415f-94db-6db5f6e45c82"
-          (reference "#PWR069") (unit 1)
+          (reference "#PWR086") (unit 1)
         )
       )
@@
   (symbol (lib_id "power:GND") (at 52.578 153.416 0) (unit 1)
     (in_bom yes) (on_board yes) (dnp no) (fields_autoplaced)
-    (property "Reference" "#PWR071" (at 52.578 159.766 0)
+    (property "Reference" "#PWR084" (at 52.578 159.766 0)
       (effects (font (size 1.27 1.27)) hide)
     )
@@
       (project "rps01"
         (path "/14930f15-c0a0-4b55-93e6-b112548415f6/70788b2e-4f8b-415f-94db-6db5f6e45c82"
-          (reference "#PWR071") (unit 1)
+          (reference "#PWR084") (unit 1)
         )
       )
@@
   (symbol (lib_id "Mechatronics TEMP:DS18B20+") (at 53.086 124.968 0) (unit 1)
     (in_bom yes) (on_board yes) (dnp no) (fields_autoplaced)
-    (property "Reference" "U17" (at 81.026 115.57 0)
+    (property "Reference" "U19" (at 81.026 115.57 0)
       (effects (font (size 1.524 1.524)))
     )
@@
       (project "rps01"
         (path "/14930f15-c0a0-4b55-93e6-b112548415f6/70788b2e-4f8b-415f-94db-6db5f6e45c82"
-          (reference "U17") (unit 1)
+          (reference "U19") (unit 1)
         )
       )
@@
         )
         (path "/14930f15-c0a0-4b55-93e6-b112548415f6/70788b2e-4f8b-415f-94db-6db5f6e45c82"
-          (reference "J13") (unit 1)
+          (reference "J17") (unit 1)
         )
       )
