File: KiCad/RPS01-Revision 2/TempSensors.kicad_sch (KiCad schematic)
At the start: 5 parts, among them U18 DS18B20+, U19 DS18B20+

Commit message: updates
Other:
- note removed: "Missing two PCB mounting TEMP sensors"
Changed lines of the file:
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@@
     (stroke (width 0) (type default))
-  )
-  (text "Missing two PCB mounting TEMP sensors" (at 127 105.918 0)
-    (effects (font (size 1.27 1.27)) (justify left bottom))
   )
   (global_label "LOGIC 5V" (shape bidirectional) (at 141.224 93.472 180) (fields_autoplaced)
