File: KiCad/RPS01-Revision 2/LLC.kicad_sch (KiCad schematic)
At the start: 12 parts, among them Q1 BSS138, Q2 BSS138

Commit message: Changed Schematic Refs (pg 2 to 4)
Parts:
- renumbered Q1 to Q5, Q2 to Q6, R17 to R24, R18 to R25, R19 to R26, R23 to R27, R22 to R28, R26 to R29, R20 to R30, R24 to R31
Changed lines of the file:
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@@
   (symbol (lib_id "Device:R_Small") (at 130.048 60.96 180) (unit 1)
     (in_bom yes) (on_board yes) (dnp no) (fields_autoplaced)
-    (property "Reference" "R17" (at 132.08 60.325 0)
+    (property "Reference" "R24" (at 132.08 60.325 0)
       (effects (font (size 1.27 1.27)) (justify right))
     )
@@
       (project "rps01"
         (path "/14930f15-c0a0-4b55-93e6-b112548415f6/c06f7478-c874-4c9c-9b0f-f3b722914738"
-          (reference "R17") (unit 1)
+          (reference "R24") (unit 1)
         )
       )
@@
   (symbol (lib_id "Transistor_FET:BSS138") (at 156.21 95.25 270) (unit 1)
     (in_bom yes) (on_board yes) (dnp no) (fields_autoplaced)
-    (property "Reference" "Q1" (at 156.21 101.6 90)
+    (property "Reference" "Q5" (at 156.21 101.6 90)
       (effects (font (size 1.27 1.27)))
     )
@@
       (project "rps01"
         (path "/14930f15-c0a0-4b55-93e6-b112548415f6/c06f7478-c874-4c9c-9b0f-f3b722914738"
-          (reference "Q1") (unit 1)
+          (reference "Q5") (unit 1)
         )
       )
@@
   (symbol (lib_id "Device:R") (at 165.1 128.27 0) (unit 1)
     (in_bom yes) (on_board yes) (dnp no) (fields_autoplaced)
-    (property "Reference" "R24" (at 167.64 127 0)
+    (property "Reference" "R31" (at 167.64 127 0)
       (effects (font (size 1.27 1.27)) (justify left))
     )
@@
       (project "rps01"
         (path "/14930f15-c0a0-4b55-93e6-b112548415f6/c06f7478-c874-4c9c-9b0f-f3b722914738"
-          (reference "R24") (unit 1)
+          (reference "R31") (unit 1)
         )
       )
@@
   (symbol (lib_id "Device:R_Small") (at 156.718 150.368 90) (unit 1)
     (in_bom yes) (on_board yes) (dnp no) (fields_autoplaced)
-    (property "Reference" "R26" (at 156.718 146.05 90)
+    (property "Reference" "R29" (at 156.718 146.05 90)
       (effects (font (size 1.27 1.27)))
     )
@@
       (project "rps01"
         (path "/14930f15-c0a0-4b55-93e6-b112548415f6/c06f7478-c874-4c9c-9b0f-f3b722914738"
-          (reference "R26") (unit 1)
+          (reference "R29") (unit 1)
         )
       )
@@
   (symbol (lib_id "Device:R_Small") (at 130.048 66.04 180) (unit 1)
     (in_bom yes) (on_board yes) (dnp no)
-    (property "Reference" "R18" (at 131.572 65.405 0)
+    (property "Reference" "R25" (at 131.572 65.405 0)
       (effects (font (size 1.27 1.27)) (justify right))
     )
@@
       (project "rps01"
         (path "/14930f15-c0a0-4b55-93e6-b112548415f6/c06f7478-c874-4c9c-9b0f-f3b722914738"
-          (reference "R18") (unit 1)
+          (reference "R25") (unit 1)
         )
       )
@@
   (symbol (lib_id "Device:R") (at 147.32 90.17 0) (unit 1)
     (in_bom yes) (on_board yes) (dnp no) (fields_autoplaced)
-    (property "Reference" "R19" (at 149.86 88.9 0)
+    (property "Reference" "R26" (at 149.86 88.9 0)
       (effects (font (size 1.27 1.27)) (justify left))
     )
@@
       (project "rps01"
         (path "/14930f15-c0a0-4b55-93e6-b112548415f6/c06f7478-c874-4c9c-9b0f-f3b722914738"
-          (reference "R19") (unit 1)
+          (reference "R26") (unit 1)
         )
       )
@@
   (symbol (lib_id "power:+3.3V") (at 147.32 120.65 0) (unit 1)
     (in_bom yes) (on_board yes) (dnp no) (fields_autoplaced)
-    (property "Reference" "#PWR066" (at 147.32 124.46 0)
+    (property "Reference" "#PWR083" (at 147.32 124.46 0)
       (effects (font (size 1.27 1.27)) hide)
     )
@@
       (project "rps01"
         (path "/14930f15-c0a0-4b55-93e6-b112548415f6/c06f7478-c874-4c9c-9b0f-f3b722914738"
-          (reference "#PWR066") (unit 1)
+          (reference "#PWR083") (unit 1)
         )
       )
@@
   (symbol (lib_id "power:+5V") (at 130.048 68.58 180) (unit 1)
     (in_bom yes) (on_board yes) (dnp no) (fields_autoplaced)
-    (property "Reference" "#PWR063" (at 130.048 64.77 0)
+    (property "Reference" "#PWR081" (at 130.048 64.77 0)
       (effects (font (size 1.27 1.27)) hide)
     )
@@
       (project "rps01"
         (path "/14930f15-c0a0-4b55-93e6-b112548415f6/c06f7478-c874-4c9c-9b0f-f3b722914738"
-          (reference "#PWR063") (unit 1)
+          (reference "#PWR081") (unit 1)
         )
       )
@@
   (symbol (lib_id "Transistor_FET:BSS138") (at 156.21 133.35 270) (unit 1)
     (in_bom yes) (on_board yes) (dnp no) (fields_autoplaced)
-    (property "Reference" "Q2" (at 156.21 139.7 90)
+    (property "Reference" "Q6" (at 156.21 139.7 90)
       (effects (font (size 1.27 1.27)))
     )
@@
       (project "rps01"
         (path "/14930f15-c0a0-4b55-93e6-b112548415f6/c06f7478-c874-4c9c-9b0f-f3b722914738"
-          (reference "Q2") (unit 1)
+          (reference "Q6") (unit 1)
         )
       )
@@
   (symbol (lib_id "Device:R") (at 147.32 128.27 0) (unit 1)
     (in_bom yes) (on_board yes) (dnp no) (fields_autoplaced)
-    (property "Reference" "R23" (at 149.86 127 0)
+    (property "Reference" "R27" (at 149.86 127 0)
       (effects (font (size 1.27 1.27)) (justify left))
     )
@@
       (project "rps01"
         (path "/14930f15-c0a0-4b55-93e6-b112548415f6/c06f7478-c874-4c9c-9b0f-f3b722914738"
-          (reference "R23") (unit 1)
+          (reference "R27") (unit 1)
         )
       )
@@
   (symbol (lib_id "power:+3.3V") (at 147.32 80.01 0) (unit 1)
     (in_bom yes) (on_board yes) (dnp no) (fields_autoplaced)
-    (property "Reference" "#PWR064" (at 147.32 83.82 0)
+    (property "Reference" "#PWR082" (at 147.32 83.82 0)
       (effects (font (size 1.27 1.27)) hide)
     )
@@
       (project "rps01"
         (path "/14930f15-c0a0-4b55-93e6-b112548415f6/c06f7478-c874-4c9c-9b0f-f3b722914738"
-          (reference "#PWR064") (unit 1)
+          (reference "#PWR082") (unit 1)
         )
       )
@@
   (symbol (lib_id "Device:R") (at 163.83 90.17 0) (unit 1)
     (in_bom yes) (on_board yes) (dnp no) (fields_autoplaced)
-    (property "Reference" "R20" (at 166.37 88.9 0)
+    (property "Reference" "R30" (at 166.37 88.9 0)
       (effects (font (size 1.27 1.27)) (justify left))
     )
@@
       (project "rps01"
         (path "/14930f15-c0a0-4b55-93e6-b112548415f6/c06f7478-c874-4c9c-9b0f-f3b722914738"
-          (reference "R20") (unit 1)
+          (reference "R30") (unit 1)
         )
       )
@@
   (symbol (lib_id "power:+3.3V") (at 130.048 58.42 0) (unit 1)
     (in_bom yes) (on_board yes) (dnp no) (fields_autoplaced)
-    (property "Reference" "#PWR062" (at 130.048 62.23 0)
+    (property "Reference" "#PWR080" (at 130.048 62.23 0)
       (effects (font (size 1.27 1.27)) hide)
     )
@@
       (project "rps01"
         (path "/14930f15-c0a0-4b55-93e6-b112548415f6/c06f7478-c874-4c9c-9b0f-f3b722914738"
-          (reference "#PWR062") (unit 1)
+          (reference "#PWR080") (unit 1)
         )
       )
@@
   (symbol (lib_id "Device:R_Small") (at 155.956 111.506 90) (unit 1)
     (in_bom yes) (on_board yes) (dnp no) (fields_autoplaced)
-    (property "Reference" "R22" (at 155.956 106.68 90)
+    (property "Reference" "R28" (at 155.956 106.68 90)
       (effects (font (size 1.27 1.27)))
     )
@@
       (project "rps01"
         (path "/14930f15-c0a0-4b55-93e6-b112548415f6/c06f7478-c874-4c9c-9b0f-f3b722914738"
-          (reference "R22") (unit 1)
+          (reference "R28") (unit 1)
         )
       )
@@
         )
         (path "/14930f15-c0a0-4b55-93e6-b112548415f6/c06f7478-c874-4c9c-9b0f-f3b722914738"
-          (reference "R25") (unit 1)
+          (reference "R33") (unit 1)
         )
       )
@@
         )
         (path "/14930f15-c0a0-4b55-93e6-b112548415f6/c06f7478-c874-4c9c-9b0f-f3b722914738"
-          (reference "R21") (unit 1)
-        )
-      )
+          (reference "R32") (unit 1)
+        )
+      )

Commit message: Reduced the References for Peter
Parts:
- renumbered R24 to R34, R25 to R35, R26 to R36, R27 to R37, R28 to R38, R29 to R39, R30 to R40, R31 to R41
Changed lines of the file:
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@@
   (symbol (lib_id "Device:R_Small") (at 130.048 60.96 180) (unit 1)
     (in_bom yes) (on_board yes) (dnp no) (fields_autoplaced)
-    (property "Reference" "R24" (at 132.08 60.325 0)
+    (property "Reference" "R34" (at 132.08 60.325 0)
       (effects (font (size 1.27 1.27)) (justify right))
     )
@@
       (project "rps01"
         (path "/14930f15-c0a0-4b55-93e6-b112548415f6/c06f7478-c874-4c9c-9b0f-f3b722914738"
-          (reference "R24") (unit 1)
+          (reference "R34") (unit 1)
         )
       )
@@
   (symbol (lib_id "Device:R") (at 165.1 128.27 0) (unit 1)
     (in_bom yes) (on_board yes) (dnp no) (fields_autoplaced)
-    (property "Reference" "R31" (at 167.64 127 0)
+    (property "Reference" "R41" (at 167.64 127 0)
       (effects (font (size 1.27 1.27)) (justify left))
     )
@@
       (project "rps01"
         (path "/14930f15-c0a0-4b55-93e6-b112548415f6/c06f7478-c874-4c9c-9b0f-f3b722914738"
-          (reference "R31") (unit 1)
+          (reference "R41") (unit 1)
         )
       )
@@
   (symbol (lib_id "Device:R_Small") (at 156.718 150.368 90) (unit 1)
     (in_bom yes) (on_board yes) (dnp no) (fields_autoplaced)
-    (property "Reference" "R29" (at 156.718 146.05 90)
+    (property "Reference" "R39" (at 156.718 146.05 90)
       (effects (font (size 1.27 1.27)))
     )
@@
       (project "rps01"
         (path "/14930f15-c0a0-4b55-93e6-b112548415f6/c06f7478-c874-4c9c-9b0f-f3b722914738"
-          (reference "R29") (unit 1)
+          (reference "R39") (unit 1)
         )
       )
@@
   (symbol (lib_id "Device:R_Small") (at 130.048 66.04 180) (unit 1)
     (in_bom yes) (on_board yes) (dnp no)
-    (property "Reference" "R25" (at 131.572 65.405 0)
+    (property "Reference" "R35" (at 131.572 65.405 0)
       (effects (font (size 1.27 1.27)) (justify right))
     )
@@
       (project "rps01"
         (path "/14930f15-c0a0-4b55-93e6-b112548415f6/c06f7478-c874-4c9c-9b0f-f3b722914738"
-          (reference "R25") (unit 1)
+          (reference "R35") (unit 1)
         )
       )
@@
   (symbol (lib_id "Device:R") (at 147.32 90.17 0) (unit 1)
     (in_bom yes) (on_board yes) (dnp no) (fields_autoplaced)
-    (property "Reference" "R26" (at 149.86 88.9 0)
+    (property "Reference" "R36" (at 149.86 88.9 0)
       (effects (font (size 1.27 1.27)) (justify left))
     )
@@
       (project "rps01"
         (path "/14930f15-c0a0-4b55-93e6-b112548415f6/c06f7478-c874-4c9c-9b0f-f3b722914738"
-          (reference "R26") (unit 1)
+          (reference "R36") (unit 1)
         )
       )
@@
   (symbol (lib_id "Device:R") (at 147.32 128.27 0) (unit 1)
     (in_bom yes) (on_board yes) (dnp no) (fields_autoplaced)
-    (property "Reference" "R27" (at 149.86 127 0)
+    (property "Reference" "R37" (at 149.86 127 0)
       (effects (font (size 1.27 1.27)) (justify left))
     )
@@
       (project "rps01"
         (path "/14930f15-c0a0-4b55-93e6-b112548415f6/c06f7478-c874-4c9c-9b0f-f3b722914738"
-          (reference "R27") (unit 1)
+          (reference "R37") (unit 1)
         )
       )
@@
   (symbol (lib_id "Device:R") (at 163.83 90.17 0) (unit 1)
     (in_bom yes) (on_board yes) (dnp no) (fields_autoplaced)
-    (property "Reference" "R30" (at 166.37 88.9 0)
+    (property "Reference" "R40" (at 166.37 88.9 0)
       (effects (font (size 1.27 1.27)) (justify left))
     )
@@
       (project "rps01"
         (path "/14930f15-c0a0-4b55-93e6-b112548415f6/c06f7478-c874-4c9c-9b0f-f3b722914738"
-          (reference "R30") (unit 1)
+          (reference "R40") (unit 1)
         )
       )
@@
   (symbol (lib_id "Device:R_Small") (at 155.956 111.506 90) (unit 1)
     (in_bom yes) (on_board yes) (dnp no) (fields_autoplaced)
-    (property "Reference" "R28" (at 155.956 106.68 90)
+    (property "Reference" "R38" (at 155.956 106.68 90)
       (effects (font (size 1.27 1.27)))
     )
@@
       (project "rps01"
         (path "/14930f15-c0a0-4b55-93e6-b112548415f6/c06f7478-c874-4c9c-9b0f-f3b722914738"
-          (reference "R28") (unit 1)
+          (reference "R38") (unit 1)
         )
       )
@@
         )
         (path "/14930f15-c0a0-4b55-93e6-b112548415f6/c06f7478-c874-4c9c-9b0f-f3b722914738"
-          (reference "R33") (unit 1)
+          (reference "R43") (unit 1)
         )
       )
@@
         )
         (path "/14930f15-c0a0-4b55-93e6-b112548415f6/c06f7478-c874-4c9c-9b0f-f3b722914738"
-          (reference "R32") (unit 1)
-        )
-      )
+          (reference "R42") (unit 1)
+        )
+      )
