File: KiCad/RPS01-Revision 2/rps01.kicad_sch (KiCad schematic)
At the start: 10 parts, among them J1 XT90 Battery VOUT 1, J10 IIC Connector, J2 BATT IN 1 XT90, J3 XT90 Battery VOUT 2, J4 XT30PW Batt VOUT, J5 BATT IN 2 XT90, J9 XT30PW 19V

Commit message: Changed Schematic Refs (pg 2 to 4)
Parts:
- renumbered J5 to J1, J9 to J10, J4 to J3, J3 to J4, J1 to J5, J10 to J9
Changed lines of the file:
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@@
   (symbol (lib_id "power:GND") (at 251.0282 34.036 0) (unit 1)
     (in_bom yes) (on_board yes) (dnp no) (fields_autoplaced)
-    (property "Reference" "#PWR01" (at 251.0282 40.386 0)
+    (property "Reference" "#PWR06" (at 251.0282 40.386 0)
       (effects (font (size 1.27 1.27)) hide)
     )
@@
       (project "rps01"
         (path "/14930f15-c0a0-4b55-93e6-b112548415f6"
+          (reference "#PWR06") (unit 1)
+        )
+      )
+    )
+  )
+  (symbol (lib_id "power:GND") (at 251.2314 66.04 0) (unit 1)
+    (in_bom yes) (on_board yes) (dnp no) (fields_autoplaced)
+    (property "Reference" "#PWR07" (at 251.2314 72.39 0)
+      (effects (font (size 1.27 1.27)) hide)
+    )
+    (property "Value" "GND" (at 251.2314 71.7296 0)
+      (effects (font (size 1.27 1.27)))
+    )
+    (property "Footprint" "" (at 251.2314 66.04 0)
+      (effects (font (size 1.27 1.27)) hide)
+    )
+    (property "Datasheet" "" (at 251.2314 66.04 0)
+      (effects (font (size 1.27 1.27)) hide)
+    )
+    (pin "1")
+    (instances
+      (project "rps01"
+        (path "/14930f15-c0a0-4b55-93e6-b112548415f6"
+          (reference "#PWR07") (unit 1)
+        )
+      )
+    )
+  )
+  (symbol (lib_id "power:GND") (at 44.196 39.624 0) (unit 1)
+    (in_bom yes) (on_board yes) (dnp no) (fields_autoplaced)
+    (property "Reference" "#PWR02" (at 44.196 45.974 0)
+      (effects (font (size 1.27 1.27)) hide)
+    )
+    (property "Value" "GND" (at 44.196 44.704 0)
+      (effects (font (size 1.27 1.27)))
+    )
+    (property "Footprint" "" (at 44.196 39.624 0)
+      (effects (font (size 1.27 1.27)) hide)
+    )
+    (property "Datasheet" "" (at 44.196 39.624 0)
+      (effects (font (size 1.27 1.27)) hide)
+    )
+    (pin "1")
+    (instances
+      (project "rps01"
+        (path "/14930f15-c0a0-4b55-93e6-b112548415f6"
+          (reference "#PWR02") (unit 1)
+        )
+      )
+    )
+  )
+  (symbol (lib_id "power:GND") (at 43.942 66.294 0) (unit 1)
+    (in_bom yes) (on_board yes) (dnp no) (fields_autoplaced)
+    (property "Reference" "#PWR01" (at 43.942 72.644 0)
+      (effects (font (size 1.27 1.27)) hide)
+    )
+    (property "Value" "GND" (at 43.942 71.374 0)
+      (effects (font (size 1.27 1.27)))
+    )
+    (property "Footprint" "" (at 43.942 66.294 0)
+      (effects (font (size 1.27 1.27)) hide)
+    )
+    (property "Datasheet" "" (at 43.942 66.294 0)
+      (effects (font (size 1.27 1.27)) hide)
+    )
+    (pin "1")
+    (instances
+      (project "rps01"
+        (path "/14930f15-c0a0-4b55-93e6-b112548415f6"
           (reference "#PWR01") (unit 1)
-        )
-      )
-    )
-  )
-  (symbol (lib_id "power:GND") (at 251.2314 66.04 0) (unit 1)
-    (in_bom yes) (on_board yes) (dnp no) (fields_autoplaced)
-    (property "Reference" "#PWR05" (at 251.2314 72.39 0)
-      (effects (font (size 1.27 1.27)) hide)
-    )
-    (property "Value" "GND" (at 251.2314 71.7296 0)
-      (effects (font (size 1.27 1.27)))
-    )
-    (property "Footprint" "" (at 251.2314 66.04 0)
-      (effects (font (size 1.27 1.27)) hide)
-    )
-    (property "Datasheet" "" (at 251.2314 66.04 0)
-      (effects (font (size 1.27 1.27)) hide)
-    )
-    (pin "1")
-    (instances
-      (project "rps01"
-        (path "/14930f15-c0a0-4b55-93e6-b112548415f6"
-          (reference "#PWR05") (unit 1)
-        )
-      )
-    )
-  )
-  (symbol (lib_id "power:GND") (at 44.196 39.624 0) (unit 1)
-    (in_bom yes) (on_board yes) (dnp no) (fields_autoplaced)
-    (property "Reference" "#PWR02" (at 44.196 45.974 0)
-      (effects (font (size 1.27 1.27)) hide)
-    )
-    (property "Value" "GND" (at 44.196 44.704 0)
-      (effects (font (size 1.27 1.27)))
-    )
-    (property "Footprint" "" (at 44.196 39.624 0)
-      (effects (font (size 1.27 1.27)) hide)
-    )
-    (property "Datasheet" "" (at 44.196 39.624 0)
-      (effects (font (size 1.27 1.27)) hide)
-    )
-    (pin "1")
-    (instances
-      (project "rps01"
-        (path "/14930f15-c0a0-4b55-93e6-b112548415f6"
-          (reference "#PWR02") (unit 1)
-        )
-      )
-    )
-  )
-  (symbol (lib_id "power:GND") (at 43.942 66.294 0) (unit 1)
-    (in_bom yes) (on_board yes) (dnp no) (fields_autoplaced)
-    (property "Reference" "#PWR06" (at 43.942 72.644 0)
-      (effects (font (size 1.27 1.27)) hide)
-    )
-    (property "Value" "GND" (at 43.942 71.374 0)
-      (effects (font (size 1.27 1.27)))
-    )
-    (property "Footprint" "" (at 43.942 66.294 0)
-      (effects (font (size 1.27 1.27)) hide)
-    )
-    (property "Datasheet" "" (at 43.942 66.294 0)
-      (effects (font (size 1.27 1.27)) hide)
-    )
-    (pin "1")
-    (instances
-      (project "rps01"
-        (path "/14930f15-c0a0-4b55-93e6-b112548415f6"
-          (reference "#PWR06") (unit 1)
         )
       )
@@
         )
         (path "/14930f15-c0a0-4b55-93e6-b112548415f6"
-          (reference "#PWR010") (unit 1)
+          (reference "#PWR08") (unit 1)
         )
       )
@@
   (symbol (lib_id "Connector:Conn_01x02_Pin") (at 265.176 147.574 180) (unit 1)
     (in_bom yes) (on_board yes) (dnp no) (fields_autoplaced)
-    (property "Reference" "J9" (at 266.7 145.669 0)
+    (property "Reference" "J10" (at 266.7 145.669 0)
       (effects (font (size 1.27 1.27)) (justify right))
     )
@@
       (project "rps01"
         (path "/14930f15-c0a0-4b55-93e6-b112548415f6"
-          (reference "J9") (unit 1)
+          (reference "J10") (unit 1)
         )
       )
@@
   (symbol (lib_id "Connector:Conn_01x02_Socket") (at 256.9718 50.292 0) (mirror x) (unit 1)
     (in_bom yes) (on_board yes) (dnp no)
-    (property "Reference" "J3" (at 258.2418 49.657 0)
+    (property "Reference" "J4" (at 258.2418 49.657 0)
       (effects (font (size 1.27 1.27)) (justify left))
     )
@@
       (project "rps01"
         (path "/14930f15-c0a0-4b55-93e6-b112548415f6"
-          (reference "J3") (unit 1)
+          (reference "J4") (unit 1)
         )
       )
@@
         )
         (path "/14930f15-c0a0-4b55-93e6-b112548415f6"
-          (reference "J6") (unit 1)
+          (reference "J8") (unit 1)
         )
       )
@@
   (symbol (lib_id "Connector:Conn_01x02_Socket") (at 38.862 66.294 180) (unit 1)
     (in_bom yes) (on_board yes) (dnp no)
-    (property "Reference" "J5" (at 26.416 64.262 0)
+    (property "Reference" "J1" (at 26.416 64.262 0)
       (effects (font (size 1.27 1.27)))
     )
@@
       (project "rps01"
         (path "/14930f15-c0a0-4b55-93e6-b112548415f6"
-          (reference "J5") (unit 1)
+          (reference "J1") (unit 1)
         )
       )
@@
         )
         (path "/14930f15-c0a0-4b55-93e6-b112548415f6"
-          (reference "#PWR08") (unit 1)
+          (reference "#PWR09") (unit 1)
         )
       )
@@
         )
         (path "/14930f15-c0a0-4b55-93e6-b112548415f6"
-          (reference "J8") (unit 1)
+          (reference "J6") (unit 1)
         )
       )
@@
   (symbol (lib_id "power:GND") (at 250.698 50.292 0) (unit 1)
     (in_bom yes) (on_board yes) (dnp no) (fields_autoplaced)
-    (property "Reference" "#PWR04" (at 250.698 56.642 0)
+    (property "Reference" "#PWR05" (at 250.698 56.642 0)
       (effects (font (size 1.27 1.27)) hide)
     )
@@
       (project "rps01"
         (path "/14930f15-c0a0-4b55-93e6-b112548415f6"
-          (reference "#PWR04") (unit 1)
+          (reference "#PWR05") (unit 1)
         )
       )
@@
         )
         (path "/14930f15-c0a0-4b55-93e6-b112548415f6"
-          (reference "#PWR07") (unit 1)
+          (reference "#PWR011") (unit 1)
         )
       )
@@
   (symbol (lib_id "Connector:Conn_01x04_Pin") (at 264.16 159.258 180) (unit 1)
     (in_bom yes) (on_board yes) (dnp no) (fields_autoplaced)
-    (property "Reference" "J10" (at 265.176 157.353 0)
+    (property "Reference" "J9" (at 265.176 157.353 0)
       (effects (font (size 1.27 1.27)) (justify right))
     )
@@
       (project "rps01"
         (path "/14930f15-c0a0-4b55-93e6-b112548415f6"
-          (reference "J10") (unit 1)
+          (reference "J9") (unit 1)
         )
       )
@@
   (symbol (lib_id "power:GND") (at 214.884 163.83 270) (unit 1)
     (in_bom yes) (on_board yes) (dnp no) (fields_autoplaced)
-    (property "Reference" "#PWR011" (at 208.534 163.83 0)
+    (property "Reference" "#PWR04" (at 208.534 163.83 0)
       (effects (font (size 1.27 1.27)) hide)
     )
@@
       (project "rps01"
         (path "/14930f15-c0a0-4b55-93e6-b112548415f6"
-          (reference "#PWR011") (unit 1)
+          (reference "#PWR04") (unit 1)
         )
       )
@@
         )
         (path "/14930f15-c0a0-4b55-93e6-b112548415f6"
-          (reference "#PWR09") (unit 1)
+          (reference "#PWR010") (unit 1)
         )
       )
@@
   (symbol (lib_id "Connector:Conn_01x02_Socket") (at 257.302 34.036 0) (mirror x) (unit 1)
     (in_bom yes) (on_board yes) (dnp no)
-    (property "Reference" "J1" (at 258.572 33.401 0)
+    (property "Reference" "J5" (at 258.572 33.401 0)
       (effects (font (size 1.27 1.27)) (justify left))
     )
@@
       (project "rps01"
         (path "/14930f15-c0a0-4b55-93e6-b112548415f6"
-          (reference "J1") (unit 1)
+          (reference "J5") (unit 1)
         )
       )
@@
   (symbol (lib_id "Connector:Conn_01x02_Pin") (at 256.3114 66.04 180) (unit 1)
     (in_bom yes) (on_board yes) (dnp no) (fields_autoplaced)
-    (property "Reference" "J4" (at 257.81 64.135 0)
+    (property "Reference" "J3" (at 257.81 64.135 0)
       (effects (font (size 1.27 1.27)) (justify right))
     )
@@
       (project "rps01"
         (path "/14930f15-c0a0-4b55-93e6-b112548415f6"
-          (reference "J4") (unit 1)
-        )
-      )
+          (reference "J3") (unit 1)
+        )
+      )

Commit message: Completed Schematic
Other:
- sheet Current Sense Rails ports: added VOUT; removed LOAD
- sheet Current Sense Total ports: added VOUT; removed LOAD
- sheet Displays and Indicators ports: added none; removed SCL, SDA
Changed lines of the file:
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@@
     (stroke (width 0) (type default))
   )
-  (wire (pts (xy 59.944 129.032) (xy 65.786 129.032))
-    (stroke (width 0) (type default))
-  )
   (wire (pts (xy 43.942 63.754) (xy 48.006 63.754))
     (stroke (width 0) (type default))
   )
-  (wire (pts (xy 59.69 140.462) (xy 65.786 140.462))
-    (stroke (width 0) (type default))
-  )
   (wire (pts (xy 184.912 159.258) (xy 184.912 130.556))
     (stroke (width 0) (type default))
@@
     )
   )
-  (global_label "SDA" (shape bidirectional) (at 59.944 129.032 180) (fields_autoplaced)
-    (effects (font (size 1.27 1.27)) (justify right))
-    (property "Intersheetrefs" "${INTERSHEET_REFS}" (at 52.3588 129.032 0)
-      (effects (font (size 1.27 1.27)) (justify right) hide)
-    )
-  )
-  (global_label "SCL" (shape bidirectional) (at 59.69 140.462 180) (fields_autoplaced)
-    (effects (font (size 1.27 1.27)) (justify right))
-    (property "Intersheetrefs" "${INTERSHEET_REFS}" (at 52.1653 140.462 0)
-      (effects (font (size 1.27 1.27)) (justify right) hide)
-    )
-  )
   (global_label "LOAD SHARING VOUT" (shape bidirectional) (at 114.808 51.308 90) (fields_autoplaced)
     (effects (font (size 1.27 1.27)) (justify left))
@@
       (effects (font (size 1.27 1.27)) (justify left top))
     )
-    (pin "LOAD" input (at 148.082 51.816 0)
+    (pin "VOUT" input (at 148.082 51.816 0)
       (effects (font (size 1.27 1.27)) (justify right))
     )
@@
       (effects (font (size 1.27 1.27)) (justify right))
     )
-    (pin "SDA" bidirectional (at 65.786 129.032 180)
-      (effects (font (size 1.27 1.27)) (justify left))
-    )
-    (pin "SCL" bidirectional (at 65.786 140.462 180)
-      (effects (font (size 1.27 1.27)) (justify left))
-    )
     (instances
       (project "rps01"
@@
       (effects (font (size 1.27 1.27)) (justify left top))
     )
-    (pin "VIN" bidirectional (at 210.82 95.25 180)
-      (effects (font (size 1.27 1.27)) (justify left))
-    )
     (pin "+5V" bidirectional (at 232.918 100.33 0)
       (effects (font (size 1.27 1.27)) (justify right))
@@
       (effects (font (size 1.27 1.27)) (justify right))
     )
+    (pin "VIN" input (at 210.82 95.25 180)
+      (effects (font (size 1.27 1.27)) (justify left))
+    )
     (instances
       (project "rps01"
@@
       (effects (font (size 1.27 1.27)) (justify left))
     )
-    (pin "LOAD" input (at 199.136 95.25 0)
+    (pin "VOUT" input (at 199.136 95.25 0)
       (effects (font (size 1.27 1.27)) (justify right))
     )

Commit message: Update
Connections:
- net +BATT: no longer J3.2 (Pin_2)
- net +BATT2: now also J3.2 (Pin_2)
Changed lines of the file:
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@@
   (junction (at 157.226 51.816) (diameter 0) (color 0 0 0 0)
   )
+  (junction (at 208.534 95.25) (diameter 0) (color 0 0 0 0)
+  )
   (junction (at 157.226 47.752) (diameter 0) (color 0 0 0 0)
   )
@@
     (stroke (width 0) (type default))
   )
-  (wire (pts (xy 230.124 63.5) (xy 251.2314 63.5))
+  (wire (pts (xy 208.534 63.5) (xy 251.2314 63.5))
     (stroke (width 0) (type default))
   )
@@
     (stroke (width 0) (type default))
   )
+  (wire (pts (xy 208.534 95.25) (xy 210.82 95.25))
+    (stroke (width 0) (type default))
+  )
   (wire (pts (xy 262.128 90.17) (xy 262.128 90.932))
     (stroke (width 0) (type default))
@@
     (stroke (width 0) (type default))
   )
+  (wire (pts (xy 208.534 63.5) (xy 208.534 95.25))
+    (stroke (width 0) (type default))
+  )
   (wire (pts (xy 157.226 47.752) (xy 230.124 47.752))
     (stroke (width 0) (type default))
@@
     (stroke (width 0) (type default))
   )
-  (wire (pts (xy 199.136 95.25) (xy 210.82 95.25))
+  (wire (pts (xy 199.136 95.25) (xy 208.534 95.25))
     (stroke (width 0) (type default))
   )
@@
     (stroke (width 0) (type default))
   )
-  (wire (pts (xy 230.124 47.752) (xy 230.124 63.5))
-    (stroke (width 0) (type default))
-  )
