File: KiCad/RPS01-Revision 2/Probe.kicad_sch (KiCad schematic)
At the start: 19 parts

Commit message: Changed Schematic Refs (pg 2 to 4)
Parts:
- renumbered H3 to H2, H5 to H3, H2 to H4, H4 to H5, TP8 to TP10, TP9 to TP11, TP10 to TP12, TP17 to TP13, TP13 to TP14, TP14 to TP15, TP15 to TP16, TP16 to TP17, TP3 to TP5, TP4 to TP6, TP5 to TP7, TP6 to TP8, TP7 to TP9

Commit message: updates
Parts:
- removed TP13: GND, Mechatronics TestP:CONN1_RCU-0C_TEC, symbol Connector:TestPoint_Probe
- removed TP14: 3.3V, Mechatronics TestP:CONN1_RCU-0C_TEC, symbol Connector:TestPoint_Probe
- removed TP15: 5V, Mechatronics TestP:CONN1_RCU-0C_TEC, symbol Connector:TestPoint_Probe
- removed TP16: 12V, Mechatronics TestP:CONN1_RCU-0C_TEC, symbol Connector:TestPoint_Probe
- removed TP17: 19V, Mechatronics TestP:CONN1_RCU-0C_TEC, symbol Connector:TestPoint_Probe
- removed TP5: SDA, Mechatronics TestP:CONN1_RCU-0C_TEC, symbol Connector:TestPoint_Probe
- removed TP6: SCL, Mechatronics TestP:CONN1_RCU-0C_TEC, symbol Connector:TestPoint_Probe
- renumbered TP12 to TP10, TP7 to TP5, TP8 to TP6, TP9 to TP7, TP10 to TP8, TP11 to TP9

Commit message: Finished PCB
Parts:
- removed TP10: LOGIC 5V, Mechatronics TestP:CONN1_RCU-0C_TEC, symbol Connector:TestPoint_Probe
- removed TP5: CURRENT1, Mechatronics TestP:CONN1_RCU-0C_TEC, symbol Connector:TestPoint_Probe
- removed TP6: CURRENT2, Mechatronics TestP:CONN1_RCU-0C_TEC, symbol Connector:TestPoint_Probe
- removed TP7: VOLT1, Mechatronics TestP:CONN1_RCU-0C_TEC, symbol Connector:TestPoint_Probe
- removed TP8: VOLT2, Mechatronics TestP:CONN1_RCU-0C_TEC, symbol Connector:TestPoint_Probe
- removed TP9: AREF, Mechatronics TestP:CONN1_RCU-0C_TEC, symbol Connector:TestPoint_Probe
Changed lines of the file:
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@@
 (kicad_sch (version 20230121) (generator eeschema)
   (paper "A4")
-  (wire (pts (xy 75.692 110.236) (xy 88.392 110.236))
-    (stroke (width 0) (type default))
-  )
-  (wire (pts (xy 75.692 130.556) (xy 88.392 130.556))
-    (stroke (width 0) (type default))
-  )
-  (wire (pts (xy 75.692 123.952) (xy 88.392 123.952))
-    (stroke (width 0) (type default))
-  )
-  (wire (pts (xy 75.438 103.632) (xy 88.138 103.632))
-    (stroke (width 0) (type default))
-  )
-  (wire (pts (xy 75.692 117.094) (xy 88.392 117.094))
-    (stroke (width 0) (type default))
-  )
-  (wire (pts (xy 75.438 97.028) (xy 88.138 97.028))
-    (stroke (width 0) (type default))
-  )
-  (global_label "CURRENT2" (shape bidirectional) (at 75.438 103.632 180) (fields_autoplaced)
-    (effects (font (size 1.27 1.27)) (justify right))
-    (property "Intersheetrefs" "${INTERSHEET_REFS}" (at 61.6238 103.632 0)
-      (effects (font (size 1.27 1.27)) (justify right) hide)
-    )
-  )
-  (global_label "LOGIC 5V" (shape bidirectional) (at 75.692 130.556 180) (fields_autoplaced)
-    (effects (font (size 1.27 1.27)) (justify right))
-    (property "Intersheetrefs" "${INTERSHEET_REFS}" (at 62.9058 130.556 0)
-      (effects (font (size 1.27 1.27)) (justify right) hide)
-    )
-  )
-  (global_label "AREF" (shape bidirectional) (at 75.692 123.952 180) (fields_autoplaced)
-    (effects (font (size 1.27 1.27)) (justify right))
-    (property "Intersheetrefs" "${INTERSHEET_REFS}" (at 67.0787 123.952 0)
-      (effects (font (size 1.27 1.27)) (justify right) hide)
-    )
-  )
-  (global_label "CURRENT1" (shape bidirectional) (at 75.438 97.028 180) (fields_autoplaced)
-    (effects (font (size 1.27 1.27)) (justify right))
-    (property "Intersheetrefs" "${INTERSHEET_REFS}" (at 61.6238 97.028 0)
-      (effects (font (size 1.27 1.27)) (justify right) hide)
-    )
-  )
-  (global_label "VOLT2" (shape bidirectional) (at 75.692 117.094 180) (fields_autoplaced)
-    (effects (font (size 1.27 1.27)) (justify right))
-    (property "Intersheetrefs" "${INTERSHEET_REFS}" (at 66.0506 117.094 0)
-      (effects (font (size 1.27 1.27)) (justify right) hide)
-    )
-  )
-  (global_label "VOLT1" (shape bidirectional) (at 75.692 110.236 180) (fields_autoplaced)
-    (effects (font (size 1.27 1.27)) (justify right))
-    (property "Intersheetrefs" "${INTERSHEET_REFS}" (at 66.0506 110.236 0)
-      (effects (font (size 1.27 1.27)) (justify right) hide)
-    )
-  )
   (symbol (lib_id "Mechanical:MountingHole_Pad") (at 143.002 84.328 0) (unit 1)
     (in_bom yes) (on_board yes) (dnp no) (fields_autoplaced)
@@
     )
   )
-  (symbol (lib_id "Connector:TestPoint_Probe") (at 88.392 130.556 0) (unit 1)
-    (in_bom yes) (on_board yes) (dnp no) (fields_autoplaced)
-    (property "Reference" "TP10" (at 92.71 128.3335 0)
-      (effects (font (size 1.27 1.27)) (justify left))
-    )
-    (property "Value" "LOGIC 5V" (at 92.71 130.8735 0)
-      (effects (font (size 1.27 1.27)) (justify left))
-    )
-    (property "Footprint" "Mechatronics TestP:CONN1_RCU-0C_TEC" (at 93.472 130.556 0)
-      (effects (font (size 1.27 1.27)) hide)
-    )
-    (property "Datasheet" "~" (at 93.472 130.556 0)
-      (effects (font (size 1.27 1.27)) hide)
-    )
-    (pin "1")
-    (instances
-      (project "rps01"
-        (path "/14930f15-c0a0-4b55-93e6-b112548415f6/577d3fc4-735f-4981-a3a1-4300f23b9ae6"
-          (reference "TP10") (unit 1)
-        )
-      )
-    )
-  )
   (symbol (lib_id "power:GND") (at 169.164 86.868 0) (unit 1)
     (in_bom yes) (on_board yes) (dnp no) (fields_autoplaced)
@@
     )
   )
-  (symbol (lib_id "Connector:TestPoint_Probe") (at 88.392 110.236 0) (unit 1)
-    (in_bom yes) (on_board yes) (dnp no) (fields_autoplaced)
-    (property "Reference" "TP7" (at 92.71 108.0135 0)
-      (effects (font (size 1.27 1.27)) (justify left))
-    )
-    (property "Value" "VOLT1" (at 92.71 110.5535 0)
-      (effects (font (size 1.27 1.27)) (justify left))
-    )
-    (property "Footprint" "Mechatronics TestP:CONN1_RCU-0C_TEC" (at 93.472 110.236 0)
-      (effects (font (size 1.27 1.27)) hide)
-    )
-    (property "Datasheet" "~" (at 93.472 110.236 0)
-      (effects (font (size 1.27 1.27)) hide)
-    )
-    (pin "1")
-    (instances
-      (project "rps01"
-        (path "/14930f15-c0a0-4b55-93e6-b112548415f6/577d3fc4-735f-4981-a3a1-4300f23b9ae6"
-          (reference "TP7") (unit 1)
-        )
-      )
-    )
-  )
   (symbol (lib_id "power:GND") (at 169.418 112.014 0) (unit 1)
     (in_bom yes) (on_board yes) (dnp no) (fields_autoplaced)
@@
     )
   )
-  (symbol (lib_id "Connector:TestPoint_Probe") (at 88.392 123.952 0) (unit 1)
-    (in_bom yes) (on_board yes) (dnp no) (fields_autoplaced)
-    (property "Reference" "TP9" (at 92.71 121.7295 0)
-      (effects (font (size 1.27 1.27)) (justify left))
-    )
-    (property "Value" "AREF" (at 92.71 124.2695 0)
-      (effects (font (size 1.27 1.27)) (justify left))
-    )
-    (property "Footprint" "Mechatronics TestP:CONN1_RCU-0C_TEC" (at 93.472 123.952 0)
-      (effects (font (size 1.27 1.27)) hide)
-    )
-    (property "Datasheet" "~" (at 93.472 123.952 0)
-      (effects (font (size 1.27 1.27)) hide)
-    )
-    (pin "1")
-    (instances
-      (project "rps01"
-        (path "/14930f15-c0a0-4b55-93e6-b112548415f6/577d3fc4-735f-4981-a3a1-4300f23b9ae6"
-          (reference "TP9") (unit 1)
-        )
-      )
-    )
-  )
-  (symbol (lib_id "Connector:TestPoint_Probe") (at 88.392 117.094 0) (unit 1)
-    (in_bom yes) (on_board yes) (dnp no) (fields_autoplaced)
-    (property "Reference" "TP8" (at 92.71 114.8715 0)
-      (effects (font (size 1.27 1.27)) (justify left))
-    )
-    (property "Value" "VOLT2" (at 92.71 117.4115 0)
-      (effects (font (size 1.27 1.27)) (justify left))
-    )
-    (property "Footprint" "Mechatronics TestP:CONN1_RCU-0C_TEC" (at 93.472 117.094 0)
-      (effects (font (size 1.27 1.27)) hide)
-    )
-    (property "Datasheet" "~" (at 93.472 117.094 0)
-      (effects (font (size 1.27 1.27)) hide)
-    )
-    (pin "1")
-    (instances
-      (project "rps01"
-        (path "/14930f15-c0a0-4b55-93e6-b112548415f6/577d3fc4-735f-4981-a3a1-4300f23b9ae6"
-          (reference "TP8") (unit 1)
-        )
-      )
-    )
-  )
-  (symbol (lib_id "Connector:TestPoint_Probe") (at 88.138 103.632 0) (unit 1)
-    (in_bom yes) (on_board yes) (dnp no) (fields_autoplaced)
-    (property "Reference" "TP6" (at 92.71 101.4095 0)
-      (effects (font (size 1.27 1.27)) (justify left))
-    )
-    (property "Value" "CURRENT2" (at 92.71 103.9495 0)
-      (effects (font (size 1.27 1.27)) (justify left))
-    )
-    (property "Footprint" "Mechatronics TestP:CONN1_RCU-0C_TEC" (at 93.218 103.632 0)
-      (effects (font (size 1.27 1.27)) hide)
-    )
-    (property "Datasheet" "~" (at 93.218 103.632 0)
-      (effects (font (size 1.27 1.27)) hide)
-    )
-    (pin "1")
-    (instances
-      (project "rps01"
-        (path "/14930f15-c0a0-4b55-93e6-b112548415f6/577d3fc4-735f-4981-a3a1-4300f23b9ae6"
-          (reference "TP6") (unit 1)
-        )
-      )
-    )
-  )
   (symbol (lib_id "power:GND") (at 143.002 99.314 0) (unit 1)
     (in_bom yes) (on_board yes) (dnp no) (fields_autoplaced)
@@
         )
       )
-    )
-  )
-  (symbol (lib_id "Connector:TestPoint_Probe") (at 88.138 97.028 0) (unit 1)
-    (in_bom yes) (on_board yes) (dnp no) (fields_autoplaced)
-    (property "Reference" "TP5" (at 92.71 94.8055 0)
-      (effects (font (size 1.27 1.27)) (justify left))
-    )
-    (property "Value" "CURRENT1" (at 92.71 97.3455 0)
-      (effects (font (size 1.27 1.27)) (justify left))
-    )
-    (property "Footprint" "Mechatronics TestP:CONN1_RCU-0C_TEC" (at 93.218 97.028 0)
-      (effects (font (size 1.27 1.27)) hide)
-    )
-    (property "Datasheet" "~" (at 93.218 97.028 0)
-      (effects (font (size 1.27 1.27)) hide)
-    )
-    (pin "1")
-    (instances
-      (project "rps01"
-        (path "/14930f15-c0a0-4b55-93e6-b112548415f6/577d3fc4-735f-4981-a3a1-4300f23b9ae6"
-          (reference "TP5") (unit 1)
-        )
-      )
